Commit message: Afjusted ROSbot model frame name to comply with ROS standard

File: src/rosbot_description/urdf/rosbot.xacro (robot description, xacro)
@@ -6,5 +6,5 @@
   <xacro:include filename="$(find rosbot_description)/urdf/materials.xacro" />
   <xacro:include filename="$(find rosbot_description)/urdf/macros.xacro" />
-  <link name='chassis'>
+  <link name='base_frame'>
     <pose>0 0 0.1 0 0 0</pose>
     <inertial>
@@ -22,5 +22,5 @@
       </geometry>
     </collision>
-    <visual name='chassis_visual'>
+    <visual name='base_frame_visual'>
       <origin xyz="0 0 -0.06" rpy=" 1.5707 0 1.5707"/>
       <geometry>
@@ -32,5 +32,5 @@
     <axis xyz="0 1 0" />
     <origin xyz="0 0 0" rpy="0 0 0"/>
-    <parent link="chassis"/>
+    <parent link="base_frame"/>
     <child link="top"/>
   </joint>
@@ -144,5 +144,5 @@
     <origin xyz="0.1 0.15 0" rpy="0 0 0"/>
     <child link="front_left_wheel"/>
-    <parent link="chassis"/>
+    <parent link="base_frame"/>
     <axis xyz="0 1 0" rpy="0 0 0"/>
     <limit effort="10000" velocity="1000"/>
@@ -152,5 +152,5 @@
     <origin xyz="0.1 -0.15 0" rpy="0 0 0"/>
     <child link="front_right_wheel"/>
-    <parent link="chassis"/>
+    <parent link="base_frame"/>
     <axis xyz="0 1 0" rpy="0 0 0"/>
     <limit effort="10000" velocity="1000"/>
@@ -160,5 +160,5 @@
     <origin xyz="-0.12 0.15 0" rpy="0 0 0"/>
     <child link="rear_left_wheel"/>
-    <parent link="chassis"/>
+    <parent link="base_frame"/>
     <axis xyz="0 1 0" rpy="0 0 0"/>
     <limit effort="10000" velocity="1000"/>
@@ -168,5 +168,5 @@
     <origin xyz="-0.12 -0.15 0" rpy="0 0 0"/>
     <child link="rear_right_wheel"/>
-    <parent link="chassis"/>
+    <parent link="base_frame"/>
     <axis xyz="0 1 0" rpy="0 0 0"/>
     <limit effort="10000" velocity="1000"/>
@@ -177,5 +177,5 @@
     <axis xyz="0 0 0" />
     <origin xyz="-0.055 0 0.308" rpy="0 0 0"/>
-    <parent link="chassis"/>
+    <parent link="base_frame"/>
     <child link="astra"/>
   </joint>
@@ -202,5 +202,5 @@
     <axis xyz="0 1 0" />
     <origin xyz="0.08 0 0.12" rpy="0 0 0"/>
-    <parent link="chassis"/>
+    <parent link="base_frame"/>
     <child link="rplidar"/>
   </joint>

Commit message: Added range sensors to model

File: src/rosbot_description/urdf/rosbot.xacro (robot description, xacro)
@@ -12,7 +12,7 @@
       <origin xyz="0 0 0.1" rpy=" 0 0 0"/>
       <inertia
-          ixx="0.1" ixy="0" ixz="0"
-          iyy="0.1" iyz="0"
-          izz="0.1"
+      ixx="0.1" ixy="0" ixz="0"
+      iyy="0.1" iyz="0"
+      izz="0.1"
       />
     </inertial>
@@ -41,7 +41,7 @@
       <origin xyz="0 0 0.1" rpy=" 0 0 0"/>
       <inertia
-          ixx="0.1" ixy="0" ixz="0"
-          iyy="0.1" iyz="0"
-          izz="0.1"
+      ixx="0.1" ixy="0" ixz="0"
+      iyy="0.1" iyz="0"
+      izz="0.1"
       />
     </inertial>
@@ -70,7 +70,7 @@
       <mass value="5"/>
       <inertia
-        ixx=".1" ixy="0.0" ixz="0.0"
-        iyy=".1" iyz="0.0"
-        izz=".1"/>
+      ixx=".1" ixy="0.0" ixz="0.0"
+      iyy=".1" iyz="0.0"
+      izz=".1"/>
     </inertial>
   </link>
@@ -92,10 +92,10 @@
       <mass value="5"/>
       <inertia
-        ixx=".1" ixy="0.0" ixz="0.0"
-        iyy=".1" iyz="0.0"
-        izz=".1"/>
-    </inertial>
-  </link>
-    <link name="rear_left_wheel">
+      ixx=".1" ixy="0.0" ixz="0.0"
+      iyy=".1" iyz="0.0"
+      izz=".1"/>
+    </inertial>
+  </link>
+  <link name="rear_left_wheel">
     <collision name="collision">
       <origin xyz="0 0.07 0" rpy="0 0 1.5707"/>
@@ -114,7 +114,7 @@
       <mass value="5"/>
       <inertia
-        ixx=".1" ixy="0.0" ixz="0.0"
-        iyy=".1" iyz="0.0"
-        izz=".1"/>
+      ixx=".1" ixy="0.0" ixz="0.0"
+      iyy=".1" iyz="0.0"
+      izz=".1"/>
     </inertial>
   </link>
@@ -136,7 +136,7 @@
       <mass value="5"/>
       <inertia
-        ixx=".1" ixy="0.0" ixz="0.0"
-        iyy=".1" iyz="0.0"
-        izz=".1"/>
+      ixx=".1" ixy="0.0" ixz="0.0"
+      iyy=".1" iyz="0.0"
+      izz=".1"/>
     </inertial>
   </link>
@@ -184,5 +184,5 @@
       <origin xyz="0.02 0 0" rpy="0 0 0"/>
       <geometry>0
-    <box size="0.01 0.01 0.01"/>
+        <box size="0.01 0.01 0.01"/>
       </geometry>
     </collision>
@@ -210,5 +210,5 @@
       <origin xyz="0 0 0" rpy="0 0 0"/>
       <geometry>
-    <box size="0.1 0.1 0.1"/>
+        <box size="0.1 0.1 0.1"/>
       </geometry>
     </collision>
@@ -225,3 +225,31 @@
     </inertial>
   </link>
+  <joint name="range_fl_joint" type="fixed">
+    <axis xyz="0 1 0" />
+    <origin xyz="0.2 0.1 0.005" rpy="0 0 0 "/>
+    <parent link="base_frame"/>
+    <child link="range_fl"/>
+  </joint>
+  <link name="range_fl"></link>
+  <joint name="range_fr_joint" type="fixed">
+    <axis xyz="0 1 0" />
+    <origin xyz="0.2 -0.1 0.005" rpy="0 0 0 "/>
+    <parent link="base_frame"/>
+    <child link="range_fr"/>
+  </joint>
+  <link name="range_fr"></link>
+  <joint name="range_rl_joint" type="fixed">
+    <axis xyz="0 1 0" />
+    <origin xyz="-0.2 0.1 0.005" rpy="0 0 3.14 "/>
+    <parent link="base_frame"/>
+    <child link="range_rl"/>
+  </joint>
+  <link name="range_rl"></link>
+  <joint name="range_rr_joint" type="fixed">
+    <axis xyz="0 1 0" />
+    <origin xyz="-0.2 -0.1 0.005" rpy="0 0 3.14 "/>
+    <parent link="base_frame"/>
+    <child link="range_rr"/>
+  </joint>
+  <link name="range_rr"></link>
 </robot>

Commit message: range sensors param update

File: src/rosbot_description/urdf/rosbot.xacro (robot description, xacro)
@@ -227,5 +227,5 @@
   <joint name="range_fl_joint" type="fixed">
     <axis xyz="0 1 0" />
-    <origin xyz="0.2 0.1 0.005" rpy="0 0 0 "/>
+    <origin xyz="0.2 0.1 0.005" rpy="0 0 0.13 "/>
     <parent link="base_frame"/>
     <child link="range_fl"/>
@@ -234,5 +234,5 @@
   <joint name="range_fr_joint" type="fixed">
     <axis xyz="0 1 0" />
-    <origin xyz="0.2 -0.1 0.005" rpy="0 0 0 "/>
+    <origin xyz="0.2 -0.1 0.005" rpy="0 0 -0.13 "/>
     <parent link="base_frame"/>
     <child link="range_fr"/>
@@ -241,5 +241,5 @@
   <joint name="range_rl_joint" type="fixed">
     <axis xyz="0 1 0" />
-    <origin xyz="-0.2 0.1 0.005" rpy="0 0 3.14 "/>
+    <origin xyz="-0.2 0.1 0.005" rpy="0 0 3.01 "/>
     <parent link="base_frame"/>
     <child link="range_rl"/>
@@ -248,5 +248,5 @@
   <joint name="range_rr_joint" type="fixed">
     <axis xyz="0 1 0" />
-    <origin xyz="-0.2 -0.1 0.005" rpy="0 0 3.14 "/>
+    <origin xyz="-0.2 -0.1 0.005" rpy="0 0 3.27 "/>
     <parent link="base_frame"/>
     <child link="range_rr"/>

Commit message: URDF model update

File: src/rosbot_description/urdf/rosbot.xacro (robot description, xacro)
@@ -9,6 +9,36 @@
     <pose>0 0 0.1 0 0 0</pose>
     <inertial>
-      <mass value="30.0"/>
-      <origin xyz="0 0 0.1" rpy=" 0 0 0"/>
+      <mass value="50.0"/>
+      <origin xyz="0 0 0.04" rpy=" 0 0 0"/>
+      <inertia
+      ixx="10" ixy="1" ixz="0"
+      iyy="10" iyz="1"
+      izz="10"
+      />
+    </inertial>
+    <collision name='collision'>
+      <origin xyz="0 0 0.02" rpy="0 0 0"/>
+      <geometry>
+        <box size="0.22 0.15 0.04"/>
+      </geometry>
+    </collision>
+    <visual name='base_frame_visual'>
+      <origin xyz="0 0 -0.02" rpy=" 1.5707 0 1.5707"/>
+      <geometry>
+        <mesh filename="package://rosbot_description/meshes/box.dae" scale="0.001 0.001 0.001" />
+      </geometry>
+    </visual>
+  </link>
+  <joint name="top_joint" type="fixed">
+    <axis xyz="0 1 0" />
+    <origin xyz="0 0 0" rpy="0 0 0"/>
+    <parent link="base_frame"/>
+    <child link="top"/>
+  </joint>
+  <link name='top'>
+    <pose>0 0 0 0 0 0</pose>
+    <inertial>
+      <mass value="50.0"/>
+      <origin xyz="0 0 0.055" rpy=" 0 0 0"/>
       <inertia
       ixx="0.1" ixy="0" ixz="0"
@@ -17,37 +47,8 @@
       />
     </inertial>
-    <collision name='collision'>
-      <geometry>
-        <box size=".4 .2 .1"/>
-      </geometry>
-    </collision>
-    <visual name='base_frame_visual'>
-      <origin xyz="0 0 -0.06" rpy=" 1.5707 0 1.5707"/>
-      <geometry>
-        <mesh filename="package://rosbot_description/meshes/box.dae" scale="0.002 0.002 0.002" />
-      </geometry>
-    </visual>
-  </link>
-  <joint name="top_joint" type="fixed">
-    <axis xyz="0 1 0" />
-    <origin xyz="0 0 0" rpy="0 0 0"/>
-    <parent link="base_frame"/>
-    <child link="top"/>
-  </joint>
-  <link name='top'>
-    <pose>0 0 0.1 0 0 0</pose>
-    <inertial>
-      <mass value="30.0"/>
-      <origin xyz="0 0 0.1" rpy=" 0 0 0"/>
-      <inertia
-      ixx="0.1" ixy="0" ixz="0"
-      iyy="0.1" iyz="0"
-      izz="0.1"
-      />
-    </inertial>
     <visual name='top'>
-      <origin xyz="0 0 0.09" rpy=" 1.5707 0 1.5707"/>
-      <geometry>
-        <mesh filename="package://rosbot_description/meshes/upper.dae" scale="0.002 0.002 0.002" />
+      <origin xyz="0 0 0.055" rpy=" 1.5707 0 1.5707"/>
+      <geometry>
+        <mesh filename="package://rosbot_description/meshes/upper.dae" scale="0.001 0.001 0.001" />
       </geometry>
     </visual>
@@ -55,18 +56,18 @@
   <link name="front_left_wheel">
     <collision name="collision">
-      <origin xyz="0 0.07 0" rpy="0 0 1.5707"/>
-      <geometry>
-        <mesh filename="package://rosbot_description/meshes/wheel.dae" scale="0.002 0.002 0.002" />
+      <origin xyz="0 0.06 0" rpy="0 0 1.5707"/>
+      <geometry>
+        <mesh filename="package://rosbot_description/meshes/wheel.dae" scale="0.001 0.001 0.001" />
       </geometry>
     </collision>
     <visual name="front_left_wheel_visual">
-      <origin xyz="0 0.07 0" rpy="0 0 1.5707"/>
-      <geometry>
-        <mesh filename="package://rosbot_description/meshes/wheel.dae" scale="0.002 0.002 0.002" />
-      </geometry>
-    </visual>
-    <inertial>
-      <origin xyz="0 0 0" rpy="0 1.5707 1.5707"/>
-      <mass value="5"/>
+      <origin xyz="0 0.06 0" rpy="0 0 1.5707"/>
+      <geometry>
+        <mesh filename="package://rosbot_description/meshes/wheel.dae" scale="0.001 0.001 0.001" />
+      </geometry>
+    </visual>
+    <inertial>
+      <origin xyz="0 0 0" rpy="0 1.5707 1.5707"/>
+      <mass value="40"/>
       <inertia
       ixx=".1" ixy="0.0" ixz="0.0"
@@ -77,18 +78,18 @@
   <link name="front_right_wheel">
     <collision name="collision">
-      <origin xyz="0 -0.07 0" rpy="0 0 -1.5707"/>
-      <geometry>
-        <mesh filename="package://rosbot_description/meshes/wheel.dae" scale="0.002 0.002 0.002" />
+      <origin xyz="0 -0.06 0" rpy="0 0 -1.5707"/>
+      <geometry>
+        <mesh filename="package://rosbot_description/meshes/wheel.dae" scale="0.001 0.001 0.001" />
       </geometry>
     </collision>
     <visual name="front_right_wheel_visual">
-      <origin xyz="0 -0.07 0" rpy="0 0 -1.5707"/>
-      <geometry>
-        <mesh filename="package://rosbot_description/meshes/wheel.dae" scale="0.002 0.002 0.002" />
-      </geometry>
-    </visual>
-    <inertial>
-      <origin xyz="0 0 0" rpy="0 1.5707 1.5707"/>
-      <mass value="5"/>
+      <origin xyz="0 -0.06 0" rpy="0 0 -1.5707"/>
+      <geometry>
+        <mesh filename="package://rosbot_description/meshes/wheel.dae" scale="0.001 0.001 0.001" />
+      </geometry>
+    </visual>
+    <inertial>
+      <origin xyz="0 0 0" rpy="0 1.5707 1.5707"/>
+      <mass value="40"/>
       <inertia
       ixx=".1" ixy="0.0" ixz="0.0"
@@ -99,18 +100,18 @@
   <link name="rear_left_wheel">
     <collision name="collision">
-      <origin xyz="0 0.07 0" rpy="0 0 1.5707"/>
-      <geometry>
-        <mesh filename="package://rosbot_description/meshes/wheel.dae" scale="0.002 0.002 0.002" />
+      <origin xyz="0 0.06 0" rpy="0 0 1.5707"/>
+      <geometry>
+        <mesh filename="package://rosbot_description/meshes/wheel.dae" scale="0.001 0.001 0.001" />
       </geometry>
     </collision>
     <visual name="rear_left_wheel_visual">
-      <origin xyz="0 0.07 0" rpy="0 0 1.5707"/>
-      <geometry>
-        <mesh filename="package://rosbot_description/meshes/wheel.dae" scale="0.002 0.002 0.002" />
-      </geometry>
-    </visual>
-    <inertial>
-      <origin xyz="0 0 0" rpy="0 1.5707 1.5707"/>
-      <mass value="5"/>
+      <origin xyz="0 0.06 0" rpy="0 0 1.5707"/>
+      <geometry>
+        <mesh filename="package://rosbot_description/meshes/wheel.dae" scale="0.001 0.001 0.001" />
+      </geometry>
+    </visual>
+    <inertial>
+      <origin xyz="0 0 0" rpy="0 1.5707 1.5707"/>
+      <mass value="40"/>
       <inertia
       ixx=".1" ixy="0.0" ixz="0.0"
@@ -121,18 +122,18 @@
   <link name="rear_right_wheel">
     <collision name="collision">
-      <origin xyz="0 -0.07 0" rpy="0 0 -1.5707"/>
-      <geometry>
-        <mesh filename="package://rosbot_description/meshes/wheel.dae" scale="0.002 0.002 0.002" />
+      <origin xyz="0 -0.06 0" rpy="0 0 -1.5707"/>
+      <geometry>
+        <mesh filename="package://rosbot_description/meshes/wheel.dae" scale="0.001 0.001 0.001" />
       </geometry>
     </collision>
     <visual name="rear_right_wheel_visual">
-      <origin xyz="0 -0.07 0" rpy="0 0 -1.5707"/>
-      <geometry>
-        <mesh filename="package://rosbot_description/meshes/wheel.dae" scale="0.002 0.002 0.002" />
-      </geometry>
-    </visual>
-    <inertial>
-      <origin xyz="0 0 0" rpy="0 1.5707 1.5707"/>
-      <mass value="5"/>
+      <origin xyz="0 -0.06 0" rpy="0 0 -1.5707"/>
+      <geometry>
+        <mesh filename="package://rosbot_description/meshes/wheel.dae" scale="0.001 0.001 0.001" />
+      </geometry>
+    </visual>
+    <inertial>
+      <origin xyz="0 0 0" rpy="0 1.5707 1.5707"/>
+      <mass value="40"/>
       <inertia
       ixx=".1" ixy="0.0" ixz="0.0"
@@ -142,39 +143,39 @@
   </link>
   <joint type="continuous" name="front_left_wheel_hinge">
-    <origin xyz="0.1 0.15 0" rpy="0 0 0"/>
+    <origin xyz="0.05 0.05 0" rpy="0 0 0"/>
     <child link="front_left_wheel"/>
     <parent link="base_frame"/>
     <axis xyz="0 1 0" rpy="0 0 0"/>
     <limit effort="10000" velocity="1000"/>
-    <joint_properties damping="1.0" friction="1.0"/>
+    <joint_properties damping="5.0" friction="1.0"/>
   </joint>
   <joint type="continuous" name="front_right_wheel_hinge">
-    <origin xyz="0.1 -0.15 0" rpy="0 0 0"/>
+    <origin xyz="0.05 -0.05 0" rpy="0 0 0"/>
     <child link="front_right_wheel"/>
     <parent link="base_frame"/>
     <axis xyz="0 1 0" rpy="0 0 0"/>
     <limit effort="10000" velocity="1000"/>
-    <joint_properties damping="1.0" friction="1.0"/>
+    <joint_properties damping="5.0" friction="1.0"/>
   </joint>
   <joint type="continuous" name="rear_left_wheel_hinge">
-    <origin xyz="-0.12 0.15 0" rpy="0 0 0"/>
+    <origin xyz="-0.055 0.05 0" rpy="0 0 0"/>
     <child link="rear_left_wheel"/>
     <parent link="base_frame"/>
     <axis xyz="0 1 0" rpy="0 0 0"/>
     <limit effort="10000" velocity="1000"/>
-    <joint_properties damping="1.0" friction="1.0"/>
+    <joint_properties damping="5.0" friction="1.0"/>
   </joint>
   <joint type="continuous" name="rear_right_wheel_hinge">
-    <origin xyz="-0.12 -0.15 0" rpy="0 0 0"/>
+    <origin xyz="-0.055 -0.05 0" rpy="0 0 0"/>
     <child link="rear_right_wheel"/>
     <parent link="base_frame"/>
     <axis xyz="0 1 0" rpy="0 0 0"/>
     <limit effort="10000" velocity="1000"/>
-    <joint_properties damping="1.0" friction="1.0"/>
+    <joint_properties damping="5.0" friction="1.0"/>
   </joint>
   <!-- Orbbec Astra RGBD Camera -->
   <joint name="astra_joint" type="fixed">
     <axis xyz="0 0 0" />
-    <origin xyz="-0.055 0 0.308" rpy="0 0 0"/>
+    <origin xyz="-0.03 0 0.18" rpy="0 0 0"/>
     <parent link="base_frame"/>
     <child link="astra"/>
@@ -184,5 +185,5 @@
       <origin xyz="0.02 0 0" rpy="0 0 0"/>
       <geometry>0
-        <box size="0.01 0.01 0.01"/>
+        <box size="0.001 0.001 0.001"/>
       </geometry>
     </collision>
@@ -190,5 +191,5 @@
       <origin xyz="-0.01 0 -0.03" rpy="1.5707 0 1.5707"/>
       <geometry>
-        <mesh filename="package://rosbot_description/meshes/astra.dae" scale="0.002 0.002 0.002" />
+        <mesh filename="package://rosbot_description/meshes/astra.dae" scale="0.001 0.001 0.001" />
       </geometry>
     </visual>
@@ -201,5 +202,5 @@
   <joint name="rplidar_joint" type="fixed">
     <axis xyz="0 1 0" />
-    <origin xyz="0.08 0 0.12" rpy="0 0 0"/>
+    <origin xyz="0.02 0 0.086" rpy="0 0 0"/>
     <parent link="base_frame"/>
     <child link="rplidar"/>
@@ -210,5 +211,5 @@
       <origin xyz="0 0 0" rpy="0 0 0"/>
       <geometry>
-        <box size="0.1 0.1 0.1"/>
+        <box size="0.001 0.001 0.001"/>
       </geometry>
     </collision>
@@ -216,5 +217,5 @@
       <origin xyz="0 0 -0.03" rpy="1.5707 0 1.5707"/>
       <geometry>
-        <mesh filename="package://rosbot_description/meshes/rplidar.dae" scale="0.002 0.002 0.002" />
+        <mesh filename="package://rosbot_description/meshes/rplidar.dae" scale="0.001 0.001 0.001" />
       </geometry>
     </visual>
@@ -227,5 +228,5 @@
   <joint name="range_fl_joint" type="fixed">
     <axis xyz="0 1 0" />
-    <origin xyz="0.2 0.1 0.005" rpy="0 0 0.13 "/>
+    <origin xyz="0.1 0.05 0.01" rpy="0 0 0.13 "/>
     <parent link="base_frame"/>
     <child link="range_fl"/>
@@ -234,5 +235,5 @@
   <joint name="range_fr_joint" type="fixed">
     <axis xyz="0 1 0" />
-    <origin xyz="0.2 -0.1 0.005" rpy="0 0 -0.13 "/>
+    <origin xyz="0.1 -0.05 0.01" rpy="0 0 -0.13 "/>
     <parent link="base_frame"/>
     <child link="range_fr"/>
@@ -241,5 +242,5 @@
   <joint name="range_rl_joint" type="fixed">
     <axis xyz="0 1 0" />
-    <origin xyz="-0.2 0.1 0.005" rpy="0 0 3.01 "/>
+    <origin xyz="-0.1 0.05 0.01" rpy="0 0 3.01 "/>
     <parent link="base_frame"/>
     <child link="range_rl"/>
@@ -248,5 +249,5 @@
   <joint name="range_rr_joint" type="fixed">
     <axis xyz="0 1 0" />
-    <origin xyz="-0.2 -0.1 0.005" rpy="0 0 3.27 "/>
+    <origin xyz="-0.1 -0.05 0.01" rpy="0 0 3.27 "/>
     <parent link="base_frame"/>
     <child link="range_rr"/>

Commit message: Changed frame names to comply with ROS REP 105

File: src/rosbot_description/urdf/rosbot.xacro (robot description, xacro)
@@ -6,5 +6,5 @@
   <xacro:include filename="$(find rosbot_description)/urdf/materials.xacro" />
   <xacro:include filename="$(find rosbot_description)/urdf/macros.xacro" />
-  <link name='base_frame'>
+  <link name='base_link'>
     <pose>0 0 0.1 0 0 0</pose>
     <inertial>
@@ -23,5 +23,5 @@
       </geometry>
     </collision>
-    <visual name='base_frame_visual'>
+    <visual name='base_link_visual'>
       <origin xyz="0 0 -0.02" rpy=" 1.5707 0 1.5707"/>
       <geometry>
@@ -33,5 +33,5 @@
     <axis xyz="0 1 0" />
     <origin xyz="0 0 0" rpy="0 0 0"/>
-    <parent link="base_frame"/>
+    <parent link="base_link"/>
     <child link="top"/>
   </joint>
@@ -145,5 +145,5 @@
     <origin xyz="0.05 0.05 0" rpy="0 0 0"/>
     <child link="front_left_wheel"/>
-    <parent link="base_frame"/>
+    <parent link="base_link"/>
     <axis xyz="0 1 0" rpy="0 0 0"/>
     <limit effort="10000" velocity="1000"/>
@@ -153,5 +153,5 @@
     <origin xyz="0.05 -0.05 0" rpy="0 0 0"/>
     <child link="front_right_wheel"/>
-    <parent link="base_frame"/>
+    <parent link="base_link"/>
     <axis xyz="0 1 0" rpy="0 0 0"/>
     <limit effort="10000" velocity="1000"/>
@@ -161,5 +161,5 @@
     <origin xyz="-0.055 0.05 0" rpy="0 0 0"/>
     <child link="rear_left_wheel"/>
-    <parent link="base_frame"/>
+    <parent link="base_link"/>
     <axis xyz="0 1 0" rpy="0 0 0"/>
     <limit effort="10000" velocity="1000"/>
@@ -169,5 +169,5 @@
     <origin xyz="-0.055 -0.05 0" rpy="0 0 0"/>
     <child link="rear_right_wheel"/>
-    <parent link="base_frame"/>
+    <parent link="base_link"/>
     <axis xyz="0 1 0" rpy="0 0 0"/>
     <limit effort="10000" velocity="1000"/>
@@ -178,5 +178,5 @@
     <axis xyz="0 0 0" />
     <origin xyz="-0.03 0 0.18" rpy="0 0 0"/>
-    <parent link="base_frame"/>
+    <parent link="base_link"/>
     <child link="astra"/>
   </joint>
@@ -202,6 +202,6 @@
   <joint name="rplidar_joint" type="fixed">
     <axis xyz="0 1 0" />
-    <origin xyz="0.02 0 0.086" rpy="0 0 0"/>
-    <parent link="base_frame"/>
+    <origin xyz="0.02 0 0.086" rpy="0 0 3.14"/>
+    <parent link="base_link"/>
     <child link="rplidar"/>
   </joint>
@@ -229,5 +229,5 @@
     <axis xyz="0 1 0" />
     <origin xyz="0.1 0.05 0.01" rpy="0 0 0.13 "/>
-    <parent link="base_frame"/>
+    <parent link="base_link"/>
     <child link="range_fl"/>
   </joint>
@@ -236,5 +236,5 @@
     <axis xyz="0 1 0" />
     <origin xyz="0.1 -0.05 0.01" rpy="0 0 -0.13 "/>
-    <parent link="base_frame"/>
+    <parent link="base_link"/>
     <child link="range_fr"/>
   </joint>
@@ -243,5 +243,5 @@
     <axis xyz="0 1 0" />
     <origin xyz="-0.1 0.05 0.01" rpy="0 0 3.01 "/>
-    <parent link="base_frame"/>
+    <parent link="base_link"/>
     <child link="range_rl"/>
   </joint>
@@ -250,5 +250,5 @@
     <axis xyz="0 1 0" />
     <origin xyz="-0.1 -0.05 0.01" rpy="0 0 3.27 "/>
-    <parent link="base_frame"/>
+    <parent link="base_link"/>
     <child link="range_rr"/>
   </joint>

Commit message: urdf update

File: src/rosbot_description/urdf/rosbot.xacro (robot description, xacro)
@@ -20,5 +20,5 @@
       <origin xyz="0 0 0.02" rpy="0 0 0"/>
       <geometry>
-        <box size="0.22 0.15 0.04"/>
+        <box size="0.20 0.15 0.04"/>
       </geometry>
     </collision>

Commit message: urdf update

File: src/rosbot_description/urdf/rosbot.xacro (robot description, xacro)
@@ -215,5 +215,5 @@
     </collision>
     <visual>
-      <origin xyz="0 0 -0.03" rpy="1.5707 0 1.5707"/>
+      <origin xyz="0 0 -0.03" rpy="1.5707 0 4.71"/>
       <geometry>
         <mesh filename="package://rosbot_description/meshes/rplidar.dae" scale="0.001 0.001 0.001" />

Commit message: Added astra optical frame to align image correctly.

File: src/rosbot_description/urdf/rosbot.xacro (robot description, xacro)
@@ -200,4 +200,11 @@
     </inertial>
   </link>
+<joint name="camera_optical_joint" type="fixed">
+  <origin xyz="0 0 0" rpy="${-pi/2} 0 ${-pi/2}"/>
+  <parent link="astra"/>
+  <child link="astra_optical"/>
+</joint>
+<link name="astra_optical">
+</link>
   <joint name="rplidar_joint" type="fixed">
     <axis xyz="0 1 0" />

Commit message: Added link to publish camera depth frame

File: src/rosbot_description/urdf/rosbot.xacro (robot description, xacro)
@@ -207,4 +207,11 @@
 <link name="astra_optical">
 </link>
+<joint name="camera_depth_joint" type="fixed">
+  <origin xyz="0 0 0" rpy="0 0 0"/>
+  <parent link="astra"/>
+  <child link="camera_depth_frame"/>
+</joint>
+<link name="camera_depth_frame">
+</link>
   <joint name="rplidar_joint" type="fixed">
     <axis xyz="0 1 0" />
