Commit message: Updated ROSbot model

File: src/rosbot_description/urdf/rosbot.xacro (robot description, xacro)
@@ -9,10 +9,10 @@
     <pose>0 0 0.1 0 0 0</pose>
     <inertial>
-      <mass value="50.0"/>
+      <mass value="5"/>
       <origin xyz="0 0 0.04" rpy=" 0 0 0"/>
       <inertia
-      ixx="10" ixy="1" ixz="0"
-      iyy="10" iyz="1"
-      izz="10"
+      ixx="0.01" ixy="0.01" ixz="0"
+      iyy="0.01" iyz="0.01"
+      izz="0.01"
       />
     </inertial>
@@ -39,10 +39,10 @@
     <pose>0 0 0 0 0 0</pose>
     <inertial>
-      <mass value="50.0"/>
+      <mass value="0.01"/>
       <origin xyz="0 0 0.055" rpy=" 0 0 0"/>
       <inertia
-      ixx="0.1" ixy="0" ixz="0"
-      iyy="0.1" iyz="0"
-      izz="0.1"
+      ixx="0.0" ixy="0" ixz="0"
+      iyy="0.0" iyz="0"
+      izz="0.0"
       />
     </inertial>
@@ -56,11 +56,19 @@
   <link name="front_left_wheel">
     <collision name="collision">
-      <origin xyz="0 0.06 0" rpy="0 0 1.5707"/>
-      <geometry>
-        <mesh filename="package://rosbot_description/meshes/wheel.dae" scale="0.001 0.001 0.001" />
-      </geometry>
+      <origin xyz="0 0 0" rpy="0 0 1.5707"/>
+      <geometry>
+        <mesh filename="package://rosbot_description/meshes/wheel.dae" scale="0.001 0.001 0.001" />
+      </geometry>
+      <surface>
+        <friction>
+          <ode>
+            <mu>10</mu>
+            <mu2>10</mu2>
+          </ode>
+        </friction>
+      </surface>
     </collision>
     <visual name="front_left_wheel_visual">
-      <origin xyz="0 0.06 0" rpy="0 0 1.5707"/>
+      <origin xyz="0 0 0" rpy="0 0 1.5707"/>
       <geometry>
         <mesh filename="package://rosbot_description/meshes/wheel.dae" scale="0.001 0.001 0.001" />
@@ -69,20 +77,28 @@
     <inertial>
       <origin xyz="0 0 0" rpy="0 1.5707 1.5707"/>
-      <mass value="40"/>
-      <inertia
-      ixx=".1" ixy="0.0" ixz="0.0"
-      iyy=".1" iyz="0.0"
-      izz=".1"/>
+      <mass value="0.5"/>
+      <inertia
+      ixx="0.001" ixy="0.0" ixz="0.0"
+      iyy="0.001" iyz="0.0"
+      izz="0.001"/>
     </inertial>
   </link>
   <link name="front_right_wheel">
     <collision name="collision">
-      <origin xyz="0 -0.06 0" rpy="0 0 -1.5707"/>
-      <geometry>
-        <mesh filename="package://rosbot_description/meshes/wheel.dae" scale="0.001 0.001 0.001" />
-      </geometry>
+      <origin xyz="0 0 0" rpy="0 0 -1.5707"/>
+      <geometry>
+        <mesh filename="package://rosbot_description/meshes/wheel.dae" scale="0.001 0.001 0.001" />
+      </geometry>
+      <surface>
+        <friction>
+          <ode>
+            <mu>10</mu>
+            <mu2>10</mu2>
+          </ode>
+        </friction>
+      </surface>
     </collision>
     <visual name="front_right_wheel_visual">
-      <origin xyz="0 -0.06 0" rpy="0 0 -1.5707"/>
+      <origin xyz="0 0 0" rpy="0 0 -1.5707"/>
       <geometry>
         <mesh filename="package://rosbot_description/meshes/wheel.dae" scale="0.001 0.001 0.001" />
@@ -91,20 +107,28 @@
     <inertial>
       <origin xyz="0 0 0" rpy="0 1.5707 1.5707"/>
-      <mass value="40"/>
-      <inertia
-      ixx=".1" ixy="0.0" ixz="0.0"
-      iyy=".1" iyz="0.0"
-      izz=".1"/>
+      <mass value="0.5"/>
+      <inertia
+      ixx="0.001" ixy="0.0" ixz="0.0"
+      iyy="0.001" iyz="0.0"
+      izz="0.001"/>
     </inertial>
   </link>
   <link name="rear_left_wheel">
     <collision name="collision">
-      <origin xyz="0 0.06 0" rpy="0 0 1.5707"/>
-      <geometry>
-        <mesh filename="package://rosbot_description/meshes/wheel.dae" scale="0.001 0.001 0.001" />
-      </geometry>
+      <origin xyz="0 0 0" rpy="0 0 1.5707"/>
+      <geometry>
+        <mesh filename="package://rosbot_description/meshes/wheel.dae" scale="0.001 0.001 0.001" />
+      </geometry>
+      <surface>
+        <friction>
+          <ode>
+            <mu>10</mu>
+            <mu2>10</mu2>
+          </ode>
+        </friction>
+      </surface>
     </collision>
     <visual name="rear_left_wheel_visual">
-      <origin xyz="0 0.06 0" rpy="0 0 1.5707"/>
+      <origin xyz="0 0 0" rpy="0 0 1.5707"/>
       <geometry>
         <mesh filename="package://rosbot_description/meshes/wheel.dae" scale="0.001 0.001 0.001" />
@@ -113,20 +137,28 @@
     <inertial>
       <origin xyz="0 0 0" rpy="0 1.5707 1.5707"/>
-      <mass value="40"/>
-      <inertia
-      ixx=".1" ixy="0.0" ixz="0.0"
-      iyy=".1" iyz="0.0"
-      izz=".1"/>
+      <mass value="0.5"/>
+      <inertia
+      ixx="0.001" ixy="0.0" ixz="0.0"
+      iyy="0.001" iyz="0.0"
+      izz="0.001"/>
     </inertial>
   </link>
   <link name="rear_right_wheel">
     <collision name="collision">
-      <origin xyz="0 -0.06 0" rpy="0 0 -1.5707"/>
-      <geometry>
-        <mesh filename="package://rosbot_description/meshes/wheel.dae" scale="0.001 0.001 0.001" />
-      </geometry>
+      <origin xyz="0 0 0" rpy="0 0 -1.5707"/>
+      <geometry>
+        <mesh filename="package://rosbot_description/meshes/wheel.dae" scale="0.001 0.001 0.001" />
+      </geometry>
+      <surface>
+        <friction>
+          <ode>
+            <mu>10</mu>
+            <mu2>10</mu2>
+          </ode>
+        </friction>
+      </surface>
     </collision>
     <visual name="rear_right_wheel_visual">
-      <origin xyz="0 -0.06 0" rpy="0 0 -1.5707"/>
+      <origin xyz="0 0 0" rpy="0 0 -1.5707"/>
       <geometry>
         <mesh filename="package://rosbot_description/meshes/wheel.dae" scale="0.001 0.001 0.001" />
@@ -135,41 +167,41 @@
     <inertial>
       <origin xyz="0 0 0" rpy="0 1.5707 1.5707"/>
-      <mass value="40"/>
-      <inertia
-      ixx=".1" ixy="0.0" ixz="0.0"
-      iyy=".1" iyz="0.0"
-      izz=".1"/>
+      <mass value="0.5"/>
+      <inertia
+      ixx="0.001" ixy="0.0" ixz="0.0"
+      iyy="0.001" iyz="0.0"
+      izz="0.001"/>
     </inertial>
   </link>
   <joint type="continuous" name="front_left_wheel_hinge">
-    <origin xyz="0.05 0.05 0" rpy="0 0 0"/>
+    <origin xyz="0.05 0.11 0" rpy="0 0 0"/>
     <child link="front_left_wheel"/>
     <parent link="base_link"/>
     <axis xyz="0 1 0" rpy="0 0 0"/>
-    <limit effort="10000" velocity="1000"/>
+    <limit effort="1" velocity="10"/>
     <joint_properties damping="5.0" friction="1.0"/>
   </joint>
   <joint type="continuous" name="front_right_wheel_hinge">
-    <origin xyz="0.05 -0.05 0" rpy="0 0 0"/>
+    <origin xyz="0.05 -0.11 0" rpy="0 0 0"/>
     <child link="front_right_wheel"/>
     <parent link="base_link"/>
     <axis xyz="0 1 0" rpy="0 0 0"/>
-    <limit effort="10000" velocity="1000"/>
+    <limit effort="1" velocity="10"/>
     <joint_properties damping="5.0" friction="1.0"/>
   </joint>
   <joint type="continuous" name="rear_left_wheel_hinge">
-    <origin xyz="-0.055 0.05 0" rpy="0 0 0"/>
+    <origin xyz="-0.055 0.11 0" rpy="0 0 0"/>
     <child link="rear_left_wheel"/>
     <parent link="base_link"/>
     <axis xyz="0 1 0" rpy="0 0 0"/>
-    <limit effort="10000" velocity="1000"/>
+    <limit effort="1" velocity="10"/>
     <joint_properties damping="5.0" friction="1.0"/>
   </joint>
   <joint type="continuous" name="rear_right_wheel_hinge">
-    <origin xyz="-0.055 -0.05 0" rpy="0 0 0"/>
+    <origin xyz="-0.055 -0.11 0" rpy="0 0 0"/>
     <child link="rear_right_wheel"/>
     <parent link="base_link"/>
     <axis xyz="0 1 0" rpy="0 0 0"/>
-    <limit effort="10000" velocity="1000"/>
+    <limit effort="1" velocity="10"/>
     <joint_properties damping="5.0" friction="1.0"/>
   </joint>
@@ -179,7 +211,7 @@
     <origin xyz="-0.03 0 0.18" rpy="0 0 0"/>
     <parent link="base_link"/>
-    <child link="astra"/>
-  </joint>
-  <link name="astra">
+    <child link="camera_link"/>
+  </joint>
+  <link name="camera_link">
     <collision>
       <origin xyz="0.02 0 0" rpy="0 0 0"/>
@@ -197,21 +229,21 @@
       <mass value="1e-5" />
       <origin xyz="0 0 0" rpy="0 0 0"/>
-      <inertia ixx="1e-6" ixy="0" ixz="0" iyy="1e-6" iyz="0" izz="1e-6" />
-    </inertial>
-  </link>
-<joint name="camera_optical_joint" type="fixed">
-  <origin xyz="0 0 0" rpy="${-pi/2} 0 ${-pi/2}"/>
-  <parent link="astra"/>
-  <child link="astra_optical"/>
-</joint>
-<link name="astra_optical">
-</link>
-<joint name="camera_depth_joint" type="fixed">
-  <origin xyz="0 0 0" rpy="0 0 0"/>
-  <parent link="astra"/>
-  <child link="camera_depth_frame"/>
-</joint>
-<link name="camera_depth_frame">
-</link>
+      <inertia ixx="0" ixy="0" ixz="0" iyy="0" iyz="0" izz="0" />
+    </inertial>
+  </link>
+  <joint name="camera_optical_joint" type="fixed">
+    <origin xyz="0 0 0" rpy="${-pi/2} 0 ${-pi/2}"/>
+    <parent link="camera_link"/>
+    <child link="camera_rgb_frame"/>
+  </joint>
+  <link name="camera_rgb_frame">
+  </link>
+  <joint name="camera_depth_joint" type="fixed">
+    <origin xyz="0 0 0" rpy="0 0 0"/>
+    <parent link="camera_link"/>
+    <child link="camera_depth_frame"/>
+  </joint>
+  <link name="camera_depth_frame">
+  </link>
   <joint name="rplidar_joint" type="fixed">
     <axis xyz="0 1 0" />
@@ -237,5 +269,5 @@
       <mass value="1e-5" />
       <origin xyz="0 0 0" rpy="0 0 0"/>
-      <inertia ixx="1e-6" ixy="0" ixz="0" iyy="1e-6" iyz="0" izz="1e-6" />
+      <inertia ixx="0" ixy="0" ixz="0" iyy="0" iyz="0" izz="0" />
     </inertial>
   </link>

Commit message: Updated frame names

File: src/rosbot_description/urdf/rosbot.xacro (robot description, xacro)
@@ -250,8 +250,8 @@
     <origin xyz="0.02 0 0.086" rpy="0 0 3.14"/>
     <parent link="base_link"/>
-    <child link="rplidar"/>
+    <child link="laser"/>
   </joint>
   <!-- rplidar Laser -->
-  <link name="rplidar">
+  <link name="laser">
     <collision>
       <origin xyz="0 0 0" rpy="0 0 0"/>

Commit message: fix tf for wheels

File: src/rosbot_description/urdf/rosbot.xacro (robot description, xacro)
@@ -248,5 +248,5 @@
   <joint name="rplidar_joint" type="fixed">
     <axis xyz="0 1 0" />
-    <origin xyz="0.02 0 0.086" rpy="0 0 3.14"/>
+    <origin xyz="0.02 0 0" rpy="0 0 3.14"/>
     <parent link="base_link"/>
     <child link="laser"/>
@@ -255,11 +255,11 @@
   <link name="laser">
     <collision>
-      <origin xyz="0 0 0" rpy="0 0 0"/>
-      <geometry>
-        <box size="0.001 0.001 0.001"/>
+      <origin xyz="0 0 0.058" rpy="1.5707 0 4.71"/>
+      <geometry>
+        <mesh filename="package://rosbot_description/meshes/rplidar.dae" scale="0.001 0.001 0.001" />
       </geometry>
     </collision>
     <visual>
-      <origin xyz="0 0 -0.03" rpy="1.5707 0 4.71"/>
+      <origin xyz="0 0 0.058" rpy="1.5707 0 4.71"/>
       <geometry>
         <mesh filename="package://rosbot_description/meshes/rplidar.dae" scale="0.001 0.001 0.001" />
@@ -268,5 +268,5 @@
     <inertial>
       <mass value="1e-5" />
-      <origin xyz="0 0 0" rpy="0 0 0"/>
+      <origin xyz="0 0 0.058" rpy="1.5707 0 4.71"/>
       <inertia ixx="0" ixy="0" ixz="0" iyy="0" iyz="0" izz="0" />
     </inertial>

Commit message: Fixed wheels tf publications

File: src/rosbot_description/urdf/rosbot.xacro (robot description, xacro)
@@ -1,4 +1,5 @@
 <?xml version='1.0'?>
-<robot name="rosbot" xmlns:xacro="http://www.ros.org/wiki/xacro">
+<robot name="rosbot"
+  xmlns:xacro="http://www.ros.org/wiki/xacro">
   <xacro:property name="cameraSize" value="0.05"/>
   <xacro:property name="cameraMass" value="0.1"/>
@@ -182,4 +183,13 @@
     <joint_properties damping="5.0" friction="1.0"/>
   </joint>
+  <transmission name="front_left_wheel_trans" type="SimpleTransmission">
+    <type>transmission_interface/SimpleTransmission</type>
+    <actuator name="front_left_wheel_motor">
+      <mechanicalReduction>1</mechanicalReduction>
+    </actuator>
+    <joint name="front_left_wheel_hinge">
+      <hardwareInterface>hardware_interface/EffortJointInterface</hardwareInterface>
+    </joint>
+  </transmission>
   <joint type="continuous" name="front_right_wheel_hinge">
     <origin xyz="0.05 -0.11 0" rpy="0 0 0"/>
@@ -190,4 +200,13 @@
     <joint_properties damping="5.0" friction="1.0"/>
   </joint>
+  <transmission name="front_right_wheel_trans" type="SimpleTransmission">
+    <type>transmission_interface/SimpleTransmission</type>
+    <actuator name="front_right_wheel_motor">
+      <mechanicalReduction>1</mechanicalReduction>
+    </actuator>
+    <joint name="front_right_wheel_hinge">
+      <hardwareInterface>hardware_interface/EffortJointInterface</hardwareInterface>
+    </joint>
+  </transmission>
   <joint type="continuous" name="rear_left_wheel_hinge">
     <origin xyz="-0.055 0.11 0" rpy="0 0 0"/>
@@ -198,4 +217,13 @@
     <joint_properties damping="5.0" friction="1.0"/>
   </joint>
+  <transmission name="rear_left_wheel_trans" type="SimpleTransmission">
+    <type>transmission_interface/SimpleTransmission</type>
+    <actuator name="rear_left_wheel_motor">
+      <mechanicalReduction>1</mechanicalReduction>
+    </actuator>
+    <joint name="rear_left_wheel_hinge">
+      <hardwareInterface>hardware_interface/EffortJointInterface</hardwareInterface>
+    </joint>
+  </transmission>
   <joint type="continuous" name="rear_right_wheel_hinge">
     <origin xyz="-0.055 -0.11 0" rpy="0 0 0"/>
@@ -206,4 +234,13 @@
     <joint_properties damping="5.0" friction="1.0"/>
   </joint>
+  <transmission name="rear_right_wheel_trans" type="SimpleTransmission">
+    <type>transmission_interface/SimpleTransmission</type>
+    <actuator name="rear_right_wheel_motor">
+      <mechanicalReduction>1</mechanicalReduction>
+    </actuator>
+    <joint name="rear_right_wheel_hinge">
+      <hardwareInterface>hardware_interface/EffortJointInterface</hardwareInterface>
+    </joint>
+  </transmission>
   <!-- Orbbec Astra RGBD Camera -->
   <joint name="astra_joint" type="fixed">

Commit message: Updated camera tf

File: src/rosbot_description/urdf/rosbot.xacro (robot description, xacro)
@@ -277,5 +277,5 @@
   </link>
   <joint name="camera_depth_joint" type="fixed">
-    <origin xyz="0 0 0" rpy="0 0 0"/>
+    <origin xyz="0 0 0" rpy="${-pi/2} 0 ${-pi/2}"/>
     <parent link="camera_link"/>
     <child link="camera_depth_frame"/>

Commit message: Add namespaces

File: src/rosbot_description/urdf/rosbot.xacro (robot description, xacro)
@@ -2,6 +2,8 @@
 <robot name="rosbot"
   xmlns:xacro="http://www.ros.org/wiki/xacro">
+  <xacro:arg name="robot_namespace" default=""/>
   <xacro:property name="cameraSize" value="0.05"/>
   <xacro:property name="cameraMass" value="0.1"/>
+  <xacro:property name="namespace" value="$(arg robot_namespace)" />
   <xacro:include filename="$(find rosbot_description)/urdf/rosbot.gazebo" />
   <xacro:include filename="$(find rosbot_description)/urdf/materials.xacro" />

Commit message: fixes in ROSbot kinematics

File: src/rosbot_description/urdf/rosbot.xacro (robot description, xacro)
@@ -61,5 +61,5 @@
       <origin xyz="0 0 0" rpy="0 0 1.5707"/>
       <geometry>
-        <mesh filename="package://rosbot_description/meshes/wheel.dae" scale="0.001 0.001 0.001" />
+        <mesh filename="package://rosbot_description/meshes/wheel-v2.stl" scale="0.001 0.001 0.001" />
       </geometry>
       <surface>
@@ -91,5 +91,5 @@
       <origin xyz="0 0 0" rpy="0 0 -1.5707"/>
       <geometry>
-        <mesh filename="package://rosbot_description/meshes/wheel.dae" scale="0.001 0.001 0.001" />
+        <mesh filename="package://rosbot_description/meshes/wheel-v2.stl" scale="0.001 0.001 0.001" />
       </geometry>
       <surface>
@@ -121,5 +121,5 @@
       <origin xyz="0 0 0" rpy="0 0 1.5707"/>
       <geometry>
-        <mesh filename="package://rosbot_description/meshes/wheel.dae" scale="0.001 0.001 0.001" />
+        <mesh filename="package://rosbot_description/meshes/wheel-v2.stl" scale="0.001 0.001 0.001" />
       </geometry>
       <surface>
@@ -151,5 +151,5 @@
       <origin xyz="0 0 0" rpy="0 0 -1.5707"/>
       <geometry>
-        <mesh filename="package://rosbot_description/meshes/wheel.dae" scale="0.001 0.001 0.001" />
+        <mesh filename="package://rosbot_description/meshes/wheel-v2.stl" scale="0.001 0.001 0.001" />
       </geometry>
       <surface>
@@ -287,5 +287,5 @@
   <joint name="rplidar_joint" type="fixed">
     <axis xyz="0 1 0" />
-    <origin xyz="0.02 0 0" rpy="0 0 3.14"/>
+    <origin xyz="0.02 0 0.058" rpy="0 0 3.14"/>
     <parent link="base_link"/>
     <child link="laser"/>
@@ -294,5 +294,5 @@
   <link name="laser">
     <collision>
-      <origin xyz="0 0 0.058" rpy="1.5707 0 4.71"/>
+      <origin xyz="0 0 0" rpy="1.5707 0 4.71"/>
       <geometry>
         <mesh filename="package://rosbot_description/meshes/rplidar.dae" scale="0.001 0.001 0.001" />
@@ -300,5 +300,5 @@
     </collision>
     <visual>
-      <origin xyz="0 0 0.058" rpy="1.5707 0 4.71"/>
+      <origin xyz="0 0 0" rpy="1.5707 0 4.71"/>
       <geometry>
         <mesh filename="package://rosbot_description/meshes/rplidar.dae" scale="0.001 0.001 0.001" />
@@ -307,5 +307,5 @@
     <inertial>
       <mass value="1e-5" />
-      <origin xyz="0 0 0.058" rpy="1.5707 0 4.71"/>
+      <origin xyz="0 0 0" rpy="1.5707 0 4.71"/>
       <inertia ixx="0" ixy="0" ixz="0" iyy="0" iyz="0" izz="0" />
     </inertial>

Commit message: fix base_link waring

File: src/rosbot_description/urdf/rosbot.xacro (robot description, xacro)
@@ -9,4 +9,9 @@
   <xacro:include filename="$(find rosbot_description)/urdf/materials.xacro" />
   <xacro:include filename="$(find rosbot_description)/urdf/macros.xacro" />
+  <link name="dummy"></link>
+  <joint name="dummy_joint" type="fixed">
+    <parent link="dummy"/>
+    <child link="base_link"/>
+  </joint>
   <link name='base_link'>
     <pose>0 0 0.1 0 0 0</pose>

Commit message: URDF fix for swarm, update Rviz

File: src/rosbot_description/urdf/rosbot.xacro (robot description, xacro)
@@ -5,13 +5,5 @@
   <xacro:property name="cameraSize" value="0.05"/>
   <xacro:property name="cameraMass" value="0.1"/>
-  <xacro:property name="namespace" value="$(arg robot_namespace)" />
   <xacro:include filename="$(find rosbot_description)/urdf/rosbot.gazebo" />
-  <xacro:include filename="$(find rosbot_description)/urdf/materials.xacro" />
-  <xacro:include filename="$(find rosbot_description)/urdf/macros.xacro" />
-  <link name="dummy"></link>
-  <joint name="dummy_joint" type="fixed">
-    <parent link="dummy"/>
-    <child link="base_link"/>
-  </joint>
   <link name='base_link'>
     <pose>0 0 0.1 0 0 0</pose>

Commit message: Bring back dummy link

File: src/rosbot_description/urdf/rosbot.xacro (robot description, xacro)
@@ -6,4 +6,9 @@
   <xacro:property name="cameraMass" value="0.1"/>
   <xacro:include filename="$(find rosbot_description)/urdf/rosbot.gazebo" />
+  <link name="dummy"></link>
+  <joint name="dummy_joint" type="fixed">
+    <parent link="dummy"/>
+    <child link="base_link"/>
+  </joint>
   <link name='base_link'>
     <pose>0 0 0.1 0 0 0</pose>
