Commit message: Rviz colors, base_link as dummy, lighter collision

File: src/rosbot_description/urdf/rosbot.xacro (robot description, xacro)
@@ -5,11 +5,12 @@
   <xacro:property name="cameraSize" value="0.05"/>
   <xacro:property name="cameraMass" value="0.1"/>
+  <xacro:include filename="$(find rosbot_description)/urdf/materials.xacro" />
   <xacro:include filename="$(find rosbot_description)/urdf/rosbot.gazebo" />
-  <link name="dummy"></link>
-  <joint name="dummy_joint" type="fixed">
-    <parent link="dummy"/>
-    <child link="base_link"/>
-  </joint>
-  <link name='base_link'>
+  <link name="base_link"></link>
+  <joint name="base_link_joint" type="fixed">
+    <parent link="base_link"/>
+    <child link="body_link"/>
+  </joint>
+  <link name='body_link'>
     <pose>0 0 0.1 0 0 0</pose>
     <inertial>
@@ -22,5 +23,5 @@
       />
     </inertial>
-    <collision name='collision'>
+    <collision>
       <origin xyz="0 0 0.02" rpy="0 0 0"/>
       <geometry>
@@ -28,9 +29,10 @@
       </geometry>
     </collision>
-    <visual name='base_link_visual'>
+    <visual>
       <origin xyz="0 0 -0.02" rpy=" 1.5707 0 1.5707"/>
       <geometry>
-        <mesh filename="package://rosbot_description/meshes/box.dae" scale="0.001 0.001 0.001" />
-      </geometry>
+        <mesh filename="package://rosbot_description/meshes/box.stl" scale="0.001 0.001 0.001" />
+      </geometry>
+      <material name="White"/>
     </visual>
   </link>
@@ -38,5 +40,5 @@
     <axis xyz="0 1 0" />
     <origin xyz="0 0 0" rpy="0 0 0"/>
-    <parent link="base_link"/>
+    <parent link="body_link"/>
     <child link="top"/>
   </joint>
@@ -52,16 +54,17 @@
       />
     </inertial>
-    <visual name='top'>
+    <visual>
       <origin xyz="0 0 0.055" rpy=" 1.5707 0 1.5707"/>
       <geometry>
-        <mesh filename="package://rosbot_description/meshes/upper.dae" scale="0.001 0.001 0.001" />
-      </geometry>
+        <mesh filename="package://rosbot_description/meshes/upper.stl" scale="0.001 0.001 0.001" />
+      </geometry>
+      <material name="Red"/>
     </visual>
   </link>
   <link name="front_left_wheel">
-    <collision name="collision">
-      <origin xyz="0 0 0" rpy="0 0 1.5707"/>
-      <geometry>
-        <mesh filename="package://rosbot_description/meshes/wheel-v2.stl" scale="0.001 0.001 0.001" />
+    <collision>
+      <origin xyz="0 -0.014 0" rpy="${pi/2} 0 0"/>
+      <geometry>
+        <cylinder length="0.036" radius="0.04"/>
       </geometry>
       <surface>
@@ -74,9 +77,10 @@
       </surface>
     </collision>
-    <visual name="front_left_wheel_visual">
+    <visual>
       <origin xyz="0 0 0" rpy="0 0 1.5707"/>
       <geometry>
-        <mesh filename="package://rosbot_description/meshes/wheel.dae" scale="0.001 0.001 0.001" />
-      </geometry>
+        <mesh filename="package://rosbot_description/meshes/wheel.stl" scale="0.001 0.001 0.001" />
+      </geometry>
+      <material name="Black"/>
     </visual>
     <inertial>
@@ -90,8 +94,8 @@
   </link>
   <link name="front_right_wheel">
-    <collision name="collision">
-      <origin xyz="0 0 0" rpy="0 0 -1.5707"/>
-      <geometry>
-        <mesh filename="package://rosbot_description/meshes/wheel-v2.stl" scale="0.001 0.001 0.001" />
+    <collision>
+      <origin xyz="0 0.014 0" rpy="${pi/2} 0 0"/>
+      <geometry>
+        <cylinder length="0.036" radius="0.04"/>
       </geometry>
       <surface>
@@ -104,9 +108,10 @@
       </surface>
     </collision>
-    <visual name="front_right_wheel_visual">
+    <visual>
       <origin xyz="0 0 0" rpy="0 0 -1.5707"/>
       <geometry>
-        <mesh filename="package://rosbot_description/meshes/wheel.dae" scale="0.001 0.001 0.001" />
-      </geometry>
+        <mesh filename="package://rosbot_description/meshes/wheel.stl" scale="0.001 0.001 0.001" />
+      </geometry>
+      <material name="Black"/>
     </visual>
     <inertial>
@@ -120,8 +125,8 @@
   </link>
   <link name="rear_left_wheel">
-    <collision name="collision">
-      <origin xyz="0 0 0" rpy="0 0 1.5707"/>
-      <geometry>
-        <mesh filename="package://rosbot_description/meshes/wheel-v2.stl" scale="0.001 0.001 0.001" />
+    <collision>
+      <origin xyz="0 -0.014 0" rpy="${pi/2} 0 0"/>
+      <geometry>
+        <cylinder length="0.036" radius="0.04"/>
       </geometry>
       <surface>
@@ -134,9 +139,10 @@
       </surface>
     </collision>
-    <visual name="rear_left_wheel_visual">
+    <visual>
       <origin xyz="0 0 0" rpy="0 0 1.5707"/>
       <geometry>
-        <mesh filename="package://rosbot_description/meshes/wheel.dae" scale="0.001 0.001 0.001" />
-      </geometry>
+        <mesh filename="package://rosbot_description/meshes/wheel.stl" scale="0.001 0.001 0.001" />
+      </geometry>
+      <material name="Black"/>
     </visual>
     <inertial>
@@ -150,8 +156,8 @@
   </link>
   <link name="rear_right_wheel">
-    <collision name="collision">
-      <origin xyz="0 0 0" rpy="0 0 -1.5707"/>
-      <geometry>
-        <mesh filename="package://rosbot_description/meshes/wheel-v2.stl" scale="0.001 0.001 0.001" />
+    <collision>
+      <origin xyz="0 0.014 0" rpy="${pi/2} 0 0"/>
+      <geometry>
+        <cylinder length="0.036" radius="0.04"/>
       </geometry>
       <surface>
@@ -164,9 +170,10 @@
       </surface>
     </collision>
-    <visual name="rear_right_wheel_visual">
+    <visual>
       <origin xyz="0 0 0" rpy="0 0 -1.5707"/>
       <geometry>
-        <mesh filename="package://rosbot_description/meshes/wheel.dae" scale="0.001 0.001 0.001" />
-      </geometry>
+        <mesh filename="package://rosbot_description/meshes/wheel.stl" scale="0.001 0.001 0.001" />
+      </geometry>
+      <material name="Black"/>
     </visual>
     <inertial>
@@ -182,5 +189,5 @@
     <origin xyz="0.05 0.11 0" rpy="0 0 0"/>
     <child link="front_left_wheel"/>
-    <parent link="base_link"/>
+    <parent link="body_link"/>
     <axis xyz="0 1 0" rpy="0 0 0"/>
     <limit effort="1" velocity="10"/>
@@ -199,5 +206,5 @@
     <origin xyz="0.05 -0.11 0" rpy="0 0 0"/>
     <child link="front_right_wheel"/>
-    <parent link="base_link"/>
+    <parent link="body_link"/>
     <axis xyz="0 1 0" rpy="0 0 0"/>
     <limit effort="1" velocity="10"/>
@@ -216,5 +223,5 @@
     <origin xyz="-0.055 0.11 0" rpy="0 0 0"/>
     <child link="rear_left_wheel"/>
-    <parent link="base_link"/>
+    <parent link="body_link"/>
     <axis xyz="0 1 0" rpy="0 0 0"/>
     <limit effort="1" velocity="10"/>
@@ -233,5 +240,5 @@
     <origin xyz="-0.055 -0.11 0" rpy="0 0 0"/>
     <child link="rear_right_wheel"/>
-    <parent link="base_link"/>
+    <parent link="body_link"/>
     <axis xyz="0 1 0" rpy="0 0 0"/>
     <limit effort="1" velocity="10"/>
@@ -251,5 +258,5 @@
     <axis xyz="0 0 0" />
     <origin xyz="-0.03 0 0.18" rpy="0 0 0"/>
-    <parent link="base_link"/>
+    <parent link="body_link"/>
     <child link="camera_link"/>
   </joint>
@@ -264,6 +271,7 @@
       <origin xyz="-0.01 0 -0.03" rpy="1.5707 0 1.5707"/>
       <geometry>
-        <mesh filename="package://rosbot_description/meshes/astra.dae" scale="0.001 0.001 0.001" />
-      </geometry>
+        <mesh filename="package://rosbot_description/meshes/astra.stl" scale="0.001 0.001 0.001" />
+      </geometry>
+      <material name="Black"/>
     </visual>
     <inertial>
@@ -290,5 +298,5 @@
     <axis xyz="0 1 0" />
     <origin xyz="0.02 0 0.058" rpy="0 0 3.14"/>
-    <parent link="base_link"/>
+    <parent link="body_link"/>
     <child link="laser"/>
   </joint>
@@ -298,5 +306,5 @@
       <origin xyz="0 0 0" rpy="1.5707 0 4.71"/>
       <geometry>
-        <mesh filename="package://rosbot_description/meshes/rplidar.dae" scale="0.001 0.001 0.001" />
+        <mesh filename="package://rosbot_description/meshes/rplidar.stl" scale="0.001 0.001 0.001" />
       </geometry>
     </collision>
@@ -304,6 +312,7 @@
       <origin xyz="0 0 0" rpy="1.5707 0 4.71"/>
       <geometry>
-        <mesh filename="package://rosbot_description/meshes/rplidar.dae" scale="0.001 0.001 0.001" />
-      </geometry>
+        <mesh filename="package://rosbot_description/meshes/rplidar.stl" scale="0.001 0.001 0.001" />
+      </geometry>
+      <material name="Black"/>
     </visual>
     <inertial>
@@ -316,5 +325,5 @@
     <axis xyz="0 1 0" />
     <origin xyz="0.1 0.05 0.01" rpy="0 0 0.13 "/>
-    <parent link="base_link"/>
+    <parent link="body_link"/>
     <child link="range_fl"/>
   </joint>
@@ -323,5 +332,5 @@
     <axis xyz="0 1 0" />
     <origin xyz="0.1 -0.05 0.01" rpy="0 0 -0.13 "/>
-    <parent link="base_link"/>
+    <parent link="body_link"/>
     <child link="range_fr"/>
   </joint>
@@ -330,5 +339,5 @@
     <axis xyz="0 1 0" />
     <origin xyz="-0.1 0.05 0.01" rpy="0 0 3.01 "/>
-    <parent link="base_link"/>
+    <parent link="body_link"/>
     <child link="range_rl"/>
   </joint>
@@ -337,5 +346,5 @@
     <axis xyz="0 1 0" />
     <origin xyz="-0.1 -0.05 0.01" rpy="0 0 3.27 "/>
-    <parent link="base_link"/>
+    <parent link="body_link"/>
     <child link="range_rr"/>
   </joint>

Commit message: Add missing origin in link joint

File: src/rosbot_description/urdf/rosbot.xacro (robot description, xacro)
@@ -9,4 +9,5 @@
   <link name="base_link"></link>
   <joint name="base_link_joint" type="fixed">
+    <origin xyz="0 0 0" rpy="0 0 0"/>
     <parent link="base_link"/>
     <child link="body_link"/>

Commit message: add robot_state_publisher in docker launch

File: src/rosbot_description/urdf/rosbot.xacro (robot description, xacro)
@@ -18,9 +18,5 @@
       <mass value="5"/>
       <origin xyz="0 0 0.04" rpy=" 0 0 0"/>
-      <inertia
-      ixx="0.01" ixy="0.01" ixz="0"
-      iyy="0.01" iyz="0.01"
-      izz="0.01"
-      />
+      <inertia ixx="0.01" ixy="0.01" ixz="0" iyy="0.01" iyz="0.01" izz="0.01" />
     </inertial>
     <collision>
@@ -49,9 +45,5 @@
       <mass value="0.01"/>
       <origin xyz="0 0 0.055" rpy=" 0 0 0"/>
-      <inertia
-      ixx="0.0" ixy="0" ixz="0"
-      iyy="0.0" iyz="0"
-      izz="0.0"
-      />
+      <inertia ixx="0.0" ixy="0" ixz="0" iyy="0.0" iyz="0" izz="0.0" />
     </inertial>
     <visual>
@@ -88,8 +80,5 @@
       <origin xyz="0 0 0" rpy="0 1.5707 1.5707"/>
       <mass value="0.5"/>
-      <inertia
-      ixx="0.001" ixy="0.0" ixz="0.0"
-      iyy="0.001" iyz="0.0"
-      izz="0.001"/>
+      <inertia ixx="0.001" ixy="0.0" ixz="0.0" iyy="0.001" iyz="0.0" izz="0.001"/>
     </inertial>
   </link>
@@ -119,8 +108,5 @@
       <origin xyz="0 0 0" rpy="0 1.5707 1.5707"/>
       <mass value="0.5"/>
-      <inertia
-      ixx="0.001" ixy="0.0" ixz="0.0"
-      iyy="0.001" iyz="0.0"
-      izz="0.001"/>
+      <inertia ixx="0.001" ixy="0.0" ixz="0.0" iyy="0.001" iyz="0.0" izz="0.001"/>
     </inertial>
   </link>
@@ -150,8 +136,5 @@
       <origin xyz="0 0 0" rpy="0 1.5707 1.5707"/>
       <mass value="0.5"/>
-      <inertia
-      ixx="0.001" ixy="0.0" ixz="0.0"
-      iyy="0.001" iyz="0.0"
-      izz="0.001"/>
+      <inertia ixx="0.001" ixy="0.0" ixz="0.0" iyy="0.001" iyz="0.0" izz="0.001"/>
     </inertial>
   </link>
@@ -181,8 +164,5 @@
       <origin xyz="0 0 0" rpy="0 1.5707 1.5707"/>
       <mass value="0.5"/>
-      <inertia
-      ixx="0.001" ixy="0.0" ixz="0.0"
-      iyy="0.001" iyz="0.0"
-      izz="0.001"/>
+      <inertia ixx="0.001" ixy="0.0" ixz="0.0" iyy="0.001" iyz="0.0" izz="0.001"/>
     </inertial>
   </link>
