Commit message: added range sensors to robot_description

File: src/rosbot_description/models/rosbot_base/body.urdf.xacro (robot description, xacro)
@@ -7,8 +7,8 @@
       <visual>
         <geometry>
-          <mesh filename="file://$(find rosbot_description)/models/rosbot_base/meshes/body.stl" scale="0.001 0.001 0.001"/>
+          <mesh filename="file://$(find rosbot_description)/models/rosbot_base/meshes/body.stl" scale="0.001 0.001 0.001" />
         </geometry>
-        <origin xyz="0.0 0.0 -0.02" rpy="${pi/2} 0.0 ${pi/2}"/>
-        <material name="White"/>
+        <origin xyz="0.0 0.0 -0.02" rpy="${pi/2} 0.0 ${pi/2}" />
+        <material name="White" />
       </visual>
       <collision>
@@ -16,11 +16,9 @@
           <box size="0.197 0.150 0.080" />
         </geometry>
-        <origin xyz="0.0 0.0 ${0.040-0.02}" rpy="0.0 0.0 0.0"/>
+        <origin xyz="0.0 0.0 ${0.040-0.02}" rpy="0.0 0.0 0.0" />
       </collision>
       <inertial>
-          <mass value="2.0" />
-          <inertia ixx="0.001" ixy="0.000"  ixz="0.000"
-                               iyy="0.001"  iyz="0.000"
-                                            izz="0.001" />
+        <mass value="2.0" />
+        <inertia ixx="0.001" ixy="0.000" ixz="0.000" iyy="0.001" iyz="0.000" izz="0.001" />
       </inertial>
     </link>
@@ -28,14 +26,12 @@
       <visual>
         <geometry>
-          <mesh filename="file://$(find rosbot_description)/models/rosbot_base/meshes/cover.stl" scale="0.001 0.001 0.001"/>
+          <mesh filename="file://$(find rosbot_description)/models/rosbot_base/meshes/cover.stl" scale="0.001 0.001 0.001" />
         </geometry>
-        <origin xyz="0.0 0.0 -0.002" rpy="${pi/2} 0.0 ${pi/2}"/>
-        <material name="Red"/>
+        <origin xyz="0.0 0.0 -0.002" rpy="${pi/2} 0.0 ${pi/2}" />
+        <material name="Red" />
       </visual>
       <inertial>
         <mass value="0.000001" />
-        <inertia ixx="1.0" ixy="0.0" ixz="0.0"
-                           iyy="1.0" iyz="0.0"
-                                     izz="0.0" />
+        <inertia ixx="1.0" ixy="0.0" ixz="0.0" iyy="1.0" iyz="0.0" izz="0.0" />
       </inertial>
     </link>
@@ -78,4 +74,32 @@
       <material>Gazebo/Red</material>
     </gazebo>
+    <joint name="range_left_front_joint" type="fixed">
+      <axis xyz="0 1 0" />
+      <origin xyz="0.1 0.05 0.01" rpy="0 0 0.13 " />
+      <parent link="body_link" />
+      <child link="range_left_front" />
+    </joint>
+    <link name="range_left_front"></link>
+    <joint name="range_right_front_joint" type="fixed">
+      <axis xyz="0 1 0" />
+      <origin xyz="0.1 -0.05 0.01" rpy="0 0 -0.13 " />
+      <parent link="body_link" />
+      <child link="range_right_front" />
+    </joint>
+    <link name="range_right_front"></link>
+    <joint name="range_left_rear_joint" type="fixed">
+      <axis xyz="0 1 0" />
+      <origin xyz="-0.1 0.05 0.01" rpy="0 0 3.01 " />
+      <parent link="body_link" />
+      <child link="range_left_rear" />
+    </joint>
+    <link name="range_left_rear"></link>
+    <joint name="range_right_rear_joint" type="fixed">
+      <axis xyz="0 1 0" />
+      <origin xyz="-0.1 -0.05 0.01" rpy="0 0 3.27 " />
+      <parent link="body_link" />
+      <child link="range_right_rear" />
+    </joint>
+    <link name="range_right_rear"></link>
   </xacro:macro>
 </robot>
