Commit message: Refactor rosbot description

File: rosbot_description/urdf/components/orbbec_astra.gazebo.xacro (robot description, xacro)
@@ -2,11 +2,18 @@
 <robot xmlns:xacro="http://www.ros.org/wiki/xacro">
   <xacro:macro name="orbbec_astra" params="xyz rpy parent_link:=base_link">
+    <joint name="body_to_orbbec_astra_joint" type="fixed">
+      <origin xyz="${xyz}" rpy="${rpy}" />
+      <parent link="${parent_link}" />
+      <child link="orbbec_astra_link" />
+    </joint>
     <link name="orbbec_astra_link">
       <visual>
         <geometry>
-            <mesh filename="file://$(find rosbot_description)/models/rosbot_base/meshes/components/astra.stl" scale="0.001 0.001 0.001" />
+          <mesh filename="file://$(find rosbot_description)/meshes/components/astra.stl" scale="0.001 0.001 0.001" />
         </geometry>
-        <origin xyz="-0.01 0 0.025" rpy="${pi/2} 0 ${pi/2}"/>
-        <material name="Black" />
+        <origin xyz="-0.01 0 0.025" rpy="${pi/2} 0 ${pi/2}" />
+        <material name="Black">
+          <color rgba="0.0 0.0 0.0 1.0" />
+        </material>
       </visual>
       <collision>
@@ -14,32 +21,27 @@
           <box size="0.165 0.04 0.05" />
         </geometry>
-        <origin xyz="-0.01 0 0.025" rpy="0 0 ${pi/2}"/>
+        <origin xyz="-0.01 0 0.025" rpy="0 0 ${pi/2}" />
       </collision>
       <inertial>
-          <mass value="0.105" />
-          <inertia ixx="0.001" ixy="0" ixz="0" iyy="0.001" iyz="0" izz="0.001" />
+        <mass value="0.105" />
+        <inertia ixx="0.001" ixy="0" ixz="0" iyy="0.001" iyz="0" izz="0.001" />
       </inertial>
     </link>
-    <link name="orbbec_astra_depth_link"></link>
-    <link name="orbbec_astra_depth_refference_link"></link>
-    <joint name="body_link_to_orbbec_astra_link_joint" type="fixed">
-      <origin xyz="${xyz}" rpy="${rpy}" />
-      <parent link="${parent_link}" />
-      <child link="orbbec_astra_link" />
-    </joint>
-    <joint name="orbbec_astra_depth_link_joint" type="fixed">
+    <joint name="orbbec_astra_depth_joint" type="fixed">
       <origin xyz="0.01 0 0.035" rpy="0.0 ${pi/2} 0.0" />
       <parent link="orbbec_astra_link" />
       <child link="orbbec_astra_depth_link" />
     </joint>
-    <joint name="orbbec_astra_depth_link_refference_joint" type="fixed">
-      <origin xyz="0.0 0.0 0.0" rpy="${pi/2} ${-pi/2} 0.0" />
-      <parent link="orbbec_astra_depth_link" />
-      <child link="orbbec_astra_depth_refference_link" />
-    </joint>
+    <link name="orbbec_astra_depth_link"></link>
     <gazebo reference="orbbec_astra_link">
       <material>Gazebo/DarkGrey</material>
     </gazebo>
-    <gazebo reference="orbbec_astra_depth_refference_link">
+    <joint name="orbbec_astra_depth_reference_joint" type="fixed">
+      <origin xyz="0.0 0.0 0.0" rpy="${pi/2} ${-pi/2} 0.0" />
+      <parent link="orbbec_astra_depth_link" />
+      <child link="orbbec_astra_depth_reference_link" />
+    </joint>
+    <link name="orbbec_astra_depth_reference_link"></link>
+    <gazebo reference="orbbec_astra_depth_reference_link">
       <sensor type="depth" name="orbbec_astra_camera">
         <always_on>1</always_on>

File: rosbot_description/urdf/wheel.urdf.xacro (robot description, xacro)
@@ -2,9 +2,9 @@
 <robot xmlns:xacro="http://www.ros.org/wiki/xacro">
   <!-- wheel defining macro -->
-  <xacro:macro name="wheel" params="wheel_type wheel_diameter prefix">
+  <xacro:macro name="wheel" params="wheel_type wheel_radius prefix">
     <xacro:property name="wheel_separation_x" value="0.106" />
     <xacro:property name="wheel_separation_y" value="0.228" />
     <xacro:property name="wheel_thickness" value="0.036" />
-    <xacro:if value="${prefix == 'front_left'}">
+    <xacro:if value="${prefix == 'fl'}">
       <xacro:property name="x" value="${wheel_separation_x/2}" />
       <xacro:property name="y" value="${wheel_separation_y/2 - wheel_thickness/2}" />
@@ -12,5 +12,5 @@
       <xacro:property name="rot" value="${pi/2}" />
     </xacro:if>
-    <xacro:if value="${prefix == 'front_right'}">
+    <xacro:if value="${prefix == 'fr'}">
       <xacro:property name="x" value="${wheel_separation_x/2}" />
       <xacro:property name="y" value="-${wheel_separation_y/2 - wheel_thickness/2}" />
@@ -18,5 +18,5 @@
       <xacro:property name="rot" value="${-pi/2}" />
     </xacro:if>
-    <xacro:if value="${prefix == 'rear_left'}">
+    <xacro:if value="${prefix == 'rl'}">
       <xacro:property name="x" value="-${wheel_separation_x/2}" />
       <xacro:property name="y" value="${wheel_separation_y/2 - wheel_thickness/2}" />
@@ -24,5 +24,5 @@
       <xacro:property name="rot" value="${pi/2}" />
     </xacro:if>
-    <xacro:if value="${prefix == 'rear_right'}">
+    <xacro:if value="${prefix == 'rr'}">
       <xacro:property name="x" value="-${wheel_separation_x/2}" />
       <xacro:property name="y" value="-${wheel_separation_y/2 - wheel_thickness/2}" />
@@ -30,25 +30,4 @@
       <xacro:property name="rot" value="${-pi/2}" />
     </xacro:if>
-    <link name="${prefix}_wheel_link">
-       <visual>
-        <geometry>
-          <mesh filename="file://$(find rosbot_description)/models/rosbot_base/meshes/wheel.stl" scale="0.001 0.001 0.001" />
-        </geometry>
-        <origin xyz="0.0 ${y_correction} 0.0" rpy="0.0 0.0 ${rot}"/>
-        <material name="Black"/>
-      </visual>
-      <collision>
-        <geometry>
-          <cylinder radius="${wheel_diameter/2}" length="${wheel_thickness}"/>
-        </geometry>
-        <origin xyz="0.0 0.0 0.0" rpy="${pi/2} 0.0 0.0" />
-      </collision>
-      <inertial>
-          <mass value="0.100" />
-          <inertia ixx="0.001" ixy="0.000"  ixz="0.000"
-                               iyy="0.001"  iyz="0.000"
-                                            izz="0.001" />
-      </inertial>
-    </link>
     <joint name="${prefix}_wheel_joint" type="continuous">
       <parent link="body_link" />
@@ -56,9 +35,30 @@
       <origin xyz="${x} ${y} 0.0" rpy="0.0 0.0 0.0" />
       <axis xyz="0.0 1.0 0.0" />
-      <limit effort="1.5"
-             velocity="5.0" />
-      <dynamics damping="0.001"
-                friction="0.001"/>
+      <limit effort="1.5" velocity="5.0" />
+      <dynamics damping="0.001" friction="0.001" />
     </joint>
+    <link name="${prefix}_wheel_link">
+      <visual>
+        <geometry>
+          <mesh filename="file://$(find rosbot_description)/meshes/wheel.stl" scale="0.001 0.001 0.001" />
+        </geometry>
+        <origin xyz="0.0 ${y_correction} 0.0" rpy="0.0 0.0 ${rot}" />
+        <material name="Black">
+          <color rgba="0.0 0.0 0.0 1.0" />
+        </material>
+      </visual>
+      <collision>
+        <geometry>
+          <cylinder radius="${wheel_radius}" length="${wheel_thickness}" />
+        </geometry>
+        <origin xyz="0.0 0.0 0.0" rpy="${pi/2} 0.0 0.0" />
+      </collision>
+      <inertial>
+        <mass value="0.100" />
+        <inertia ixx="0.001" ixy="0.000" ixz="0.000"
+                             iyy="0.001" iyz="0.000"
+                                         izz="0.001" />
+      </inertial>
+    </link>
     <gazebo reference="${prefix}_wheel_link">
       <material>Gazebo/DarkGrey</material>

Commit message: added configuration for webots simulator

File: rosbot_description/urdf/components/orbbec_astra.gazebo.xacro (robot description, xacro)
@@ -1,5 +1,5 @@
 <?xml version="1.0"?>
 <robot xmlns:xacro="http://www.ros.org/wiki/xacro">
-  <xacro:macro name="orbbec_astra" params="xyz rpy parent_link:=base_link">
+  <xacro:macro name="orbbec_astra" params="xyz rpy parent_link:=base_link simulation_engine:=gazebo-classic">
     <joint name="body_to_orbbec_astra_joint" type="fixed">
       <origin xyz="${xyz}" rpy="${rpy}" />
@@ -43,35 +43,37 @@
     </joint>
     <link name="orbbec_astra_depth_reference_link"></link>
-    <gazebo reference="orbbec_astra_depth_reference_link">
-      <sensor type="depth" name="orbbec_astra_camera">
-        <always_on>1</always_on>
-        <update_rate>10</update_rate>
-        <camera name="camera">
-          <distortion>
-            <k1>0.07</k1>
-            <k2>0.00</k2>
-            <k3>0.00</k3>
-            <p1>0.00</p1>
-            <p2>0.00</p2>
-            <center>0.0 0.0</center>
-          </distortion>
-        </camera>
-        <plugin name="rgbd_camera" filename="libgazebo_ros_camera.so">
-          <ros>
-            <namespace>orbbec_astra_camera</namespace>
-            <argument>--ros-args --remap custom_camera/image_raw:=rgb/image_raw</argument>
-            <argument>--ros-args --remap custom_camera/image_depth:=depth/image_raw</argument>
-            <argument>--ros-args --remap custom_camera/camera_info:=rgb/camera_info</argument>
-            <argument>--ros-args --remap custom_camera/camera_info_depth:=depth/camera_info</argument>
-            <argument>--ros-args --remap custom_camera/points:=depth/points</argument>
-          </ros>
-          <camera_name>camera</camera_name>
-          <frame_name>orbbec_astra_depth_link</frame_name>
-          <hack_baseline>0.07</hack_baseline>
-          <min_depth>0.6</min_depth>
-          <max_depth>8.0</max_depth>
-        </plugin>
-      </sensor>
-    </gazebo>
+    <xacro:unless value="${simulation_engine == 'webots'}">
+      <gazebo reference="orbbec_astra_depth_reference_link">
+        <sensor type="depth" name="orbbec_astra_camera">
+          <always_on>1</always_on>
+          <update_rate>10</update_rate>
+          <camera name="camera">
+            <distortion>
+              <k1>0.07</k1>
+              <k2>0.00</k2>
+              <k3>0.00</k3>
+              <p1>0.00</p1>
+              <p2>0.00</p2>
+              <center>0.0 0.0</center>
+            </distortion>
+          </camera>
+          <plugin name="rgbd_camera" filename="libgazebo_ros_camera.so">
+            <ros>
+              <namespace>orbbec_astra_camera</namespace>
+              <argument>--ros-args --remap custom_camera/image_raw:=rgb/image_raw</argument>
+              <argument>--ros-args --remap custom_camera/image_depth:=depth/image_raw</argument>
+              <argument>--ros-args --remap custom_camera/camera_info:=rgb/camera_info</argument>
+              <argument>--ros-args --remap custom_camera/camera_info_depth:=depth/camera_info</argument>
+              <argument>--ros-args --remap custom_camera/points:=depth/points</argument>
+            </ros>
+            <camera_name>camera</camera_name>
+            <frame_name>orbbec_astra_depth_link</frame_name>
+            <hack_baseline>0.07</hack_baseline>
+            <min_depth>0.6</min_depth>
+            <max_depth>8.0</max_depth>
+          </plugin>
+        </sensor>
+      </gazebo>
+    </xacro:unless>
   </xacro:macro>
 </robot>

File: rosbot_description/urdf/components/rplidar_a2.gazebo.xacro (robot description, xacro)
@@ -55,51 +55,53 @@
     </joint>
     <link name="${tf_prefix_ext}${frame_id}"></link>
-    <gazebo reference="${tf_prefix_ext}${frame_id}">
-      <sensor type="${ray_type}" name="${tf_prefix_ext}rplidar_a2_sensor">
-        <topic>${topic}</topic>
-        <frame_id>${tf_prefix_ext}${frame_id}</frame_id>
-        <ignition_frame_id>${tf_prefix_ext}${frame_id}</ignition_frame_id>
-        <update_rate>10</update_rate>
-        <ray>
-          <scan>
-            <horizontal>
-              <samples>400</samples>
-              <resolution>1</resolution>
-              <min_angle>-${pi}</min_angle>
-              <max_angle>${pi}</max_angle>
-            </horizontal>
-          </scan>
-          <range>
-            <min>0.2</min>
-            <max>16.0</max>
-            <resolution>0.08</resolution>
-          </range>
-          <noise>
-            <type>gaussian</type>
-            <mean>0.05</mean>
-            <stddev>0.01</stddev>
-          </noise>
-        </ray>
-        <always_on>1</always_on>
-        <visualize>false</visualize>
-      </sensor>
-    </gazebo>
-    <gazebo>
-      <xacro:if value="${simulation_engine == 'ignition-gazebo'}">
-        <plugin filename="libignition-gazebo-sensors-system.so" name="ignition::gazebo::systems::Sensors">
-          <render_engine>ogre2</render_engine>
-        </plugin>
-      </xacro:if>
-      <xacro:if value="${simulation_engine == 'gazebo-classic'}">
-        <plugin name="scan" filename="libgazebo_ros_ray_sensor.so">
-          <ros>
-            <namespace>/</namespace>
-            <argument>~/out:=${topic}</argument>
-          </ros>
-          <output_type>sensor_msgs/LaserScan</output_type>
-          <frame_name>${tf_prefix_ext}${frame_id}</frame_name>
-        </plugin>
-      </xacro:if>
-    </gazebo>
+    <xacro:unless value="${simulation_engine == 'webots'}">
+      <gazebo reference="${tf_prefix_ext}${frame_id}">
+        <sensor type="${ray_type}" name="${tf_prefix_ext}rplidar_a2_sensor">
+          <topic>${topic}</topic>
+          <frame_id>${tf_prefix_ext}${frame_id}</frame_id>
+          <ignition_frame_id>${tf_prefix_ext}${frame_id}</ignition_frame_id>
+          <update_rate>10</update_rate>
+          <ray>
+            <scan>
+              <horizontal>
+                <samples>400</samples>
+                <resolution>1</resolution>
+                <min_angle>-${pi}</min_angle>
+                <max_angle>${pi}</max_angle>
+              </horizontal>
+            </scan>
+            <range>
+              <min>0.2</min>
+              <max>16.0</max>
+              <resolution>0.08</resolution>
+            </range>
+            <noise>
+              <type>gaussian</type>
+              <mean>0.05</mean>
+              <stddev>0.01</stddev>
+            </noise>
+          </ray>
+          <always_on>1</always_on>
+          <visualize>false</visualize>
+        </sensor>
+      </gazebo>
+      <gazebo>
+        <xacro:if value="${simulation_engine == 'ignition-gazebo'}">
+          <plugin filename="libignition-gazebo-sensors-system.so" name="ignition::gazebo::systems::Sensors">
+            <render_engine>ogre2</render_engine>
+          </plugin>
+        </xacro:if>
+        <xacro:if value="${simulation_engine == 'gazebo-classic'}">
+          <plugin name="scan" filename="libgazebo_ros_ray_sensor.so">
+            <ros>
+              <namespace>/</namespace>
+              <argument>~/out:=${topic}</argument>
+            </ros>
+            <output_type>sensor_msgs/LaserScan</output_type>
+            <frame_name>${tf_prefix_ext}${frame_id}</frame_name>
+          </plugin>
+        </xacro:if>
+      </gazebo>
+    </xacro:unless>
   </xacro:macro>
 </robot>

File: rosbot_description/urdf/rosbot.urdf.xacro (robot description, xacro)
@@ -3,6 +3,7 @@
   <xacro:arg name="use_sim" default="false" />
   <xacro:arg name="use_gpu" default="false" />
+  <xacro:arg name="simulation_engine" default="" />
   <xacro:include filename="$(find rosbot_description)/urdf/rosbot_macro.urdf.xacro" ns="husarion" />
-  <xacro:husarion.rosbot_robot use_sim="$(arg use_sim)" />
+  <xacro:husarion.rosbot_robot use_sim="$(arg use_sim)" simulation_engine="$(arg simulation_engine)"/>
   <xacro:include filename="$(find rosbot_description)/urdf/components/rplidar_a2.gazebo.xacro" ns="lidar" />
   <xacro:lidar.rplidar_a2
@@ -11,6 +12,6 @@
     rpy="0.0 0.0 ${-pi}"
     use_gpu="$(arg use_gpu)"
-    simulation_engine="gazebo-classic" />
+    simulation_engine="$(arg simulation_engine)" />
   <xacro:include filename="$(find rosbot_description)/urdf/components/orbbec_astra.gazebo.xacro" ns="camera" />
-  <xacro:camera.orbbec_astra parent_link="camera_link" xyz="0.0 0.0 0.0" rpy="0.0 0.0 0.0" />
+  <xacro:camera.orbbec_astra parent_link="camera_link" xyz="0.0 0.0 0.0" rpy="0.0 0.0 0.0" simulation_engine="$(arg simulation_engine)"/>
 </robot>

File: rosbot_description/urdf/rosbot_macro.urdf.xacro (robot description, xacro)
@@ -1,5 +1,5 @@
 <?xml version='1.0'?>
 <robot xmlns:xacro="http://wiki.ros.org/xacro">
-  <xacro:macro name="rosbot_robot" params="use_sim">
+  <xacro:macro name="rosbot_robot" params="use_sim simulation_engine">
     <xacro:property name="wheel_radius" value="0.0425" />
     <!-- INCLUDE ROBOT PARTS DEFINITIONS -->
@@ -50,7 +50,12 @@
                 rl_wheel_joint,
                 fr_wheel_joint,
-                fl_wheel_joint
+                fl_wheel_jointunless
           </param>
         </xacro:unless>
+        <xacro:if value="$(arg use_sim)">
+          <xacro:if value="${simulation_engine == 'webots'}">
+            <plugin>webots_ros2_control::Ros2ControlSystem</plugin>
+          </xacro:if>
+        </xacro:if>
       </hardware>
       <joint name="fl_wheel_joint">
@@ -77,48 +82,89 @@
     <!-- GAZEBO PLUGINS DECLARATION -->
     <xacro:if value="${use_sim}">
-      <!-- Controll robot wheels -->
-      <gazebo>
-        <plugin name='skid_steer_drive' filename='libgazebo_ros_diff_drive.so'>
-          <ros></ros>
-          <update_rate>10</update_rate>
-          <num_wheel_pairs>2</num_wheel_pairs>
-          <left_joint>fl_wheel_joint</left_joint>
-          <right_joint>fr_wheel_joint</right_joint>
-          <left_joint>rl_wheel_joint</left_joint>
-          <right_joint>rr_wheel_joint</right_joint>
-          <wheel_separation>0.192</wheel_separation>
-          <wheel_separation>0.192</wheel_separation>
-          <wheel_diameter>${wheel_radius*2.0}</wheel_diameter>
-          <wheel_diameter>${wheel_radius*2.0}</wheel_diameter>
-          <max_wheel_torque>1.5</max_wheel_torque>
-          <max_wheel_acceleration>1.0</max_wheel_acceleration>
-          <publish_odom>true</publish_odom>
-          <publish_odom_tf>true</publish_odom_tf>
-          <publish_wheel_tf>true</publish_wheel_tf>
-          <odometry_frame>odom</odometry_frame>
-          <robot_base_frame>base_link</robot_base_frame>
-        </plugin>
-      </gazebo>
-      <!-- publish joint states -->
-      <gazebo>
-        <plugin name="joint_states" filename="libgazebo_ros_joint_state_publisher.so">
-          <joint_name>fl_wheel_joint</joint_name>
-          <joint_name>fr_wheel_joint</joint_name>
-          <joint_name>rl_wheel_joint</joint_name>
-          <joint_name>rr_wheel_joint</joint_name>
-        </plugin>
-      </gazebo>
-      <!-- publish IMU -->
-      <gazebo reference="imu_link">
-        <sensor type="imu" name="imu">
-          <always_on>true</always_on>
-          <update_rate>25</update_rate>
-          <plugin name="bno055_imu_plugin" filename="libgazebo_ros_imu_sensor.so">
+      <xacro:unless value="${simulation_engine == 'webots'}">
+        <!-- Control robot wheels -->
+        <gazebo>
+          <plugin name='skid_steer_drive' filename='libgazebo_ros_diff_drive.so'>
+            <ros></ros>
+            <update_rate>10</update_rate>
+            <num_wheel_pairs>2</num_wheel_pairs>
+            <left_joint>fl_wheel_joint</left_joint>
+            <right_joint>fr_wheel_joint</right_joint>
+            <left_joint>rl_wheel_joint</left_joint>
+            <right_joint>rr_wheel_joint</right_joint>
+            <wheel_separation>0.192</wheel_separation>
+            <wheel_separation>0.192</wheel_separation>
+            <wheel_diameter>${wheel_radius*2.0}</wheel_diameter>
+            <wheel_diameter>${wheel_radius*2.0}</wheel_diameter>
+            <max_wheel_torque>1.5</max_wheel_torque>
+            <max_wheel_acceleration>1.0</max_wheel_acceleration>
+            <publish_odom>true</publish_odom>
+            <publish_odom_tf>true</publish_odom_tf>
+            <publish_wheel_tf>true</publish_wheel_tf>
+            <odometry_frame>odom</odometry_frame>
+            <robot_base_frame>base_link</robot_base_frame>
+          </plugin>
+        </gazebo>
+        <!-- publish joint states -->
+        <gazebo>
+          <plugin name="joint_states" filename="libgazebo_ros_joint_state_publisher.so">
+            <joint_name>fl_wheel_joint</joint_name>
+            <joint_name>fr_wheel_joint</joint_name>
+            <joint_name>rl_wheel_joint</joint_name>
+            <joint_name>rr_wheel_joint</joint_name>
+          </plugin>
+        </gazebo>
+        <!-- publish IMU -->
+        <gazebo reference="imu_link">
+          <sensor type="imu" name="imu">
+            <always_on>true</always_on>
+            <update_rate>25</update_rate>
+            <plugin name="bno055_imu_plugin" filename="libgazebo_ros_imu_sensor.so">
+              <ros>
+                <argument>~/out:=imu/data/raw</argument>
+              </ros>
+            </plugin>
+          </sensor>
+        </gazebo>
+      </xacro:unless>
+      <xacro:if value="${simulation_engine == 'webots'}">
+        <webots>
+          <plugin type="webots_ros2_control::Ros2Control" />
+          <device reference="laser" type="Lidar">
             <ros>
-              <argument>~/out:=imu/data/raw</argument>
+              <topicName>/scan</topicName>
             </ros>
+          </device>
+          <device reference="fl_range" type="DistanceSensor">
+            <ros>
+              <topicName>/range/fl</topicName>
+            </ros>
+          </device>
+          <device reference="fr_range" type="DistanceSensor">
+            <ros>
+              <topicName>/range/fr</topicName>
+            </ros>
+          </device>
+          <device reference="rl_range" type="DistanceSensor">
+            <ros>
+              <topicName>/range/rl</topicName>
+            </ros>
+          </device>
+          <device reference="rr_range" type="DistanceSensor">
+            <ros>
+              <topicName>/range/rr</topicName>
+            </ros>
+          </device>
+          <plugin type="webots_ros2_driver::Ros2IMU">
+            <enabled>true</enabled>
+            <topicName>/imu_broadcaster/imu</topicName>
+            <alwaysOn>true</alwaysOn>
+            <frameName>imu_link</frameName>
+            <gyroName>imu gyro</gyroName>
+            <accelerometerName>imu accelerometer</accelerometerName>
+            <inertialUnitName>imu inertial_unit</inertialUnitName>
           </plugin>
-        </sensor>
-      </gazebo>
+        </webots>
+      </xacro:if>
     </xacro:if>
   </xacro:macro>
