Commit message: Add namespaces (#81)
* added namespaces to ros2_control

Signed-off-by: Jakub Delicat <jakub.delicat@husarion.com>

* removed action group

Signed-off-by: Jakub Delicat <jakub.delicat@husarion.com>

* Added namespace to robot description

Signed-off-by: Jakub Delicat <jakub.delicat@husarion.com>

* added tests for namespaces in rosbot_controller

Signed-off-by: Jakub Delicat <jakub.delicat@husarion.com>

* update worldlist

Signed-off-by: Jakub Delicat <jakub.delicat@husarion.com>

* fixed ros2_control namespaces | added namespace to ekf

Signed-off-by: Jakub Delicat <jakub.delicat@husarion.com>

* added mecanum

Signed-off-by: Jakub Delicat <jakub.delicat@husarion.com>

* added ros2_controllers to .gitignore

Signed-off-by: Jakub Delicat <jakub.delicat@husarion.com>

* ignored ros2_controllers during Industrial CI

Signed-off-by: Jakub Delicat <jakub.delicat@husarion.com>

* fixed tests

Signed-off-by: Jakub Delicat <jakub.delicat@husarion.com>

* added tf_prefix to imu_sensor_broadcaster

Signed-off-by: Jakub Delicat <jakub.delicat@husarion.com>

* copied only diff_drive and imu_broadcaster

Signed-off-by: Jakub Delicat <jakub.delicat@husarion.com>

* changed comments | changed timeout for controller test

Signed-off-by: Jakub Delicat <jakub.delicat@husarion.com>

* param changed to parameter

Signed-off-by: Jakub Delicat <jakub.delicat@husarion.com>

* Multi robot diff drive example

Signed-off-by: Jakub Delicat <jakub.delicat@husarion.com>

* imu also works

Signed-off-by: Jakub Delicat <jakub.delicat@husarion.com>

* Added use_multirobot_system | found imu error

Signed-off-by: Jakub Delicat <jakub.delicat@husarion.com>

* changed all topics to ns

Signed-off-by: Jakub Delicat <jakub.delicat@husarion.com>

* removed tf_prefix from xacro tests

Signed-off-by: Jakub Delicat <jakub.delicat@husarion.com>

* removed comments | add use_multirobot_system arg

Signed-off-by: Jakub Delicat <jakub.delicat@husarion.com>

* moved multi robot system controllers config to rosbot_controller

Signed-off-by: Jakub Delicat <jakub.delicat@husarion.com>

* fixed rosbot_gazebo test

Signed-off-by: Jakub Delicat <jakub.delicat@husarion.com>

* separated namespaced tests | added multirobot gazebo example with broken imu

Signed-off-by: Jakub Delicat <jakub.delicat@husarion.com>

* add multicontroller test

Signed-off-by: Jakub Delicat <jakub.delicat@husarion.com>

* add multibringup test

Signed-off-by: Jakub Delicat <jakub.delicat@husarion.com>

* add multibringup test

Signed-off-by: Jakub Delicat <jakub.delicat@husarion.com>

* Added remove rosbot_macro

Signed-off-by: Jakub Delicat <jakub.delicat@husarion.com>

* fixed miss spelling

Signed-off-by: Jakub Delicat <jakub.delicat@husarion.com>

* The change from robot_hardware_interface seems to be unnecessary

Signed-off-by: Jakub Delicat <jakub.delicat@husarion.com>

* moved multirobot tests to arrays

Signed-off-by: Jakub Delicat <jakub.delicat@husarion.com>

* move rosbot_hardware_interfaces to main

Signed-off-by: Jakub Delicat <jakub.delicat@husarion.com>

* Fixed len

Signed-off-by: Jakub Delicat <jakub.delicat@husarion.com>

* Added updated controllers info to readme

Signed-off-by: Jakub Delicat <jakub.delicat@husarion.com>

* Update README.md

Co-authored-by: rafal-gorecki <126687345+rafal-gorecki@users.noreply.github.com>

* Update README.md

---------

Signed-off-by: Jakub Delicat <jakub.delicat@husarion.com>
Co-authored-by: rafal-gorecki <126687345+rafal-gorecki@users.noreply.github.com>

File: rosbot_description/urdf/components/vl53lox.urdf.xacro (robot description, xacro)
@@ -41,4 +41,7 @@
           <visualize>false</visualize>
         </sensor>
+        <plugin filename="libignition-gazebo-sensors-system.so"  name="ignition::gazebo::systems::Sensors">
+          <render_engine>ogre2</render_engine>
+        </plugin>
       </gazebo>
     </xacro:if>

File: rosbot_description/urdf/rosbot.urdf.xacro (robot description, xacro)
@@ -5,18 +5,28 @@
   <xacro:arg name="mecanum" default="false" />
   <xacro:arg name="simulation_engine" default="" />
+  <xacro:arg name="namespace" default="None" />
+  <xacro:arg name="use_multirobot_system" default="false"/>
   <xacro:include filename="$(find rosbot_description)/urdf/rosbot_macro.urdf.xacro" ns="husarion" />
-  <xacro:husarion.rosbot_robot mecanum="$(arg mecanum)" use_sim="$(arg use_sim)" use_gpu="$(arg use_gpu)" simulation_engine="$(arg simulation_engine)"/>
-  <xacro:include filename="$(find ros_components_description)/urdf/slamtec_rplidar_a2.urdf.xacro" ns="lidar" />
-  <xacro:lidar.slamtec_rplidar_a2
-    parent_link="cover_link"
-    xyz="0.02 0.0 0.0"
-    rpy="0.0 0.0 0.0"
+  <xacro:husarion.rosbot_robot
+    mecanum="$(arg mecanum)"
+    use_sim="$(arg use_sim)"
     use_gpu="$(arg use_gpu)"
-    simulation_engine="$(arg simulation_engine)" />
-  <xacro:include filename="$(find ros_components_description)/urdf/orbbec_astra.urdf.xacro" ns="camera" />
-  <xacro:camera.orbbec_astra
-    parent_link="camera_link"
-    xyz="0.0 0.0 0.0"
-    rpy="0.0 0.0 0.0"
-    simulation_engine="$(arg simulation_engine)" />
+    simulation_engine="$(arg simulation_engine)"
+    namespace="$(arg namespace)"
+    use_multirobot_system="$(arg use_multirobot_system)" />
+    <xacro:unless value="$(arg use_multirobot_system)">
+      <xacro:include filename="$(find ros_components_description)/urdf/slamtec_rplidar_a2.urdf.xacro" ns="lidar" />
+      <xacro:lidar.slamtec_rplidar_a2
+        parent_link="cover_link"
+        xyz="0.02 0.0 0.0"
+        rpy="0.0 0.0 0.0"
+        use_gpu="$(arg use_gpu)"
+        simulation_engine="$(arg simulation_engine)" />
+      <xacro:include filename="$(find ros_components_description)/urdf/orbbec_astra.urdf.xacro" ns="camera" />
+      <xacro:camera.orbbec_astra
+        parent_link="camera_link"
+        xyz="0.0 0.0 0.0"
+        rpy="0.0 0.0 0.0"
+        simulation_engine="$(arg simulation_engine)" />
+    </xacro:unless>
 </robot>

File: rosbot_description/urdf/rosbot_macro.urdf.xacro (robot description, xacro)
@@ -1,5 +1,17 @@
 <?xml version='1.0'?>
 <robot xmlns:xacro="http://wiki.ros.org/xacro">
-  <xacro:macro name="rosbot_robot" params="mecanum use_sim use_gpu simulation_engine">
+  <xacro:macro name="rosbot_robot" params="mecanum use_sim use_gpu simulation_engine namespace use_multirobot_system">
+    <!-- Namespaces are necessary only with multiple robot system in Ignition Gazebo because
+         the same joint states crashes the simulator.
+    -->
+    <xacro:unless value="${use_multirobot_system}">
+      <xacro:property name="namespace" value="None" />
+    </xacro:unless>
+    <xacro:if value="${namespace == 'None'}">
+      <xacro:property name="namespace_ext" value="" />
+    </xacro:if>
+    <xacro:unless value="${namespace == 'None'}">
+        <xacro:property name="namespace_ext" value="${namespace}/" />
+    </xacro:unless>
     <xacro:if value="${mecanum}">
       <xacro:property name="wheel_radius" value="0.0470" />
@@ -12,13 +24,13 @@
     <xacro:include filename="$(find rosbot_description)/urdf/wheel.urdf.xacro" ns="wheel" />
     <!-- BODY DECLARATION -->
-    <xacro:body.body wheel_radius="${wheel_radius}" mecanum="${mecanum}" use_gpu="${use_gpu}" />
+    <xacro:body.body wheel_radius="${wheel_radius}" mecanum="${mecanum}" use_gpu="${use_gpu}" use_multirobot_system="${use_multirobot_system}"/>
     <!-- WHEEL DECLARATION -->
-    <xacro:wheel.wheel wheel_radius="${wheel_radius}" prefix="fr" mecanum="${mecanum}" />
-    <xacro:wheel.wheel wheel_radius="${wheel_radius}" prefix="fl" mecanum="${mecanum}" />
-    <xacro:wheel.wheel wheel_radius="${wheel_radius}" prefix="rl" mecanum="${mecanum}" />
-    <xacro:wheel.wheel wheel_radius="${wheel_radius}" prefix="rr" mecanum="${mecanum}" />
+    <xacro:wheel.wheel wheel_radius="${wheel_radius}" side="fr" mecanum="${mecanum}" namespace="${namespace}" />
+    <xacro:wheel.wheel wheel_radius="${wheel_radius}" side="fl" mecanum="${mecanum}" namespace="${namespace}" />
+    <xacro:wheel.wheel wheel_radius="${wheel_radius}" side="rl" mecanum="${mecanum}" namespace="${namespace}" />
+    <xacro:wheel.wheel wheel_radius="${wheel_radius}" side="rr" mecanum="${mecanum}" namespace="${namespace}" />
     <!-- ROS2 CONTROL -->
     <xacro:unless value="$(arg use_sim)">
-      <ros2_control name="imu" type="sensor">
+      <ros2_control name="${namespace_ext}imu" type="sensor">
         <hardware>
           <plugin>rosbot_hardware_interfaces/RosbotImuSensor</plugin>
@@ -26,5 +38,5 @@
           <param name="connection_check_period_ms">500</param>
         </hardware>
-        <sensor name="imu">
+        <sensor name="${namespace_ext}imu">
           <state_interface name="orientation.x" />
           <state_interface name="orientation.y" />
@@ -40,5 +52,5 @@
       </ros2_control>
     </xacro:unless>
-    <ros2_control name="wheels" type="system">
+    <ros2_control name="${namespace_ext}wheels" type="system">
       <hardware>
         <xacro:unless value="$(arg use_sim)">
@@ -46,5 +58,5 @@
           <param name="connection_timeout_ms">120000</param>
           <param name="connection_check_period_ms">500</param>
-          <!-- order of velocity commands to be published in motors_cmd Float32MultiArray msg -->
+          <!-- Firmware from https://github.com/husarion/rosbot_ros2_firmware could not override this names -->
           <param name="velocity_command_joint_order">
                 rr_wheel_joint,
@@ -63,20 +75,20 @@
         </xacro:if>
       </hardware>
-      <joint name="fl_wheel_joint">
-        <command_interface name="velocity" />
-        <state_interface name="position" />
-        <state_interface name="velocity" />
-      </joint>
-      <joint name="fr_wheel_joint">
-        <command_interface name="velocity" />
-        <state_interface name="position" />
-        <state_interface name="velocity" />
-      </joint>
-      <joint name="rl_wheel_joint">
-        <command_interface name="velocity" />
-        <state_interface name="position" />
-        <state_interface name="velocity" />
-      </joint>
-      <joint name="rr_wheel_joint">
+      <joint name="${namespace_ext}fl_wheel_joint">
+        <command_interface name="velocity" />
+        <state_interface name="position" />
+        <state_interface name="velocity" />
+      </joint>
+      <joint name="${namespace_ext}fr_wheel_joint">
+        <command_interface name="velocity" />
+        <state_interface name="position" />
+        <state_interface name="velocity" />
+      </joint>
+      <joint name="${namespace_ext}rl_wheel_joint">
+        <command_interface name="velocity" />
+        <state_interface name="position" />
+        <state_interface name="velocity" />
+      </joint>
+      <joint name="${namespace_ext}rr_wheel_joint">
         <command_interface name="velocity" />
         <state_interface name="position" />
@@ -85,5 +97,5 @@
       <xacro:if value="${use_sim}">
         <xacro:if value="${simulation_engine == 'ignition-gazebo'}">
-          <sensor name="imu">
+          <sensor name="${namespace_ext}imu">
             <state_interface name="orientation.x" />
             <state_interface name="orientation.y" />
@@ -105,26 +117,40 @@
         <gazebo>
           <plugin filename="ign_ros2_control-system" name="ign_ros2_control::IgnitionROS2ControlPlugin">
+            <xacro:if value="${use_multirobot_system}">
+              <xacro:property name="controller_config_prefix" value="multi_" />
+            </xacro:if>
+            <xacro:unless value="${use_multirobot_system}">
+              <xacro:property name="controller_config_prefix" value="" />
+            </xacro:unless>
             <xacro:if value="${mecanum}">
-              <parameters>$(find rosbot_controller)/config/mecanum_drive_controller.yaml</parameters>
+              <parameters>$(find rosbot_controller)/config/${controller_config_prefix}mecanum_drive_controller.yaml</parameters>
             </xacro:if>
             <xacro:unless value="${mecanum}">
-              <parameters>$(find rosbot_controller)/config/diff_drive_controller.yaml</parameters>
+              <parameters>$(find rosbot_controller)/config/${controller_config_prefix}diff_drive_controller.yaml</parameters>
             </xacro:unless>
-            <controller_manager_prefix_node_name>simulation</controller_manager_prefix_node_name>
             <ros>
-              <remapping>/rosbot_base_controller/cmd_vel_unstamped:=/cmd_vel</remapping>
+              <xacro:unless value="${namespace == 'None'}">
+                <namespace>${namespace}</namespace>
+              </xacro:unless>
+              <remapping>rosbot_base_controller/cmd_vel_unstamped:=cmd_vel</remapping>
+              <remapping>/tf:=tf</remapping>
             </ros>
           </plugin>
         </gazebo>
         <gazebo reference="imu_link">
-          <sensor name="imu" type="imu">
+          <sensor name="${namespace_ext}imu" type="imu">
             <plugin filename="ignition-gazebo-imu-system" name="ignition::gazebo::systems::Imu"></plugin>
             <always_on>true</always_on>
             <update_rate>25</update_rate>
-            <topic>imu/data_raw</topic>
+            <topic>${namespace_ext}imu/data_raw</topic>
             <visualize>false</visualize>
             <enable_metrics>false</enable_metrics>
             <frame_id>imu_link</frame_id>
             <ignition_frame_id>imu_link</ignition_frame_id>
+            <xacro:unless value="${namespace == 'None'}">
+              <ros>
+                <namespace>${namespace}</namespace>
+              </ros>
+            </xacro:unless>
           </sensor>
         </gazebo>

File: rosbot_description/urdf/wheel.urdf.xacro (robot description, xacro)
@@ -2,5 +2,11 @@
 <robot xmlns:xacro="http://www.ros.org/wiki/xacro">
   <!-- wheel defining macro -->
-  <xacro:macro name="wheel" params="wheel_radius prefix mecanum">
+  <xacro:macro name="wheel" params="wheel_radius side mecanum namespace=None">
+    <xacro:if value="${namespace == 'None'}">
+      <xacro:property name="namespace_ext" value="" />
+    </xacro:if>
+    <xacro:unless value="${namespace == 'None'}">
+      <xacro:property name="namespace_ext" value="${namespace}/" />
+    </xacro:unless>
     <xacro:property name="wheel_separation_x" value="0.106" />
     <xacro:if value="${mecanum}">
@@ -22,5 +28,5 @@
       <xacro:property name="wheel_separation_y" value="0.192" />
     </xacro:unless>
-    <xacro:if value="${prefix == 'fl'}">
+    <xacro:if value="${side == 'fl'}">
       <xacro:property name="x" value="${wheel_separation_x/2.0}" />
       <xacro:property name="y" value="${wheel_separation_y/2.0}" />
@@ -29,5 +35,5 @@
       <xacro:property name="fdir" value="1.0 -1.0 0.0" />
     </xacro:if>
-    <xacro:if value="${prefix == 'fr'}">
+    <xacro:if value="${side == 'fr'}">
       <xacro:property name="x" value="${wheel_separation_x/2.0}" />
       <xacro:property name="y" value="${-wheel_separation_y/2.0}" />
@@ -36,5 +42,5 @@
       <xacro:property name="fdir" value="1.0 1.0 0.0" />
     </xacro:if>
-    <xacro:if value="${prefix == 'rl'}">
+    <xacro:if value="${side == 'rl'}">
       <xacro:property name="x" value="${-wheel_separation_x/2}" />
       <xacro:property name="y" value="${wheel_separation_y/2}" />
@@ -43,5 +49,5 @@
       <xacro:property name="fdir" value="1.0 1.0 0.0" />
     </xacro:if>
-    <xacro:if value="${prefix == 'rr'}">
+    <xacro:if value="${side == 'rr'}">
       <xacro:property name="x" value="${-wheel_separation_x/2}" />
       <xacro:property name="y" value="${-wheel_separation_y/2}" />
@@ -50,7 +56,7 @@
       <xacro:property name="fdir" value="1.0 -1.0 0.0" />
     </xacro:if>
-    <joint name="${prefix}_wheel_joint" type="continuous">
+    <joint name="${namespace_ext}${side}_wheel_joint" type="continuous">
       <parent link="body_link" />
-      <child link="${prefix}_wheel_link" />
+      <child link="${side}_wheel_link" />
       <origin xyz="${x} ${y} 0.0" rpy="0.0 0.0 0.0" />
       <axis xyz="0.0 1.0 0.0" />
@@ -58,5 +64,5 @@
       <dynamics damping="0.001" friction="0.001" />
     </joint>
-    <link name="${prefix}_wheel_link">
+    <link name="${side}_wheel_link">
       <visual>
         <geometry>
@@ -78,5 +84,5 @@
       </inertial>
     </link>
-    <gazebo reference="${prefix}_wheel_link" xmlns:ignition="http://ignitionrobotics.org/schema">
+    <gazebo reference="${side}_wheel_link" xmlns:ignition="http://ignitionrobotics.org/schema">
       <collision>
         <surface>

Commit message: Added tests for ranges and camera
Signed-off-by: Jakub Delicat <jakub.delicat@husarion.com>

File: rosbot_description/urdf/components/vl53lox.urdf.xacro (robot description, xacro)
@@ -5,9 +5,7 @@
     <xacro:if value="${namespace == 'None'}">
       <xacro:property name="namespace_ext" value="" />
-      <xacro:property name="gz_control_namespace" value="/" />
     </xacro:if>
     <xacro:unless value="${namespace == 'None'}">
         <xacro:property name="namespace_ext" value="${namespace}/" />
-        <xacro:property name="gz_control_namespace" value="${namespace}" />
     </xacro:unless>
     <joint name="${parent}_${prefix}_range_joint" type="fixed">
@@ -22,5 +20,5 @@
       <gazebo reference="${prefix}_range">
         <sensor name="${namespace_ext}${prefix}_range" type='gpu_lidar'>
-          <topic>${gz_control_namespace}range/${prefix}</topic>
+          <topic>${namespace_ext}range/${prefix}</topic>
           <frame_id>${prefix}_range</frame_id>
           <ignition_frame_id>${prefix}_range</ignition_frame_id>
@@ -49,10 +47,7 @@
           <visualize>false</visualize>
           <ros>
-            <namespace></namespace>
+            <namespace>${namespace_ext}</namespace>
           </ros>
         </sensor>
-        <plugin filename="libignition-gazebo-sensors-system.so"  name="ignition::gazebo::systems::Sensors">
-          <render_engine>ogre2</render_engine>
-        </plugin>
       </gazebo>
     </xacro:if>

File: rosbot_description/urdf/rosbot.urdf.xacro (robot description, xacro)
@@ -14,17 +14,17 @@
     namespace="$(arg namespace)" />
     <xacro:include filename="$(find ros_components_description)/urdf/slamtec_rplidar_a2.urdf.xacro" ns="lidar" />
-      <xacro:lidar.slamtec_rplidar_a2
-        parent_link="cover_link"
-        xyz="0.02 0.0 0.0"
-        rpy="0.0 0.0 0.0"
-        use_gpu="$(arg use_gpu)"
-        namespace="$(arg namespace)"
-        simulation_engine="$(arg simulation_engine)" />
-      <xacro:include filename="$(find ros_components_description)/urdf/orbbec_astra.urdf.xacro" ns="camera" />
-      <xacro:camera.orbbec_astra
-        parent_link="camera_link"
-        xyz="0.0 0.0 0.0"
-        rpy="0.0 0.0 0.0"
-        namespace="$(arg namespace)"
-        simulation_engine="$(arg simulation_engine)" />
+    <xacro:lidar.slamtec_rplidar_a2
+      parent_link="cover_link"
+      xyz="0.02 0.0 0.0"
+      rpy="0.0 0.0 0.0"
+      use_gpu="$(arg use_gpu)"
+      namespace="$(arg namespace)"
+      simulation_engine="$(arg simulation_engine)" />
+    <xacro:include filename="$(find ros_components_description)/urdf/orbbec_astra.urdf.xacro" ns="camera" />
+    <xacro:camera.orbbec_astra
+      parent_link="camera_link"
+      xyz="0.0 0.0 0.0"
+      rpy="0.0 0.0 0.0"
+      namespace="$(arg namespace)"
+      simulation_engine="$(arg simulation_engine)" />
 </robot>
