Commit message: CHange formatting of inertial of wheels

File: rosbot_description/urdf/wheel.urdf.xacro (robot description, xacro)
@@ -56,5 +56,7 @@
       <inertial>
         <mass value="0.100" />
-        <inertia ixx="0.00007" ixy="0" ixz="0" iyy="0.0001263" iyz="0" izz="0.00007" />
+        <inertia ixx="0.00007" ixy="0.0"       ixz="0.0"
+                               iyy="0.0001263" iyz="0.0"
+                                               izz="0.00007" />
       </inertial>
     </link>

Commit message: moved ranges to another file | change mass and inertia for wheels

File: rosbot_description/urdf/wheel.urdf.xacro (robot description, xacro)
@@ -8,8 +8,7 @@
       <xacro:property name="wheel_thickness" value="0.0455" />
       <xacro:property name="mass" value="0.153" />
-      <!-- Normal wheel inertia. Mecanum not implemented yet. -->
-      <xacro:property name="ixx" value="0.00007" />
-      <xacro:property name="iyy" value="0.0001263" />
-      <xacro:property name="izz" value="0.00007" />
+      <xacro:property name="ixx" value="0.000111" />
+      <xacro:property name="iyy" value="0.000111" />
+      <xacro:property name="izz" value="0.000169" />
       <xacro:property name="wheel_separation_y" value="0.205" />
     </xacro:if>
@@ -17,8 +16,8 @@
       <xacro:property name="wheel_file" value="wheel" />
       <xacro:property name="wheel_thickness" value="0.036" />
-      <xacro:property name="mass" value="0.1" />
-      <xacro:property name="ixx" value="0.00007" />
-      <xacro:property name="iyy" value="0.0001263" />
-      <xacro:property name="izz" value="0.00007" />
+      <xacro:property name="mass" value="0.074" />
+      <xacro:property name="ixx" value="0.000041" />
+      <xacro:property name="iyy" value="0.000041" />
+      <xacro:property name="izz" value="0.000067" />
       <xacro:property name="wheel_separation_y" value="0.192" />
     </xacro:unless>

Commit message: changed max vel wheel joint | changed testing velocities to the maximum velocity
Signed-off-by: Jakub Delicat <jakub.delicat@husarion.com>

File: rosbot_description/urdf/wheel.urdf.xacro (robot description, xacro)
@@ -55,5 +55,5 @@
       <origin xyz="${x} ${y} 0.0" rpy="0.0 0.0 0.0" />
       <axis xyz="0.0 1.0 0.0" />
-      <limit effort="1.5" velocity="5.0" />
+      <limit effort="1.5" velocity="24.0" />
       <dynamics damping="0.001" friction="0.001" />
     </joint>
