Commit message: fixed ros2_control namespaces | added namespace to ekf
Signed-off-by: Jakub Delicat <jakub.delicat@husarion.com>

File: rosbot_description/urdf/rosbot_macro.urdf.xacro (robot description, xacro)
@@ -52,10 +52,11 @@
           <param name="connection_timeout_ms">120000</param>
           <param name="connection_check_period_ms">500</param>
+          <!-- Namespaces have not been implemented in microros jet -->
           <!-- order of velocity commands to be published in motors_cmd Float32MultiArray msg -->
           <param name="velocity_command_joint_order">
-                ${tf_prefix_ext}rr_wheel_joint,
-                ${tf_prefix_ext}rl_wheel_joint,
-                ${tf_prefix_ext}fr_wheel_joint,
-                ${tf_prefix_ext}fl_wheel_joint
+                rr_wheel_joint,
+                rl_wheel_joint,
+                fr_wheel_joint,
+                fl_wheel_joint
           </param>
         </xacro:unless>
@@ -69,20 +70,21 @@
         </xacro:if>
       </hardware>
-      <joint name="${tf_prefix_ext}fl_wheel_joint">
-        <command_interface name="velocity" />
-        <state_interface name="position" />
-        <state_interface name="velocity" />
-      </joint>
-      <joint name="${tf_prefix_ext}fr_wheel_joint">
-        <command_interface name="velocity" />
-        <state_interface name="position" />
-        <state_interface name="velocity" />
-      </joint>
-      <joint name="${tf_prefix_ext}rl_wheel_joint">
-        <command_interface name="velocity" />
-        <state_interface name="position" />
-        <state_interface name="velocity" />
-      </joint>
-      <joint name="${tf_prefix_ext}rr_wheel_joint">
+       <!-- Namespaces have not been implemented in microros jet -->
+      <joint name="fl_wheel_joint">
+        <command_interface name="velocity" />
+        <state_interface name="position" />
+        <state_interface name="velocity" />
+      </joint>
+      <joint name="fr_wheel_joint">
+        <command_interface name="velocity" />
+        <state_interface name="position" />
+        <state_interface name="velocity" />
+      </joint>
+      <joint name="rl_wheel_joint">
+        <command_interface name="velocity" />
+        <state_interface name="position" />
+        <state_interface name="velocity" />
+      </joint>
+      <joint name="rr_wheel_joint">
         <command_interface name="velocity" />
         <state_interface name="position" />

File: rosbot_description/urdf/wheel.urdf.xacro (robot description, xacro)
@@ -56,4 +56,5 @@
       <xacro:property name="fdir" value="1.0 -1.0 0.0" />
     </xacro:if>
+    <!-- Namespaces have not been implemented in microros jet -->
     <joint name="${tf_prefix_ext}${side}_wheel_joint" type="continuous">
       <parent link="${tf_prefix_ext}body_link" />

Commit message: added mecanum
Signed-off-by: Jakub Delicat <jakub.delicat@husarion.com>

File: rosbot_description/urdf/rosbot_macro.urdf.xacro (robot description, xacro)
@@ -60,4 +60,5 @@
                 fl_wheel_joint
           </param>
+          <param name="tf_prefix">${tf_prefix_ext}</param>
         </xacro:unless>
         <xacro:if value="$(arg use_sim)">
@@ -71,20 +72,20 @@
       </hardware>
        <!-- Namespaces have not been implemented in microros jet -->
-      <joint name="fl_wheel_joint">
-        <command_interface name="velocity" />
-        <state_interface name="position" />
-        <state_interface name="velocity" />
-      </joint>
-      <joint name="fr_wheel_joint">
-        <command_interface name="velocity" />
-        <state_interface name="position" />
-        <state_interface name="velocity" />
-      </joint>
-      <joint name="rl_wheel_joint">
-        <command_interface name="velocity" />
-        <state_interface name="position" />
-        <state_interface name="velocity" />
-      </joint>
-      <joint name="rr_wheel_joint">
+      <joint name="${tf_prefix_ext}fl_wheel_joint">
+        <command_interface name="velocity" />
+        <state_interface name="position" />
+        <state_interface name="velocity" />
+      </joint>
+      <joint name="${tf_prefix_ext}fr_wheel_joint">
+        <command_interface name="velocity" />
+        <state_interface name="position" />
+        <state_interface name="velocity" />
+      </joint>
+      <joint name="${tf_prefix_ext}rl_wheel_joint">
+        <command_interface name="velocity" />
+        <state_interface name="position" />
+        <state_interface name="velocity" />
+      </joint>
+      <joint name="${tf_prefix_ext}rr_wheel_joint">
         <command_interface name="velocity" />
         <state_interface name="position" />

Commit message: fixed rosbot_gazebo test
Signed-off-by: Jakub Delicat <jakub.delicat@husarion.com>

File: rosbot_description/urdf/rosbot_macro.urdf.xacro (robot description, xacro)
@@ -115,21 +115,17 @@
           <plugin filename="ign_ros2_control-system" name="ign_ros2_control::IgnitionROS2ControlPlugin">
             <xacro:if value="${use_multirobot_system}">
-              <xacro:if value="${mecanum}">
-                <parameters>$(find rosbot_bringup)/config/multi_mecanum_drive_controller.yaml</parameters>
-              </xacro:if>
-              <xacro:unless value="${mecanum}">
-                <parameters>$(find rosbot_bringup)/config/multi_diff_drive_controller.yaml</parameters>
-              </xacro:unless>
+              <xacro:property name="controller_config_prefix" value="multi_" />
             </xacro:if>
             <xacro:unless value="${use_multirobot_system}">
-              <xacro:if value="${mecanum}">
-                <parameters>$(find rosbot_bringup)/config/mecanum_drive_controller.yaml</parameters>
-              </xacro:if>
-              <xacro:unless value="${mecanum}">
-                <parameters>$(find rosbot_bringup)/config/diff_drive_controller.yaml</parameters>
-              </xacro:unless>
+              <xacro:property name="controller_config_prefix" value="simulation_" />
+            </xacro:unless>
+            <xacro:if value="${mecanum}">
+              <parameters>$(find rosbot_controller)/config/${controller_config_prefix}mecanum_drive_controller.yaml</parameters>
+            </xacro:if>
+            <xacro:unless value="${mecanum}">
+              <parameters>$(find rosbot_controller)/config/${controller_config_prefix}diff_drive_controller.yaml</parameters>
             </xacro:unless>
             <ros>
-              <namespace>${namespace}</namespace>
+              <namespace>${namespace_ext}</namespace>
               <remapping>rosbot_base_controller/cmd_vel_unstamped:=cmd_vel</remapping>
               <remapping>/tf:=tf</remapping>
@@ -148,5 +144,5 @@
             <ignition_frame_id>imu_link</ignition_frame_id>
             <ros>
-              <namespace>${namespace}</namespace>
+              <namespace>${namespace_ext}</namespace>
             </ros>
           </sensor>

Commit message: added name for ign_ros2_controller
Signed-off-by: Jakub Delicat <jakub.delicat@husarion.com>

File: rosbot_description/urdf/rosbot_macro.urdf.xacro (robot description, xacro)
@@ -3,5 +3,5 @@
   <xacro:macro name="rosbot_robot" params="mecanum use_sim use_gpu simulation_engine namespace ">
     <xacro:if value="${namespace == 'None'}">
-      <xacro:property name="namespace_ext" value="/" />
+      <xacro:property name="namespace_ext" value="" />
       <xacro:property name="gz_control_namespace" value="/" />
     </xacro:if>
@@ -119,4 +119,5 @@
               <parameters>$(find rosbot_controller)/config/diff_drive_controller.yaml</parameters>
             </xacro:unless>
+            <controller_manager_name>simulation_controller_manager</controller_manager_name>
             <ros>
               <namespace>${gz_control_namespace}</namespace>

Commit message: merged multiple_simulation.launch.py with simulation.launch.py
Signed-off-by: Jakub Delicat <jakub.delicat@husarion.com>

File: rosbot_description/urdf/rosbot_macro.urdf.xacro (robot description, xacro)
@@ -4,9 +4,7 @@
     <xacro:if value="${namespace == 'None'}">
       <xacro:property name="namespace_ext" value="" />
-      <xacro:property name="gz_control_namespace" value="/" />
     </xacro:if>
     <xacro:unless value="${namespace == 'None'}">
         <xacro:property name="namespace_ext" value="${namespace}/" />
-        <xacro:property name="gz_control_namespace" value="${namespace}" />
     </xacro:unless>
     <xacro:if value="${mecanum}">
@@ -120,5 +118,7 @@
             </xacro:unless>
             <ros>
-              <namespace>${gz_control_namespace}</namespace>
+              <xacro:unless value="${namespace == 'None'}">
+                <namespace>${namespace}</namespace>
+              </xacro:unless>
               <remapping>rosbot_base_controller/cmd_vel_unstamped:=cmd_vel</remapping>
               <remapping>/tf:=tf</remapping>

Commit message: hardware jazzy with namespaces
Signed-off-by: Jakub Delicat <jakub.delicat@husarion.com>

File: rosbot_description/urdf/rosbot_macro.urdf.xacro (robot description, xacro)
@@ -62,5 +62,5 @@
         <xacro:if value="$(arg use_sim)">
           <xacro:if value="${simulation_engine == 'ignition-gazebo'}">
-            <plugin>ign_ros2_control/IgnitionSystem</plugin>
+            <plugin>gz_ros2_control/GazeboSimSystem</plugin>
           </xacro:if>
           <xacro:if value="${simulation_engine == 'webots'}">
@@ -110,5 +110,5 @@
       <xacro:if value="${simulation_engine == 'ignition-gazebo'}">
         <gazebo>
-          <plugin filename="ign_ros2_control-system" name="ign_ros2_control::IgnitionROS2ControlPlugin">
+          <plugin filename="gz_ros2_control-system" name="gz_ros2_control::GazeboSimROS2ControlPlugin">
             <xacro:if value="${mecanum}">
               <parameters>$(find rosbot_controller)/config/mecanum_drive_controller.yaml</parameters>
@@ -121,5 +121,5 @@
                 <namespace>${namespace}</namespace>
               </xacro:unless>
-              <remapping>rosbot_base_controller/cmd_vel_unstamped:=cmd_vel</remapping>
+              <remapping>rosbot_base_controller/cmd_vel:=cmd_vel</remapping>
               <remapping>/tf:=tf</remapping>
             </ros>

File: rosbot_description/urdf/wheel.urdf.xacro (robot description, xacro)
@@ -78,17 +78,19 @@
       </inertial>
     </link>
-    <gazebo reference="${side}_wheel_link" xmlns:ignition="http://ignitionrobotics.org/schema">
-      <collision>
-        <surface>
-          <friction>
-            <ode>
-              <mu>1.0</mu>
-              <mu2>0.0</mu2>
-              <fdir1 ignition:expressed_in="base_link">${fdir}</fdir1>
-            </ode>
-          </friction>
-        </surface>
-      </collision>
-    </gazebo>
+    <xacro:if value="${mecanum}">
+      <gazebo reference="${side}_wheel_link" xmlns:ignition="http://ignitionrobotics.org/schema">
+        <collision>
+          <surface>
+            <friction>
+              <ode>
+                <mu>1.0</mu>
+                <mu2>0.0</mu2>
+                <fdir1 ignition:expressed_in="base_link">${fdir}</fdir1>
+              </ode>
+            </friction>
+          </surface>
+        </collision>
+      </gazebo>
+    </xacro:if>
   </xacro:macro>
 </robot>

Commit message: Add scan_filtered test and improve workpace tree

File: rosbot_description/urdf/rosbot_macro.urdf.xacro (robot description, xacro)
@@ -2,16 +2,6 @@
 <robot xmlns:xacro="http://wiki.ros.org/xacro">
   <xacro:macro name="rosbot_robot" params="mecanum use_sim simulation_engine namespace ">
-    <xacro:if value="${namespace == 'None'}">
-      <xacro:property name="namespace_ext" value="" />
-    </xacro:if>
-    <xacro:unless value="${namespace == 'None'}">
-        <xacro:property name="namespace_ext" value="${namespace}/" />
-    </xacro:unless>
-    <xacro:if value="${mecanum}">
-      <xacro:property name="wheel_radius" value="0.0470" />
-    </xacro:if>
-    <xacro:unless value="${mecanum}">
-      <xacro:property name="wheel_radius" value="0.0425" />
-    </xacro:unless>
+    <xacro:property name="ns" value="${namespace + '/' if namespace != 'None' else ''}" />
+    <xacro:property name="wheel_radius" value="${0.0470 if mecanum else 0.0425}" />
     <!-- INCLUDE ROBOT PARTS DEFINITIONS -->
     <xacro:include filename="$(find rosbot_description)/urdf/body.urdf.xacro" ns="body" />
@@ -26,5 +16,5 @@
     <!-- ROS2 CONTROL -->
     <xacro:unless value="$(arg use_sim)">
-      <ros2_control name="${namespace_ext}imu" type="sensor">
+      <ros2_control name="${ns}imu" type="sensor">
         <hardware>
           <plugin>rosbot_hardware_interfaces/RosbotImuSensor</plugin>
@@ -32,5 +22,5 @@
           <param name="connection_check_period_ms">500</param>
         </hardware>
-        <sensor name="${namespace_ext}imu">
+        <sensor name="${ns}imu">
           <state_interface name="orientation.x" />
           <state_interface name="orientation.y" />
@@ -46,5 +36,5 @@
       </ros2_control>
     </xacro:unless>
-    <ros2_control name="${namespace_ext}wheels" type="system">
+    <ros2_control name="${ns}wheels" type="system">
       <hardware>
         <xacro:unless value="$(arg use_sim)">
@@ -91,5 +81,5 @@
       <xacro:if value="${use_sim}">
         <xacro:if value="${simulation_engine == 'ignition-gazebo'}">
-          <sensor name="${namespace_ext}imu">
+          <sensor name="${ns}imu">
             <state_interface name="orientation.x" />
             <state_interface name="orientation.y" />
@@ -127,8 +117,8 @@
         </gazebo>
         <gazebo reference="imu_link">
-          <sensor name="${namespace_ext}imu" type="imu">
+          <sensor name="${ns}imu" type="imu">
             <always_on>true</always_on>
             <update_rate>25</update_rate>
-            <topic>${namespace_ext}imu/data_raw</topic>
+            <topic>${ns}imu/data_raw</topic>
             <visualize>false</visualize>
             <enable_metrics>false</enable_metrics>
@@ -136,5 +126,5 @@
             <ignition_frame_id>imu_link</ignition_frame_id>
             <ros>
-              <namespace>${namespace_ext}</namespace>
+              <namespace>${namespace}</namespace>
             </ros>
           </sensor>

Commit message: Clean up unused arguments (#118)
* Add scan filter

* Clean up

* undo

* added docker setup for local build

* broken ros2 controller - previous worked fine

* Clean up unused arguments

* Fix workflow: Remove spellcheck (redundant), fix integration check

* Fix multiple robot spawn

* fixes

* Delete tools folder

* Pre-commit update and remove redundant flake8

* Fix some tests and set hash in vcs

* Clean up

* Move controller test to bringup and reduce test time

* Fix lidar in simulation

* Rename test files

* Fix tests

* Add scan_filtered test and improve workpace tree

---------

Co-authored-by: Dominik Nowak <dominik.nwk@gmail.com>

File: rosbot_description/urdf/rosbot_macro.urdf.xacro (robot description, xacro)
@@ -1,22 +1,12 @@
 <?xml version='1.0'?>
 <robot xmlns:xacro="http://wiki.ros.org/xacro">
-  <xacro:macro name="rosbot_robot" params="mecanum use_sim use_gpu simulation_engine namespace ">
-    <xacro:if value="${namespace == 'None'}">
-      <xacro:property name="namespace_ext" value="" />
-    </xacro:if>
-    <xacro:unless value="${namespace == 'None'}">
-        <xacro:property name="namespace_ext" value="${namespace}/" />
-    </xacro:unless>
-    <xacro:if value="${mecanum}">
-      <xacro:property name="wheel_radius" value="0.0470" />
-    </xacro:if>
-    <xacro:unless value="${mecanum}">
-      <xacro:property name="wheel_radius" value="0.0425" />
-    </xacro:unless>
+  <xacro:macro name="rosbot_robot" params="mecanum use_sim simulation_engine namespace ">
+    <xacro:property name="ns" value="${namespace + '/' if namespace != 'None' else ''}" />
+    <xacro:property name="wheel_radius" value="${0.0470 if mecanum else 0.0425}" />
     <!-- INCLUDE ROBOT PARTS DEFINITIONS -->
     <xacro:include filename="$(find rosbot_description)/urdf/body.urdf.xacro" ns="body" />
     <xacro:include filename="$(find rosbot_description)/urdf/wheel.urdf.xacro" ns="wheel" />
     <!-- BODY DECLARATION -->
-    <xacro:body.body wheel_radius="${wheel_radius}" mecanum="${mecanum}" use_gpu="${use_gpu}" namespace="${namespace}" />
+    <xacro:body.body wheel_radius="${wheel_radius}" mecanum="${mecanum}" namespace="${namespace}" />
     <!-- WHEEL DECLARATION -->
     <xacro:wheel.wheel wheel_radius="${wheel_radius}" side="fr" mecanum="${mecanum}" />
@@ -26,5 +16,5 @@
     <!-- ROS2 CONTROL -->
     <xacro:unless value="$(arg use_sim)">
-      <ros2_control name="${namespace_ext}imu" type="sensor">
+      <ros2_control name="${ns}imu" type="sensor">
         <hardware>
           <plugin>rosbot_hardware_interfaces/RosbotImuSensor</plugin>
@@ -32,5 +22,5 @@
           <param name="connection_check_period_ms">500</param>
         </hardware>
-        <sensor name="${namespace_ext}imu">
+        <sensor name="${ns}imu">
           <state_interface name="orientation.x" />
           <state_interface name="orientation.y" />
@@ -46,5 +36,5 @@
       </ros2_control>
     </xacro:unless>
-    <ros2_control name="${namespace_ext}wheels" type="system">
+    <ros2_control name="${ns}wheels" type="system">
       <hardware>
         <xacro:unless value="$(arg use_sim)">
@@ -91,5 +81,5 @@
       <xacro:if value="${use_sim}">
         <xacro:if value="${simulation_engine == 'ignition-gazebo'}">
-          <sensor name="${namespace_ext}imu">
+          <sensor name="${ns}imu">
             <state_interface name="orientation.x" />
             <state_interface name="orientation.y" />
@@ -127,8 +117,8 @@
         </gazebo>
         <gazebo reference="imu_link">
-          <sensor name="${namespace_ext}imu" type="imu">
+          <sensor name="${ns}imu" type="imu">
             <always_on>true</always_on>
             <update_rate>25</update_rate>
-            <topic>${namespace_ext}imu/data_raw</topic>
+            <topic>${ns}imu/data_raw</topic>
             <visualize>false</visualize>
             <enable_metrics>false</enable_metrics>
@@ -136,5 +126,5 @@
             <ignition_frame_id>imu_link</ignition_frame_id>
             <ros>
-              <namespace>${namespace_ext}</namespace>
+              <namespace>${namespace}</namespace>
             </ros>
           </sensor>
