Commit message: Fix transforms

File: rosbot_description/urdf/body.urdf.xacro (robot description, xacro)
@@ -14,5 +14,5 @@
           <mesh filename="file://$(find rosbot_description)/meshes/body.stl" scale="0.001 0.001 0.001" />
         </geometry>
-        <origin xyz="0.0 0.0 -0.02" rpy="${pi/2} 0.0 ${pi/2}" />
+        <origin xyz="0.0 0.0 -0.0173" rpy="${pi/2} 0.0 ${pi/2}" />
         <material name="White">
           <color rgba="1.0 1.0 1.0 1.0" />
@@ -34,5 +34,5 @@
     </gazebo>
     <joint name="body_to_cover_joint" type="fixed">
-      <origin xyz="0.0 0.0 0.060" rpy="0.0 0.0 0.0" />
+      <origin xyz="0.0 0.0 0.0603" rpy="0.0 0.0 0.0" />
       <parent link="body_link" />
       <child link="cover_link" />
@@ -57,5 +57,5 @@
     </link>
     <joint name="body_to_imu_joint" type="fixed">
-      <origin xyz="-0.1369 -0.0419 0.0370" rpy="0.0 0.0 0.0" />
+      <origin xyz="0.003 -0.0495 0.04332" rpy="0.0 0.0 0.0" />
       <parent link="body_link" />
       <child link="imu_link" />
@@ -80,5 +80,5 @@
     <joint name="fl_range_joint" type="fixed">
       <axis xyz="0 1 0" />
-      <origin xyz="0.1 0.05 0.01" rpy="0 0 0.13 " />
+      <origin xyz="0.0926 0.05 0.015" rpy="0 0 0.218 " />
       <parent link="body_link" />
       <child link="fl_range" />
@@ -87,5 +87,5 @@
     <joint name="fr_range_joint" type="fixed">
       <axis xyz="0 1 0" />
-      <origin xyz="0.1 -0.05 0.01" rpy="0 0 -0.13 " />
+      <origin xyz="0.0926 -0.05 0.015" rpy="0 0 -0.218 " />
       <parent link="body_link" />
       <child link="fr_range" />
@@ -94,5 +94,5 @@
     <joint name="rl_range_joint" type="fixed">
       <axis xyz="0 1 0" />
-      <origin xyz="-0.1 0.05 0.01" rpy="0 0 3.01 " />
+      <origin xyz="-0.0926 0.05 0.0115" rpy="0 0 2.924 " />
       <parent link="body_link" />
       <child link="rl_range" />
@@ -101,5 +101,5 @@
     <joint name="rr_range_joint" type="fixed">
       <axis xyz="0 1 0" />
-      <origin xyz="-0.1 -0.05 0.01" rpy="0 0 3.27 " />
+      <origin xyz="-0.0926 -0.05 0.0115" rpy="0 0 3.360" />
       <parent link="body_link" />
       <child link="rr_range" />

File: rosbot_description/urdf/components/orbbec_astra.gazebo.xacro (robot description, xacro)
@@ -12,5 +12,5 @@
           <mesh filename="file://$(find rosbot_description)/meshes/components/astra.stl" scale="0.001 0.001 0.001" />
         </geometry>
-        <origin xyz="-0.01 0 0.025" rpy="${pi/2} 0 ${pi/2}" />
+        <origin xyz="-0.01 0 0.0277" rpy="${pi/2} 0 ${pi/2}" />
         <material name="Black">
           <color rgba="0.0 0.0 0.0 1.0" />

File: rosbot_description/urdf/components/rplidar_a2.gazebo.xacro (robot description, xacro)
@@ -30,5 +30,5 @@
           <mesh filename="file://$(find rosbot_description)/meshes/components/rplidar.stl" scale="0.001 0.001 0.001" />
         </geometry>
-        <origin xyz="0.0 0.0 0.0" rpy="${pi/2} 0.0 ${pi/2}" />
+        <origin xyz="0.0 0.0 0.0" rpy="${pi/2} 0.0 ${-pi/2}" />
         <material name="Black">
           <color rgba="0.0 0.0 0.0 1.0" />

Commit message: Add ignition support

File: rosbot_description/urdf/body.urdf.xacro (robot description, xacro)
@@ -27,5 +27,5 @@
       <inertial>
         <mass value="2.0" />
-        <inertia ixx="0.001" ixy="0.000" ixz="0.000" iyy="0.001" iyz="0.000" izz="0.001" />
+        <inertia ixx="0.00721" ixy="0" ixz="0" iyy="0.01035" iyz="0" izz="0.01006" />
       </inertial>
     </link>
@@ -51,8 +51,4 @@
         <material>Gazebo/Red</material>
       </gazebo>
-      <inertial>
-        <mass value="0.000001" />
-        <inertia ixx="1.0" ixy="0.0" ixz="0.0" iyy="1.0" iyz="0.0" izz="0.0" />
-      </inertial>
     </link>
     <joint name="body_to_imu_joint" type="fixed">
@@ -61,10 +57,5 @@
       <child link="imu_link" />
     </joint>
-    <link name="imu_link">
-      <inertial>
-        <mass value="0.001" />
-        <inertia ixx="1" ixy="0" ixz="0" iyy="1" iyz="0" izz="1" />
-      </inertial>
-    </link>
+    <link name="imu_link" />
     <joint name="body_to_camera_joint" type="fixed">
       <origin xyz="-0.0141 0.0 0.125" rpy="0.0 0.0 0.0" />
@@ -72,10 +63,5 @@
       <child link="camera_link" />
     </joint>
-    <link name="camera_link">
-      <inertial>
-        <mass value="0.000001" />
-        <inertia ixx="1" ixy="0" ixz="0" iyy="1" iyz="0" izz="1" />
-      </inertial>
-    </link>
+    <link name="camera_link" />
     <joint name="fl_range_joint" type="fixed">
       <axis xyz="0 1 0" />
@@ -84,5 +70,5 @@
       <child link="fl_range" />
     </joint>
-    <link name="fl_range"></link>
+    <link name="fl_range" />
     <joint name="fr_range_joint" type="fixed">
       <axis xyz="0 1 0" />
@@ -91,5 +77,5 @@
       <child link="fr_range" />
     </joint>
-    <link name="fr_range"></link>
+    <link name="fr_range" />
     <joint name="rl_range_joint" type="fixed">
       <axis xyz="0 1 0" />
@@ -98,5 +84,5 @@
       <child link="rl_range" />
     </joint>
-    <link name="rl_range"></link>
+    <link name="rl_range" />
     <joint name="rr_range_joint" type="fixed">
       <axis xyz="0 1 0" />
@@ -105,5 +91,5 @@
       <child link="rr_range" />
     </joint>
-    <link name="rr_range"></link>
+    <link name="rr_range" />
   </xacro:macro>
 </robot>

File: rosbot_description/urdf/rosbot_macro.urdf.xacro (robot description, xacro)
@@ -50,4 +50,7 @@
         </xacro:unless>
         <xacro:if value="$(arg use_sim)">
+          <xacro:if value="${simulation_engine == 'ignition-gazebo'}">
+            <plugin>ign_ros2_control/IgnitionSystem</plugin>
+          </xacro:if>
           <xacro:if value="${simulation_engine == 'webots'}">
             <plugin>webots_ros2_control::Ros2ControlSystem</plugin>
@@ -75,7 +78,46 @@
         <state_interface name="velocity" />
       </joint>
+      <xacro:if value="${use_sim}">
+        <xacro:if value="${simulation_engine == 'ignition-gazebo'}">
+          <sensor name="imu">
+            <state_interface name="orientation.x" />
+            <state_interface name="orientation.y" />
+            <state_interface name="orientation.z" />
+            <state_interface name="orientation.w" />
+            <state_interface name="angular_velocity.x" />
+            <state_interface name="angular_velocity.y" />
+            <state_interface name="angular_velocity.z" />
+            <state_interface name="linear_acceleration.x" />
+            <state_interface name="linear_acceleration.y" />
+            <state_interface name="linear_acceleration.z" />
+          </sensor>
+        </xacro:if>
+      </xacro:if>
     </ros2_control>
     <!-- GAZEBO PLUGINS DECLARATION -->
     <xacro:if value="${use_sim}">
+      <xacro:if value="${simulation_engine == 'ignition-gazebo'}">
+        <gazebo>
+          <plugin filename="ign_ros2_control-system" name="ign_ros2_control::IgnitionROS2ControlPlugin">
+            <parameters>$(find rosbot_controller)/config/rosbot_controllers.yaml</parameters>
+            <controller_manager_prefix_node_name>simulation</controller_manager_prefix_node_name>
+            <ros>
+              <remapping>/rosbot_base_controller/cmd_vel_unstamped:=/cmd_vel</remapping>
+            </ros>
+          </plugin>
+        </gazebo>
+        <gazebo reference="imu_link">
+          <sensor name="imu" type="imu">
+            <plugin filename="ignition-gazebo-imu-system" name="ignition::gazebo::systems::Imu"></plugin>
+            <always_on>true</always_on>
+            <update_rate>25</update_rate>
+            <topic>imu/data_raw</topic>
+            <visualize>false</visualize>
+            <enable_metrics>false</enable_metrics>
+            <frame_id>imu_link</frame_id>
+            <ignition_frame_id>imu_link</ignition_frame_id>
+          </sensor>
+        </gazebo>
+      </xacro:if>
       <xacro:if value="${simulation_engine == 'gazebo-classic'}">
         <!-- Control robot wheels -->

File: rosbot_description/urdf/wheel.urdf.xacro (robot description, xacro)
@@ -56,7 +56,5 @@
       <inertial>
         <mass value="0.100" />
-        <inertia ixx="0.001" ixy="0.000" ixz="0.000"
-                             iyy="0.001" iyz="0.000"
-                                         izz="0.001" />
+        <inertia ixx="0.00007" ixy="0" ixz="0" iyy="0.0001263" iyz="0" izz="0.00007" />
       </inertial>
     </link>

Commit message: changed wheels models | added mecanum controller

File: rosbot_description/urdf/body.urdf.xacro (robot description, xacro)
@@ -2,5 +2,5 @@
 <robot xmlns:xacro="http://www.ros.org/wiki/xacro">
   <!-- body defining macro -->
-  <xacro:macro name="body" params="wheel_radius">
+  <xacro:macro name="body" params="wheel_radius mecanum">
     <link name="base_link" />
     <joint name="base_to_body_joint" type="fixed">

File: rosbot_description/urdf/rosbot.urdf.xacro (robot description, xacro)
@@ -3,7 +3,8 @@
   <xacro:arg name="use_sim" default="false" />
   <xacro:arg name="use_gpu" default="false" />
+  <xacro:arg name="mecanum" default="false" />
   <xacro:arg name="simulation_engine" default="" />
   <xacro:include filename="$(find rosbot_description)/urdf/rosbot_macro.urdf.xacro" ns="husarion" />
-  <xacro:husarion.rosbot_robot use_sim="$(arg use_sim)" simulation_engine="$(arg simulation_engine)"/>
+  <xacro:husarion.rosbot_robot mecanum="$(arg mecanum)" use_sim="$(arg use_sim)" simulation_engine="$(arg simulation_engine)"/>
   <xacro:include filename="$(find ros_components_description)/urdf/slamtec_rplidar_a2.urdf.xacro" ns="lidar" />
   <xacro:lidar.slamtec_rplidar_a2

File: rosbot_description/urdf/rosbot_macro.urdf.xacro (robot description, xacro)
@@ -1,16 +1,21 @@
 <?xml version='1.0'?>
 <robot xmlns:xacro="http://wiki.ros.org/xacro">
-  <xacro:macro name="rosbot_robot" params="use_sim simulation_engine">
-    <xacro:property name="wheel_radius" value="0.0425" />
+  <xacro:macro name="rosbot_robot" params="mecanum use_sim simulation_engine">
+    <xacro:if value="${mecanum}">
+      <xacro:property name="wheel_radius" value="0.0470" />
+    </xacro:if>
+    <xacro:unless value="${mecanum}">
+      <xacro:property name="wheel_radius" value="0.0425" />
+    </xacro:unless>
     <!-- INCLUDE ROBOT PARTS DEFINITIONS -->
     <xacro:include filename="$(find rosbot_description)/urdf/body.urdf.xacro" ns="body" />
     <xacro:include filename="$(find rosbot_description)/urdf/wheel.urdf.xacro" ns="wheel" />
     <!-- BODY DECLARATION -->
-    <xacro:body.body wheel_radius="${wheel_radius}" />
+    <xacro:body.body wheel_radius="${wheel_radius}" mecanum="${mecanum}" />
     <!-- WHEEL DECLARATION -->
-    <xacro:wheel.wheel wheel_type="differential" wheel_radius="${wheel_radius}" prefix="fl" />
-    <xacro:wheel.wheel wheel_type="differential" wheel_radius="${wheel_radius}" prefix="fr" />
-    <xacro:wheel.wheel wheel_type="differential" wheel_radius="${wheel_radius}" prefix="rl" />
-    <xacro:wheel.wheel wheel_type="differential" wheel_radius="${wheel_radius}" prefix="rr" />
+    <xacro:wheel.wheel wheel_radius="${wheel_radius}" prefix="fr" mecanum="${mecanum}" use_sim="${use_sim}" />
+    <xacro:wheel.wheel wheel_radius="${wheel_radius}" prefix="fl" mecanum="${mecanum}" use_sim="${use_sim}" />
+    <xacro:wheel.wheel wheel_radius="${wheel_radius}" prefix="rl" mecanum="${mecanum}" use_sim="${use_sim}" />
+    <xacro:wheel.wheel wheel_radius="${wheel_radius}" prefix="rr" mecanum="${mecanum}" use_sim="${use_sim}" />
     <!-- ROS2 CONTROL -->
     <xacro:unless value="$(arg use_sim)">
@@ -80,26 +85,28 @@
       <xacro:if value="${simulation_engine == 'gazebo-classic'}">
         <!-- Control robot wheels -->
-        <gazebo>
-          <plugin name='skid_steer_drive' filename='libgazebo_ros_diff_drive.so'>
-            <ros></ros>
-            <update_rate>10</update_rate>
-            <num_wheel_pairs>2</num_wheel_pairs>
-            <left_joint>fl_wheel_joint</left_joint>
-            <right_joint>fr_wheel_joint</right_joint>
-            <left_joint>rl_wheel_joint</left_joint>
-            <right_joint>rr_wheel_joint</right_joint>
-            <wheel_separation>0.192</wheel_separation>
-            <wheel_separation>0.192</wheel_separation>
-            <wheel_diameter>${wheel_radius*2.0}</wheel_diameter>
-            <wheel_diameter>${wheel_radius*2.0}</wheel_diameter>
-            <max_wheel_torque>1.5</max_wheel_torque>
-            <max_wheel_acceleration>1.0</max_wheel_acceleration>
-            <publish_odom>true</publish_odom>
-            <publish_odom_tf>true</publish_odom_tf>
-            <publish_wheel_tf>true</publish_wheel_tf>
-            <odometry_frame>odom</odometry_frame>
-            <robot_base_frame>base_link</robot_base_frame>
-          </plugin>
-        </gazebo>
+        <xacro:unless value="${mecanum}">
+          <gazebo>
+            <plugin name='skid_steer_drive' filename='libgazebo_ros_diff_drive.so'>
+              <ros></ros>
+              <update_rate>10</update_rate>
+              <num_wheel_pairs>2</num_wheel_pairs>
+              <left_joint>fl_wheel_joint</left_joint>
+              <right_joint>fr_wheel_joint</right_joint>
+              <left_joint>rl_wheel_joint</left_joint>
+              <right_joint>rr_wheel_joint</right_joint>
+              <wheel_separation>0.192</wheel_separation>
+              <wheel_separation>0.192</wheel_separation>
+              <wheel_diameter>${wheel_radius*2.0}</wheel_diameter>
+              <wheel_diameter>${wheel_radius*2.0}</wheel_diameter>
+              <max_wheel_torque>1.5</max_wheel_torque>
+              <max_wheel_acceleration>1.0</max_wheel_acceleration>
+              <publish_odom>true</publish_odom>
+              <publish_odom_tf>true</publish_odom_tf>
+              <publish_wheel_tf>true</publish_wheel_tf>
+              <odometry_frame>odom</odometry_frame>
+              <robot_base_frame>base_link</robot_base_frame>
+            </plugin>
+          </gazebo>
+        </xacro:unless>
         <!-- publish joint states -->
         <gazebo>

File: rosbot_description/urdf/wheel.urdf.xacro (robot description, xacro)
@@ -2,31 +2,52 @@
 <robot xmlns:xacro="http://www.ros.org/wiki/xacro">
   <!-- wheel defining macro -->
-  <xacro:macro name="wheel" params="wheel_type wheel_radius prefix">
+  <xacro:macro name="wheel" params="wheel_radius prefix mecanum use_sim">
     <xacro:property name="wheel_separation_x" value="0.106" />
-    <xacro:property name="wheel_separation_y" value="0.228" />
-    <xacro:property name="wheel_thickness" value="0.036" />
+    <xacro:if value="${mecanum}">
+      <xacro:property name="wheel_file" value="mecanum" />
+      <xacro:property name="wheel_thickness" value="0.0455" />
+      <!-- Normal wheel inertia and mass. Mecanum not implemented yet. -->
+      <xacro:property name="mass" value="0.1" />
+      <xacro:property name="ixx" value="0.00007" />
+      <xacro:property name="iyy" value="0.0001263" />
+      <xacro:property name="izz" value="0.00007" />
+      <xacro:property name="wheel_separation_y" value="0.205" />
+    </xacro:if>
+    <xacro:unless value="${mecanum}">
+      <xacro:property name="wheel_file" value="wheel" />
+      <xacro:property name="wheel_thickness" value="0.036" />
+      <xacro:property name="mass" value="0.1" />
+      <xacro:property name="ixx" value="0.00007" />
+      <xacro:property name="iyy" value="0.0001263" />
+      <xacro:property name="izz" value="0.00007" />
+      <xacro:property name="wheel_separation_y" value="0.192" />
+    </xacro:unless>
     <xacro:if value="${prefix == 'fl'}">
       <xacro:property name="x" value="${wheel_separation_x/2}" />
-      <xacro:property name="y" value="${wheel_separation_y/2 - wheel_thickness/2}" />
-      <xacro:property name="y_correction" value="${wheel_thickness/2 - 0.005}" />
-      <xacro:property name="rot" value="${pi/2}" />
+      <xacro:property name="y" value="${wheel_separation_y/2}" />
+      <xacro:property name="mesh" value="file://$(find rosbot_description)/meshes/${wheel_file}_b.dae" />
+      <xacro:property name="visual_rotation" value="${pi}" />
+      <xacro:property name="fdir" value="1 -1 0" />
     </xacro:if>
     <xacro:if value="${prefix == 'fr'}">
       <xacro:property name="x" value="${wheel_separation_x/2}" />
-      <xacro:property name="y" value="-${wheel_separation_y/2 - wheel_thickness/2}" />
-      <xacro:property name="y_correction" value="-${wheel_thickness/2 - 0.005}" />
-      <xacro:property name="rot" value="${-pi/2}" />
+      <xacro:property name="y" value="${-wheel_separation_y/2}" />
+      <xacro:property name="mesh" value="file://$(find rosbot_description)/meshes/${wheel_file}_a.dae" />
+      <xacro:property name="visual_rotation" value="${pi}" />
+      <xacro:property name="fdir" value="1 1 0" />
     </xacro:if>
     <xacro:if value="${prefix == 'rl'}">
-      <xacro:property name="x" value="-${wheel_separation_x/2}" />
-      <xacro:property name="y" value="${wheel_separation_y/2 - wheel_thickness/2}" />
-      <xacro:property name="y_correction" value="${wheel_thickness/2 - 0.005}" />
-      <xacro:property name="rot" value="${pi/2}" />
+      <xacro:property name="x" value="${-wheel_separation_x/2}" />
+      <xacro:property name="y" value="${wheel_separation_y/2}" />
+      <xacro:property name="mesh" value="file://$(find rosbot_description)/meshes/${wheel_file}_a.dae" />
+      <xacro:property name="visual_rotation" value="${0.0}" />
+      <xacro:property name="fdir" value="1 1 0" />
     </xacro:if>
     <xacro:if value="${prefix == 'rr'}">
-      <xacro:property name="x" value="-${wheel_separation_x/2}" />
-      <xacro:property name="y" value="-${wheel_separation_y/2 - wheel_thickness/2}" />
-      <xacro:property name="y_correction" value="-${wheel_thickness/2 - 0.005}" />
-      <xacro:property name="rot" value="${-pi/2}" />
+      <xacro:property name="x" value="${-wheel_separation_x/2}" />
+      <xacro:property name="y" value="${-wheel_separation_y/2}" />
+      <xacro:property name="mesh" value="file://$(find rosbot_description)/meshes/${wheel_file}_b.dae" />
+      <xacro:property name="visual_rotation" value="${0.0}" />
+      <xacro:property name="fdir" value="1 -1 0" />
     </xacro:if>
     <joint name="${prefix}_wheel_joint" type="continuous">
@@ -41,10 +62,7 @@
       <visual>
         <geometry>
-          <mesh filename="file://$(find rosbot_description)/meshes/wheel.stl" scale="0.001 0.001 0.001" />
+          <mesh filename="${mesh}" scale="1 1 1" />
         </geometry>
-        <origin xyz="0.0 ${y_correction} 0.0" rpy="0.0 0.0 ${rot}" />
-        <material name="Black">
-          <color rgba="0.0 0.0 0.0 1.0" />
-        </material>
+        <origin xyz="0.0 0.0 0.0" rpy="0 0 ${visual_rotation}" />
       </visual>
       <collision>
@@ -55,13 +73,25 @@
       </collision>
       <inertial>
-        <mass value="0.100" />
-        <inertia ixx="0.001" ixy="0.000" ixz="0.000"
-                             iyy="0.001" iyz="0.000"
-                                         izz="0.001" />
+        <mass value="${mass}" />
+        <inertia ixx="${ixx}" ixy="0.0"    ixz="0.0"
+                              iyy="${iyy}" iyz="0.0"
+                                           izz="${izz}" />
       </inertial>
     </link>
-    <gazebo reference="${prefix}_wheel_link">
-      <material>Gazebo/DarkGrey</material>
-    </gazebo>
+    <xacro:if value="${use_sim}">
+      <gazebo reference="${prefix}_wheel_link" xmlns:ignition="http://ignitionrobotics.org/schema">
+        <collision>
+          <surface>
+            <friction>
+              <ode>
+                <mu>1.0</mu>
+                <mu2>0.0</mu2>
+                <fdir1 ignition:expressed_in="base_link">${fdir}</fdir1>
+              </ode>
+            </friction>
+          </surface>
+        </collision>
+      </gazebo>
+    </xacro:if>
   </xacro:macro>
 </robot>
