Commit message: move range sensors to other xacro

File: rosbot_description/urdf/body.urdf.xacro (robot description, xacro)
@@ -3,4 +3,5 @@
   <!-- body defining macro -->
   <xacro:macro name="body" params="wheel_radius mecanum">
+    <xacro:include filename="$(find rosbot_description)/urdf/components/vl53lox.urdf.xacro" ns="range_sensor" />
     <link name="base_link" />
     <joint name="base_to_body_joint" type="fixed">
@@ -64,32 +65,8 @@
     </joint>
     <link name="camera_link" />
-    <joint name="fl_range_joint" type="fixed">
-      <axis xyz="0 1 0" />
-      <origin xyz="0.0926 0.05 0.015" rpy="0 0 0.218 " />
-      <parent link="body_link" />
-      <child link="fl_range" />
-    </joint>
-    <link name="fl_range" />
-    <joint name="fr_range_joint" type="fixed">
-      <axis xyz="0 1 0" />
-      <origin xyz="0.0926 -0.05 0.015" rpy="0 0 -0.218 " />
-      <parent link="body_link" />
-      <child link="fr_range" />
-    </joint>
-    <link name="fr_range" />
-    <joint name="rl_range_joint" type="fixed">
-      <axis xyz="0 1 0" />
-      <origin xyz="-0.0926 0.05 0.0115" rpy="0 0 2.924 " />
-      <parent link="body_link" />
-      <child link="rl_range" />
-    </joint>
-    <link name="rl_range" />
-    <joint name="rr_range_joint" type="fixed">
-      <axis xyz="0 1 0" />
-      <origin xyz="-0.0926 -0.05 0.0115" rpy="0 0 3.360" />
-      <parent link="body_link" />
-      <child link="rr_range" />
-    </joint>
-    <link name="rr_range" />
+    <xacro:range_sensor.vl53lox xyz="0.0926  0.05 0.015"   parent="body_link" z="12.5"  prefix="fl" />
+    <xacro:range_sensor.vl53lox xyz="0.0926 -0.05 0.015"   parent="body_link" z="-12.5" prefix="fr" />
+    <xacro:range_sensor.vl53lox xyz="-0.0926 0.05 0.0115"  parent="body_link" z="167.5" prefix="rl" />
+    <xacro:range_sensor.vl53lox xyz="-0.0926 -0.05 0.0115" parent="body_link" z="192.5" prefix="rr" />
   </xacro:macro>
 </robot>

File: rosbot_description/urdf/rosbot_macro.urdf.xacro (robot description, xacro)
@@ -14,8 +14,8 @@
     <xacro:body.body wheel_radius="${wheel_radius}" mecanum="${mecanum}" />
     <!-- WHEEL DECLARATION -->
-    <xacro:wheel.wheel wheel_radius="${wheel_radius}" prefix="fr" mecanum="${mecanum}" use_sim="${use_sim}" />
-    <xacro:wheel.wheel wheel_radius="${wheel_radius}" prefix="fl" mecanum="${mecanum}" use_sim="${use_sim}" />
-    <xacro:wheel.wheel wheel_radius="${wheel_radius}" prefix="rl" mecanum="${mecanum}" use_sim="${use_sim}" />
-    <xacro:wheel.wheel wheel_radius="${wheel_radius}" prefix="rr" mecanum="${mecanum}" use_sim="${use_sim}" />
+    <xacro:wheel.wheel wheel_radius="${wheel_radius}" prefix="fr" mecanum="${mecanum}" />
+    <xacro:wheel.wheel wheel_radius="${wheel_radius}" prefix="fl" mecanum="${mecanum}" />
+    <xacro:wheel.wheel wheel_radius="${wheel_radius}" prefix="rl" mecanum="${mecanum}" />
+    <xacro:wheel.wheel wheel_radius="${wheel_radius}" prefix="rr" mecanum="${mecanum}" />
     <!-- ROS2 CONTROL -->
     <xacro:unless value="$(arg use_sim)">

File: rosbot_description/urdf/wheel.urdf.xacro (robot description, xacro)
@@ -2,11 +2,11 @@
 <robot xmlns:xacro="http://www.ros.org/wiki/xacro">
   <!-- wheel defining macro -->
-  <xacro:macro name="wheel" params="wheel_radius prefix mecanum use_sim">
+  <xacro:macro name="wheel" params="wheel_radius prefix mecanum">
     <xacro:property name="wheel_separation_x" value="0.106" />
     <xacro:if value="${mecanum}">
       <xacro:property name="wheel_file" value="mecanum" />
       <xacro:property name="wheel_thickness" value="0.0455" />
-      <!-- Normal wheel inertia and mass. Mecanum not implemented yet. -->
-      <xacro:property name="mass" value="0.1" />
+      <xacro:property name="mass" value="0.153" />
+      <!-- Normal wheel inertia. Mecanum not implemented yet. -->
       <xacro:property name="ixx" value="0.00007" />
       <xacro:property name="iyy" value="0.0001263" />
@@ -28,5 +28,5 @@
       <xacro:property name="mesh" value="file://$(find rosbot_description)/meshes/${wheel_file}_b.dae" />
       <xacro:property name="visual_rotation" value="${pi}" />
-      <xacro:property name="fdir" value="1 -1 0" />
+      <xacro:property name="fdir" value="1.0 -1.0 0.0" />
     </xacro:if>
     <xacro:if value="${prefix == 'fr'}">
@@ -35,5 +35,5 @@
       <xacro:property name="mesh" value="file://$(find rosbot_description)/meshes/${wheel_file}_a.dae" />
       <xacro:property name="visual_rotation" value="${pi}" />
-      <xacro:property name="fdir" value="1 1 0" />
+      <xacro:property name="fdir" value="1.0 1.0 0.0" />
     </xacro:if>
     <xacro:if value="${prefix == 'rl'}">
@@ -42,5 +42,5 @@
       <xacro:property name="mesh" value="file://$(find rosbot_description)/meshes/${wheel_file}_a.dae" />
       <xacro:property name="visual_rotation" value="${0.0}" />
-      <xacro:property name="fdir" value="1 1 0" />
+      <xacro:property name="fdir" value="1.0 1.0 0.0" />
     </xacro:if>
     <xacro:if value="${prefix == 'rr'}">
@@ -49,5 +49,5 @@
       <xacro:property name="mesh" value="file://$(find rosbot_description)/meshes/${wheel_file}_b.dae" />
       <xacro:property name="visual_rotation" value="${0.0}" />
-      <xacro:property name="fdir" value="1 -1 0" />
+      <xacro:property name="fdir" value="1.0 -1.0 0.0" />
     </xacro:if>
     <joint name="${prefix}_wheel_joint" type="continuous">
@@ -62,7 +62,7 @@
       <visual>
         <geometry>
-          <mesh filename="${mesh}" scale="1 1 1" />
+          <mesh filename="${mesh}" scale="1.0 1.0 1.0" />
         </geometry>
-        <origin xyz="0.0 0.0 0.0" rpy="0 0 ${visual_rotation}" />
+        <origin xyz="0.0 0.0 0.0" rpy="0.0 0.0 ${visual_rotation}" />
       </visual>
       <collision>
@@ -79,19 +79,17 @@
       </inertial>
     </link>
-    <xacro:if value="${use_sim}">
-      <gazebo reference="${prefix}_wheel_link" xmlns:ignition="http://ignitionrobotics.org/schema">
-        <collision>
-          <surface>
-            <friction>
-              <ode>
-                <mu>1.0</mu>
-                <mu2>0.0</mu2>
-                <fdir1 ignition:expressed_in="base_link">${fdir}</fdir1>
-              </ode>
-            </friction>
-          </surface>
-        </collision>
-      </gazebo>
-    </xacro:if>
+    <gazebo reference="${prefix}_wheel_link" xmlns:ignition="http://ignitionrobotics.org/schema">
+      <collision>
+        <surface>
+          <friction>
+            <ode>
+              <mu>1.0</mu>
+              <mu2>0.0</mu2>
+              <fdir1 ignition:expressed_in="base_link">${fdir}</fdir1>
+            </ode>
+          </friction>
+        </surface>
+      </collision>
+    </gazebo>
   </xacro:macro>
 </robot>

Commit message: rpy arg

File: rosbot_description/urdf/body.urdf.xacro (robot description, xacro)
@@ -65,8 +65,8 @@
     </joint>
     <link name="camera_link" />
-    <xacro:range_sensor.vl53lox xyz="0.0926  0.05 0.015"   parent="body_link" z="12.5"  prefix="fl" />
-    <xacro:range_sensor.vl53lox xyz="0.0926 -0.05 0.015"   parent="body_link" z="-12.5" prefix="fr" />
-    <xacro:range_sensor.vl53lox xyz="-0.0926 0.05 0.0115"  parent="body_link" z="167.5" prefix="rl" />
-    <xacro:range_sensor.vl53lox xyz="-0.0926 -0.05 0.0115" parent="body_link" z="192.5" prefix="rr" />
+    <xacro:range_sensor.vl53lox xyz="0.0926  0.05 0.015"   parent="body_link" rpy="0.0 0.0 ${12.5  * pi/180}"  prefix="fl" />
+    <xacro:range_sensor.vl53lox xyz="0.0926 -0.05 0.015"   parent="body_link" rpy="0.0 0.0 ${-12.5 * pi/180}" prefix="fr" />
+    <xacro:range_sensor.vl53lox xyz="-0.0926 0.05 0.0115"  parent="body_link" rpy="0.0 0.0 ${167.5 * pi/180}" prefix="rl" />
+    <xacro:range_sensor.vl53lox xyz="-0.0926 -0.05 0.0115" parent="body_link" rpy="0.0 0.0 ${192.5 * pi/180}" prefix="rr" />
   </xacro:macro>
 </robot>

File: rosbot_description/urdf/components/vl53lox.urdf.xacro (robot description, xacro)
@@ -2,7 +2,7 @@
 <robot xmlns:xacro="http://www.ros.org/wiki/xacro">
   <!-- vl53lox defining macro -->
-  <xacro:macro name="vl53lox" params="xyz z prefix parent">
+  <xacro:macro name="vl53lox" params="xyz rpy prefix parent">
     <joint name="${parent}_${prefix}_range_joint" type="fixed">
-        <origin xyz="${xyz}" rpy="0.0 0.0 ${z * pi/180}" />
+        <origin xyz="${xyz}" rpy="${rpy}" />
         <parent link="${parent}" />
         <child link="${prefix}_range" />

Commit message: changed args order

File: rosbot_description/urdf/body.urdf.xacro (robot description, xacro)
@@ -65,8 +65,8 @@
     </joint>
     <link name="camera_link" />
-    <xacro:range_sensor.vl53lox xyz="0.0926  0.05 0.015"   parent="body_link" rpy="0.0 0.0 ${12.5  * pi/180}"  prefix="fl" />
-    <xacro:range_sensor.vl53lox xyz="0.0926 -0.05 0.015"   parent="body_link" rpy="0.0 0.0 ${-12.5 * pi/180}" prefix="fr" />
-    <xacro:range_sensor.vl53lox xyz="-0.0926 0.05 0.0115"  parent="body_link" rpy="0.0 0.0 ${167.5 * pi/180}" prefix="rl" />
-    <xacro:range_sensor.vl53lox xyz="-0.0926 -0.05 0.0115" parent="body_link" rpy="0.0 0.0 ${192.5 * pi/180}" prefix="rr" />
+    <xacro:range_sensor.vl53lox parent="body_link" xyz="0.0926  0.05 0.015"   rpy="0.0 0.0 ${12.5  * pi/180}" prefix="fl" />
+    <xacro:range_sensor.vl53lox parent="body_link" xyz="0.0926 -0.05 0.015"   rpy="0.0 0.0 ${-12.5 * pi/180}" prefix="fr" />
+    <xacro:range_sensor.vl53lox parent="body_link" xyz="-0.0926 0.05 0.0115"  rpy="0.0 0.0 ${167.5 * pi/180}" prefix="rl" />
+    <xacro:range_sensor.vl53lox parent="body_link" xyz="-0.0926 -0.05 0.0115" rpy="0.0 0.0 ${192.5 * pi/180}" prefix="rr" />
   </xacro:macro>
 </robot>

File: rosbot_description/urdf/components/vl53lox.urdf.xacro (robot description, xacro)
@@ -2,5 +2,5 @@
 <robot xmlns:xacro="http://www.ros.org/wiki/xacro">
   <!-- vl53lox defining macro -->
-  <xacro:macro name="vl53lox" params="xyz rpy prefix parent">
+  <xacro:macro name="vl53lox" params="parent xyz rpy prefix">
     <joint name="${parent}_${prefix}_range_joint" type="fixed">
         <origin xyz="${xyz}" rpy="${rpy}" />

Commit message: inertia update

File: rosbot_description/urdf/body.urdf.xacro (robot description, xacro)
@@ -2,5 +2,5 @@
 <robot xmlns:xacro="http://www.ros.org/wiki/xacro">
   <!-- body defining macro -->
-  <xacro:macro name="body" params="wheel_radius mecanum">
+  <xacro:macro name="body" params="wheel_radius mecanum use_gpu">
     <xacro:include filename="$(find rosbot_description)/urdf/components/vl53lox.urdf.xacro" ns="range_sensor" />
     <link name="base_link" />
@@ -28,5 +28,7 @@
       <inertial>
         <mass value="2.0" />
-        <inertia ixx="0.00721" ixy="0" ixz="0" iyy="0.01035" iyz="0" izz="0.01006" />
+        <inertia ixx="0.00721" ixy="0" ixz="0"
+                               iyy="0.01035" iyz="0"
+                                             izz="0.01006" />
       </inertial>
     </link>
@@ -65,8 +67,8 @@
     </joint>
     <link name="camera_link" />
-    <xacro:range_sensor.vl53lox parent="body_link" xyz="0.0926  0.05 0.015"   rpy="0.0 0.0 ${12.5/180.0*pi}" prefix="fl" />
-    <xacro:range_sensor.vl53lox parent="body_link" xyz="0.0926 -0.05 0.015"   rpy="0.0 0.0 ${-12.5/180.0*pi}" prefix="fr" />
-    <xacro:range_sensor.vl53lox parent="body_link" xyz="-0.0926 0.05 0.0115"  rpy="0.0 0.0 ${167.5/180.0*pi}" prefix="rl" />
-    <xacro:range_sensor.vl53lox parent="body_link" xyz="-0.0926 -0.05 0.0115" rpy="0.0 0.0 ${192.5/180.0*pi}" prefix="rr" />
+    <xacro:range_sensor.vl53lox parent="body_link" xyz="0.0926  0.05 0.015"   rpy="0.0 0.0 ${radians(12.5)}"  prefix="fl" use_gpu="${use_gpu}" />
+    <xacro:range_sensor.vl53lox parent="body_link" xyz="0.0926 -0.05 0.015"   rpy="0.0 0.0 ${radians(-12.5)}" prefix="fr" use_gpu="${use_gpu}" />
+    <xacro:range_sensor.vl53lox parent="body_link" xyz="-0.0926 0.05 0.0115"  rpy="0.0 0.0 ${radians(167.5)}" prefix="rl" use_gpu="${use_gpu}" />
+    <xacro:range_sensor.vl53lox parent="body_link" xyz="-0.0926 -0.05 0.0115" rpy="0.0 0.0 ${radians(192.5)}" prefix="rr" use_gpu="${use_gpu}" />
   </xacro:macro>
 </robot>

File: rosbot_description/urdf/components/vl53lox.urdf.xacro (robot description, xacro)
@@ -2,5 +2,5 @@
 <robot xmlns:xacro="http://www.ros.org/wiki/xacro">
   <!-- vl53lox defining macro -->
-  <xacro:macro name="vl53lox" params="parent xyz rpy prefix">
+  <xacro:macro name="vl53lox" params="parent xyz rpy prefix use_gpu">
     <joint name="${parent}_${prefix}_range_joint" type="fixed">
         <origin xyz="${xyz}" rpy="${rpy}" />
@@ -9,4 +9,47 @@
     </joint>
     <link name="${prefix}_range" />
+    <!-- <xacro:if value="${simulation_engine == 'ignition-gazebo'}">
+      <xacro:if value="${use_gpu}">
+        <xacro:property name="ray_type" value="gpu_lidar" />
+      </xacro:if>
+      <xacro:unless value="${use_gpu}">
+          <xacro:property name="ray_type" value="lidar" />
+      </xacro:unless>
+      <gazebo reference="${prefix}_range">
+        <sensor type="${ray_type}" name="${prefix}_range">
+          <topic>${prefix}_range</topic>
+          <frame_id>${prefix}_range</frame_id>
+          <ignition_frame_id>${prefix}_range</ignition_frame_id>
+          <update_rate>10.0</update_rate>
+          <ray>
+            <scan>
+              <horizontal>
+                <samples>1</samples>
+                <resolution>1</resolution>
+                <min_angle>-0.1</min_angle>
+                <max_angle>0.1</max_angle>
+              </horizontal>
+            </scan>
+            <range>
+              <min>0.01</min>
+              <max>0.9</max>
+              <resolution>1</resolution>
+            </range>
+            <noise>
+              <type>gaussian</type>
+              <mean>0.0</mean>
+              <stddev>0.001</stddev>
+            </noise>
+          </ray>
+          <always_on>1</always_on>
+          <visualize>true</visualize>
+        </sensor>
+      </gazebo>
+      <gazebo>
+        <plugin filename="libignition-gazebo-sensors-system.so" name="ignition::gazebo::systems::Sensors">
+          <render_engine>ogre2</render_engine>
+        </plugin>
+      </gazebo>
+    </xacro:if> -->
   </xacro:macro>
 </robot>

File: rosbot_description/urdf/rosbot.urdf.xacro (robot description, xacro)
@@ -6,5 +6,5 @@
   <xacro:arg name="simulation_engine" default="" />
   <xacro:include filename="$(find rosbot_description)/urdf/rosbot_macro.urdf.xacro" ns="husarion" />
-  <xacro:husarion.rosbot_robot mecanum="$(arg mecanum)" use_sim="$(arg use_sim)" simulation_engine="$(arg simulation_engine)"/>
+  <xacro:husarion.rosbot_robot mecanum="$(arg mecanum)" use_sim="$(arg use_sim)" use_gpu="$(arg use_gpu)" simulation_engine="$(arg simulation_engine)"/>
   <xacro:include filename="$(find ros_components_description)/urdf/slamtec_rplidar_a2.urdf.xacro" ns="lidar" />
   <xacro:lidar.slamtec_rplidar_a2

File: rosbot_description/urdf/rosbot_macro.urdf.xacro (robot description, xacro)
@@ -1,5 +1,5 @@
 <?xml version='1.0'?>
 <robot xmlns:xacro="http://wiki.ros.org/xacro">
-  <xacro:macro name="rosbot_robot" params="mecanum use_sim simulation_engine">
+  <xacro:macro name="rosbot_robot" params="mecanum use_sim use_gpu simulation_engine">
     <xacro:if value="${mecanum}">
       <xacro:property name="wheel_radius" value="0.0470" />
@@ -12,5 +12,5 @@
     <xacro:include filename="$(find rosbot_description)/urdf/wheel.urdf.xacro" ns="wheel" />
     <!-- BODY DECLARATION -->
-    <xacro:body.body wheel_radius="${wheel_radius}" mecanum="${mecanum}" />
+    <xacro:body.body wheel_radius="${wheel_radius}" mecanum="${mecanum}" use_gpu="${use_gpu}" />
     <!-- WHEEL DECLARATION -->
     <xacro:wheel.wheel wheel_radius="${wheel_radius}" prefix="fr" mecanum="${mecanum}" />
@@ -136,5 +136,5 @@
             <plugin name='skid_steer_drive' filename='libgazebo_ros_diff_drive.so'>
               <ros></ros>
-              <update_rate>10</update_rate>
+              <update_rate>10.0</update_rate>
               <num_wheel_pairs>2</num_wheel_pairs>
               <left_joint>fl_wheel_joint</left_joint>

File: rosbot_description/urdf/wheel.urdf.xacro (robot description, xacro)
@@ -9,6 +9,6 @@
       <xacro:property name="mass" value="0.153" />
       <xacro:property name="ixx" value="0.000111" />
-      <xacro:property name="iyy" value="0.000111" />
-      <xacro:property name="izz" value="0.000169" />
+      <xacro:property name="iyy" value="0.000169" />
+      <xacro:property name="izz" value="0.000111" />
       <xacro:property name="wheel_separation_y" value="0.205" />
     </xacro:if>
@@ -18,11 +18,11 @@
       <xacro:property name="mass" value="0.074" />
       <xacro:property name="ixx" value="0.000041" />
-      <xacro:property name="iyy" value="0.000041" />
-      <xacro:property name="izz" value="0.000067" />
+      <xacro:property name="iyy" value="0.000067" />
+      <xacro:property name="izz" value="0.000041" />
       <xacro:property name="wheel_separation_y" value="0.192" />
     </xacro:unless>
     <xacro:if value="${prefix == 'fl'}">
-      <xacro:property name="x" value="${wheel_separation_x/2}" />
-      <xacro:property name="y" value="${wheel_separation_y/2}" />
+      <xacro:property name="x" value="${wheel_separation_x/2.0}" />
+      <xacro:property name="y" value="${wheel_separation_y/2.0}" />
       <xacro:property name="mesh" value="file://$(find rosbot_description)/meshes/${wheel_file}_b.dae" />
       <xacro:property name="visual_rotation" value="${pi}" />
@@ -30,6 +30,6 @@
     </xacro:if>
     <xacro:if value="${prefix == 'fr'}">
-      <xacro:property name="x" value="${wheel_separation_x/2}" />
-      <xacro:property name="y" value="${-wheel_separation_y/2}" />
+      <xacro:property name="x" value="${wheel_separation_x/2.0}" />
+      <xacro:property name="y" value="${-wheel_separation_y/2.0}" />
       <xacro:property name="mesh" value="file://$(find rosbot_description)/meshes/${wheel_file}_a.dae" />
       <xacro:property name="visual_rotation" value="${pi}" />

Commit message: updated body inertia

File: rosbot_description/urdf/body.urdf.xacro (robot description, xacro)
@@ -27,8 +27,9 @@
       </collision>
       <inertial>
-        <mass value="2.0" />
-        <inertia ixx="0.00721" ixy="0" ixz="0"
-                               iyy="0.01035" iyz="0"
-                                             izz="0.01006" />
+        <mass value="1.728" />
+        <inertia ixx="0.004162" ixy="0.0"     ixz="0.0"
+                                iyy="0.00651" iyz="0.0"
+                                              izz="0.008828" />
+        <origin xyz="0.0 0.0 ${0.040-0.02}" rpy="0.0 0.0 0.0" />
       </inertial>
     </link>

Commit message: removed ignition distance sensors

File: rosbot_description/urdf/body.urdf.xacro (robot description, xacro)
@@ -24,5 +24,5 @@
           <box size="0.197 0.150 0.080" />
         </geometry>
-        <origin xyz="0.0 0.0 ${0.040-0.02}" rpy="0.0 0.0 0.0" />
+        <origin xyz="0.0 0.0 ${0.040 - 0.02}" rpy="0.0 0.0 0.0" />
       </collision>
       <inertial>
@@ -31,5 +31,5 @@
                                 iyy="0.00651" iyz="0.0"
                                               izz="0.008828" />
-        <origin xyz="0.0 0.0 ${0.040-0.02}" rpy="0.0 0.0 0.0" />
+        <origin xyz="0.0 0.0 ${0.040 - 0.02}" rpy="0.0 0.0 0.0" />
       </inertial>
     </link>

File: rosbot_description/urdf/components/vl53lox.urdf.xacro (robot description, xacro)
@@ -9,47 +9,4 @@
     </joint>
     <link name="${prefix}_range" />
-    <!-- <xacro:if value="${simulation_engine == 'ignition-gazebo'}">
-      <xacro:if value="${use_gpu}">
-        <xacro:property name="ray_type" value="gpu_lidar" />
-      </xacro:if>
-      <xacro:unless value="${use_gpu}">
-          <xacro:property name="ray_type" value="lidar" />
-      </xacro:unless>
-      <gazebo reference="${prefix}_range">
-        <sensor type="${ray_type}" name="${prefix}_range">
-          <topic>${prefix}_range</topic>
-          <frame_id>${prefix}_range</frame_id>
-          <ignition_frame_id>${prefix}_range</ignition_frame_id>
-          <update_rate>10.0</update_rate>
-          <ray>
-            <scan>
-              <horizontal>
-                <samples>1</samples>
-                <resolution>1</resolution>
-                <min_angle>-0.1</min_angle>
-                <max_angle>0.1</max_angle>
-              </horizontal>
-            </scan>
-            <range>
-              <min>0.01</min>
-              <max>0.9</max>
-              <resolution>1</resolution>
-            </range>
-            <noise>
-              <type>gaussian</type>
-              <mean>0.0</mean>
-              <stddev>0.001</stddev>
-            </noise>
-          </ray>
-          <always_on>1</always_on>
-          <visualize>true</visualize>
-        </sensor>
-      </gazebo>
-      <gazebo>
-        <plugin filename="libignition-gazebo-sensors-system.so" name="ignition::gazebo::systems::Sensors">
-          <render_engine>ogre2</render_engine>
-        </plugin>
-      </gazebo>
-    </xacro:if> -->
   </xacro:macro>
 </robot>

Commit message: removed unused GPU

File: rosbot_description/urdf/body.urdf.xacro (robot description, xacro)
@@ -68,8 +68,8 @@
     </joint>
     <link name="camera_link" />
-    <xacro:range_sensor.vl53lox parent="body_link" xyz="0.0926  0.05 0.015"   rpy="0.0 0.0 ${radians(12.5)}"  prefix="fl" use_gpu="${use_gpu}" />
-    <xacro:range_sensor.vl53lox parent="body_link" xyz="0.0926 -0.05 0.015"   rpy="0.0 0.0 ${radians(-12.5)}" prefix="fr" use_gpu="${use_gpu}" />
-    <xacro:range_sensor.vl53lox parent="body_link" xyz="-0.0926 0.05 0.0115"  rpy="0.0 0.0 ${radians(167.5)}" prefix="rl" use_gpu="${use_gpu}" />
-    <xacro:range_sensor.vl53lox parent="body_link" xyz="-0.0926 -0.05 0.0115" rpy="0.0 0.0 ${radians(192.5)}" prefix="rr" use_gpu="${use_gpu}" />
+    <xacro:range_sensor.vl53lox parent="body_link" xyz="0.0926  0.05 0.015"   rpy="0.0 0.0 ${radians(12.5)}"  prefix="fl" />
+    <xacro:range_sensor.vl53lox parent="body_link" xyz="0.0926 -0.05 0.015"   rpy="0.0 0.0 ${radians(-12.5)}" prefix="fr" />
+    <xacro:range_sensor.vl53lox parent="body_link" xyz="-0.0926 0.05 0.0115"  rpy="0.0 0.0 ${radians(167.5)}" prefix="rl" />
+    <xacro:range_sensor.vl53lox parent="body_link" xyz="-0.0926 -0.05 0.0115" rpy="0.0 0.0 ${radians(192.5)}" prefix="rr" />
   </xacro:macro>
 </robot>

File: rosbot_description/urdf/components/vl53lox.urdf.xacro (robot description, xacro)
@@ -2,5 +2,5 @@
 <robot xmlns:xacro="http://www.ros.org/wiki/xacro">
   <!-- vl53lox defining macro -->
-  <xacro:macro name="vl53lox" params="parent xyz rpy prefix use_gpu">
+  <xacro:macro name="vl53lox" params="parent xyz rpy prefix">
     <joint name="${parent}_${prefix}_range_joint" type="fixed">
         <origin xyz="${xyz}" rpy="${rpy}" />
