Commit message: Added namespace to robot description
Signed-off-by: Jakub Delicat <jakub.delicat@husarion.com>

File: rosbot_description/urdf/body.urdf.xacro (robot description, xacro)
@@ -2,13 +2,19 @@
 <robot xmlns:xacro="http://www.ros.org/wiki/xacro">
   <!-- body defining macro -->
-  <xacro:macro name="body" params="wheel_radius mecanum use_gpu">
+  <xacro:macro name="body" params="wheel_radius mecanum use_gpu tf_prefix">
     <xacro:include filename="$(find rosbot_description)/urdf/components/vl53lox.urdf.xacro" ns="range_sensor" />
-    <link name="base_link" />
-    <joint name="base_to_body_joint" type="fixed">
+    <xacro:if value="${tf_prefix == 'None'}">
+      <xacro:property name="tf_prefix_ext" value="" />
+    </xacro:if>
+    <xacro:unless value="${tf_prefix == 'None'}">
+      <xacro:property name="tf_prefix_ext" value="${tf_prefix}_" />
+    </xacro:unless>
+    <link name="${tf_prefix_ext}base_link" />
+    <joint name="${tf_prefix_ext}base_to_${tf_prefix_ext}body_joint" type="fixed">
       <origin xyz="0.0 0.0 ${wheel_radius}" rpy="0.0 0.0 0.0" />
-      <parent link="base_link" />
-      <child link="body_link" />
+      <parent link="${tf_prefix_ext}base_link" />
+      <child link="${tf_prefix_ext}body_link" />
     </joint>
-    <link name="body_link">
+    <link name="${tf_prefix_ext}body_link">
       <visual>
         <geometry>
@@ -34,13 +40,13 @@
       </inertial>
     </link>
-    <gazebo reference="body_link">
+    <gazebo reference="${tf_prefix_ext}body_link">
       <material>Gazebo/White</material>
     </gazebo>
-    <joint name="body_to_cover_joint" type="fixed">
+    <joint name="${tf_prefix_ext}body_to_${tf_prefix_ext}cover_joint" type="fixed">
       <origin xyz="0.0 0.0 0.0603" rpy="0.0 0.0 0.0" />
-      <parent link="body_link" />
-      <child link="cover_link" />
+      <parent link="${tf_prefix_ext}body_link" />
+      <child link="${tf_prefix_ext}cover_link" />
     </joint>
-    <link name="cover_link">
+    <link name="${tf_prefix_ext}cover_link">
       <visual>
         <geometry>
@@ -52,24 +58,24 @@
         </material>
       </visual>
-      <gazebo reference="cover_link">
+      <gazebo reference="${tf_prefix_ext}cover_link">
         <material>Gazebo/Red</material>
       </gazebo>
     </link>
-    <joint name="body_to_imu_joint" type="fixed">
+    <joint name="${tf_prefix_ext}body_to_${tf_prefix_ext}imu_joint" type="fixed">
       <origin xyz="0.003 -0.0495 0.04332" rpy="0.0 0.0 0.0" />
-      <parent link="body_link" />
-      <child link="imu_link" />
+      <parent link="${tf_prefix_ext}body_link" />
+      <child link="${tf_prefix_ext}imu_link" />
     </joint>
-    <link name="imu_link" />
-    <joint name="body_to_camera_joint" type="fixed">
+    <link name="${tf_prefix_ext}imu_link" />
+    <joint name="${tf_prefix_ext}body_to_${tf_prefix_ext}camera_joint" type="fixed">
       <origin xyz="-0.0141 0.0 0.125" rpy="0.0 0.0 0.0" />
-      <parent link="body_link" />
-      <child link="camera_link" />
+      <parent link="${tf_prefix_ext}body_link" />
+      <child link="${tf_prefix_ext}camera_link" />
     </joint>
-    <link name="camera_link" />
-    <xacro:range_sensor.vl53lox parent="body_link" xyz="0.0926  0.05 0.015"   rpy="0.0 0.0 ${radians(12.5)}"  prefix="fl" />
-    <xacro:range_sensor.vl53lox parent="body_link" xyz="0.0926 -0.05 0.015"   rpy="0.0 0.0 ${radians(-12.5)}" prefix="fr" />
-    <xacro:range_sensor.vl53lox parent="body_link" xyz="-0.0926 0.05 0.0115"  rpy="0.0 0.0 ${radians(167.5)}" prefix="rl" />
-    <xacro:range_sensor.vl53lox parent="body_link" xyz="-0.0926 -0.05 0.0115" rpy="0.0 0.0 ${radians(192.5)}" prefix="rr" />
+    <link name="${tf_prefix_ext}camera_link" />
+    <xacro:range_sensor.vl53lox parent="${tf_prefix_ext}body_link" xyz="0.0926  0.05 0.015"   rpy="0.0 0.0 ${radians(12.5)}"  side="fl" tf_prefix="${tf_prefix}" />
+    <xacro:range_sensor.vl53lox parent="${tf_prefix_ext}body_link" xyz="0.0926 -0.05 0.015"   rpy="0.0 0.0 ${radians(-12.5)}" side="fr" tf_prefix="${tf_prefix}" />
+    <xacro:range_sensor.vl53lox parent="${tf_prefix_ext}body_link" xyz="-0.0926 0.05 0.0115"  rpy="0.0 0.0 ${radians(167.5)}" side="rl" tf_prefix="${tf_prefix}" />
+    <xacro:range_sensor.vl53lox parent="${tf_prefix_ext}body_link" xyz="-0.0926 -0.05 0.0115" rpy="0.0 0.0 ${radians(192.5)}" side="rr" tf_prefix="${tf_prefix}" />
   </xacro:macro>
 </robot>

File: rosbot_description/urdf/components/vl53lox.urdf.xacro (robot description, xacro)
@@ -2,19 +2,25 @@
 <robot xmlns:xacro="http://www.ros.org/wiki/xacro">
   <!-- vl53lox defining macro -->
-  <xacro:macro name="vl53lox" params="parent xyz rpy prefix">
-    <joint name="${parent}_${prefix}_range_joint" type="fixed">
+  <xacro:macro name="vl53lox" params="parent xyz rpy side tf_prefix">
+    <xacro:if value="${tf_prefix == 'None'}">
+      <xacro:property name="tf_prefix_ext" value="" />
+    </xacro:if>
+    <xacro:unless value="${tf_prefix == 'None'}">
+      <xacro:property name="tf_prefix_ext" value="${tf_prefix}_" />
+    </xacro:unless>
+    <joint name="${parent.rstrip('_link')}_${tf_prefix_ext}${side}_range_joint" type="fixed">
       <origin xyz="${xyz}" rpy="${rpy}" />
       <parent link="${parent}" />
-      <child link="${prefix}_range" />
+      <child link="${tf_prefix_ext}${side}_range" />
     </joint>
-    <link name="${prefix}_range" />
+    <link name="${tf_prefix_ext}${side}_range" />
     <!-- an IR sensor or a sonar are not implemented yet
     https://github.com/gazebosim/gz-sensors/issues/19 -->
     <xacro:if value="${simulation_engine == 'ignition-gazebo'}">
-      <gazebo reference="${prefix}_range">
-        <sensor name="${prefix}_range" type='gpu_lidar'>
-          <topic>/range/${prefix}</topic>
-          <frame_id>${prefix}_range</frame_id>
-          <ignition_frame_id>${prefix}_range</ignition_frame_id>
+      <gazebo reference="${tf_prefix_ext}${side}_range">
+        <sensor name="${tf_prefix_ext}${side}_range" type='gpu_lidar'>
+          <topic>/range/${side}</topic>
+          <frame_id>${tf_prefix_ext}${side}_range</frame_id>
+          <ignition_frame_id>${tf_prefix_ext}${side}_range</ignition_frame_id>
           <update_rate>5.0</update_rate>
           <ray>

File: rosbot_description/urdf/rosbot.urdf.xacro (robot description, xacro)
@@ -5,18 +5,33 @@
   <xacro:arg name="mecanum" default="false" />
   <xacro:arg name="simulation_engine" default="" />
+  <xacro:arg name="tf_prefix" default="None" />
+  <xacro:property name="tf_prefix" value="$(arg tf_prefix)" />
+  <xacro:if value="${tf_prefix == 'None'}">
+    <xacro:property name="tf_prefix_ext" value="" />
+  </xacro:if>
+  <xacro:unless value="${ tf_prefix == 'None'}">
+    <xacro:property name="tf_prefix_ext" value="${tf_prefix}_" />
+  </xacro:unless>
   <xacro:include filename="$(find rosbot_description)/urdf/rosbot_macro.urdf.xacro" ns="husarion" />
-  <xacro:husarion.rosbot_robot mecanum="$(arg mecanum)" use_sim="$(arg use_sim)" use_gpu="$(arg use_gpu)" simulation_engine="$(arg simulation_engine)"/>
+  <xacro:husarion.rosbot_robot
+    mecanum="$(arg mecanum)"
+    use_sim="$(arg use_sim)"
+    use_gpu="$(arg use_gpu)"
+    simulation_engine="$(arg simulation_engine)"
+    tf_prefix="$(arg tf_prefix)" />
   <xacro:include filename="$(find ros_components_description)/urdf/slamtec_rplidar_a2.urdf.xacro" ns="lidar" />
   <xacro:lidar.slamtec_rplidar_a2
-    parent_link="cover_link"
+    parent_link="${tf_prefix_ext}cover_link"
     xyz="0.02 0.0 0.0"
     rpy="0.0 0.0 0.0"
     use_gpu="$(arg use_gpu)"
-    simulation_engine="$(arg simulation_engine)" />
+    simulation_engine="$(arg simulation_engine)"
+    tf_prefix="$(arg tf_prefix)" />
   <xacro:include filename="$(find ros_components_description)/urdf/orbbec_astra.urdf.xacro" ns="camera" />
   <xacro:camera.orbbec_astra
-    parent_link="camera_link"
+    parent_link="${tf_prefix_ext}camera_link"
     xyz="0.0 0.0 0.0"
     rpy="0.0 0.0 0.0"
-    simulation_engine="$(arg simulation_engine)" />
+    simulation_engine="$(arg simulation_engine)"
+    tf_prefix="$(arg tf_prefix)" />
 </robot>

File: rosbot_description/urdf/rosbot_macro.urdf.xacro (robot description, xacro)
@@ -1,5 +1,5 @@
 <?xml version='1.0'?>
 <robot xmlns:xacro="http://wiki.ros.org/xacro">
-  <xacro:macro name="rosbot_robot" params="mecanum use_sim use_gpu simulation_engine">
+  <xacro:macro name="rosbot_robot" params="mecanum use_sim use_gpu tf_prefix simulation_engine">
     <xacro:if value="${mecanum}">
       <xacro:property name="wheel_radius" value="0.0470" />
@@ -8,14 +8,20 @@
       <xacro:property name="wheel_radius" value="0.0425" />
     </xacro:unless>
+    <xacro:if value="${tf_prefix == 'None'}">
+      <xacro:property name="tf_prefix_ext" value="" />
+    </xacro:if>
+    <xacro:unless value="${tf_prefix == 'None'}">
+      <xacro:property name="tf_prefix_ext" value="${tf_prefix}_" />
+    </xacro:unless>
     <!-- INCLUDE ROBOT PARTS DEFINITIONS -->
     <xacro:include filename="$(find rosbot_description)/urdf/body.urdf.xacro" ns="body" />
     <xacro:include filename="$(find rosbot_description)/urdf/wheel.urdf.xacro" ns="wheel" />
     <!-- BODY DECLARATION -->
-    <xacro:body.body wheel_radius="${wheel_radius}" mecanum="${mecanum}" use_gpu="${use_gpu}" />
+    <xacro:body.body wheel_radius="${wheel_radius}" mecanum="${mecanum}" use_gpu="${use_gpu}" tf_prefix="${tf_prefix}" />
     <!-- WHEEL DECLARATION -->
-    <xacro:wheel.wheel wheel_radius="${wheel_radius}" prefix="fr" mecanum="${mecanum}" />
-    <xacro:wheel.wheel wheel_radius="${wheel_radius}" prefix="fl" mecanum="${mecanum}" />
-    <xacro:wheel.wheel wheel_radius="${wheel_radius}" prefix="rl" mecanum="${mecanum}" />
-    <xacro:wheel.wheel wheel_radius="${wheel_radius}" prefix="rr" mecanum="${mecanum}" />
+    <xacro:wheel.wheel wheel_radius="${wheel_radius}" side="fr" mecanum="${mecanum}" tf_prefix="${tf_prefix}" />
+    <xacro:wheel.wheel wheel_radius="${wheel_radius}" side="fl" mecanum="${mecanum}" tf_prefix="${tf_prefix}" />
+    <xacro:wheel.wheel wheel_radius="${wheel_radius}" side="rl" mecanum="${mecanum}" tf_prefix="${tf_prefix}" />
+    <xacro:wheel.wheel wheel_radius="${wheel_radius}" side="rr" mecanum="${mecanum}" tf_prefix="${tf_prefix}" />
     <!-- ROS2 CONTROL -->
     <xacro:unless value="$(arg use_sim)">
@@ -48,8 +54,8 @@
           <!-- order of velocity commands to be published in motors_cmd Float32MultiArray msg -->
           <param name="velocity_command_joint_order">
-                rr_wheel_joint,
-                rl_wheel_joint,
-                fr_wheel_joint,
-                fl_wheel_joint
+                ${tf_prefix_ext}rr_wheel_joint,
+                ${tf_prefix_ext}rl_wheel_joint,
+                ${tf_prefix_ext}fr_wheel_joint,
+                ${tf_prefix_ext}fl_wheel_joint
           </param>
         </xacro:unless>
@@ -63,20 +69,20 @@
         </xacro:if>
       </hardware>
-      <joint name="fl_wheel_joint">
-        <command_interface name="velocity" />
-        <state_interface name="position" />
-        <state_interface name="velocity" />
-      </joint>
-      <joint name="fr_wheel_joint">
-        <command_interface name="velocity" />
-        <state_interface name="position" />
-        <state_interface name="velocity" />
-      </joint>
-      <joint name="rl_wheel_joint">
-        <command_interface name="velocity" />
-        <state_interface name="position" />
-        <state_interface name="velocity" />
-      </joint>
-      <joint name="rr_wheel_joint">
+      <joint name="${tf_prefix_ext}fl_wheel_joint">
+        <command_interface name="velocity" />
+        <state_interface name="position" />
+        <state_interface name="velocity" />
+      </joint>
+      <joint name="${tf_prefix_ext}fr_wheel_joint">
+        <command_interface name="velocity" />
+        <state_interface name="position" />
+        <state_interface name="velocity" />
+      </joint>
+      <joint name="${tf_prefix_ext}rl_wheel_joint">
+        <command_interface name="velocity" />
+        <state_interface name="position" />
+        <state_interface name="velocity" />
+      </joint>
+      <joint name="${tf_prefix_ext}rr_wheel_joint">
         <command_interface name="velocity" />
         <state_interface name="position" />
@@ -117,5 +123,5 @@
           </plugin>
         </gazebo>
-        <gazebo reference="imu_link">
+        <gazebo reference="${tf_prefix_ext}imu_link">
           <sensor name="imu" type="imu">
             <plugin filename="ignition-gazebo-imu-system" name="ignition::gazebo::systems::Imu"></plugin>
@@ -125,6 +131,6 @@
             <visualize>false</visualize>
             <enable_metrics>false</enable_metrics>
-            <frame_id>imu_link</frame_id>
-            <ignition_frame_id>imu_link</ignition_frame_id>
+            <frame_id>${tf_prefix_ext}imu_link</frame_id>
+            <ignition_frame_id>${tf_prefix_ext}imu_link</ignition_frame_id>
           </sensor>
         </gazebo>
@@ -138,8 +144,8 @@
               <update_rate>10.0</update_rate>
               <num_wheel_pairs>2</num_wheel_pairs>
-              <left_joint>fl_wheel_joint</left_joint>
-              <right_joint>fr_wheel_joint</right_joint>
-              <left_joint>rl_wheel_joint</left_joint>
-              <right_joint>rr_wheel_joint</right_joint>
+              <left_joint>${tf_prefix_ext}fl_wheel_joint</left_joint>
+              <right_joint>${tf_prefix_ext}fr_wheel_joint</right_joint>
+              <left_joint>${tf_prefix_ext}rl_wheel_joint</left_joint>
+              <right_joint>${tf_prefix_ext}rr_wheel_joint</right_joint>
               <wheel_separation>0.192</wheel_separation>
               <wheel_separation>0.192</wheel_separation>
@@ -151,6 +157,6 @@
               <publish_odom_tf>true</publish_odom_tf>
               <publish_wheel_tf>true</publish_wheel_tf>
-              <odometry_frame>odom</odometry_frame>
-              <robot_base_frame>base_link</robot_base_frame>
+              <odometry_frame>${tf_prefix_ext}odom</odometry_frame>
+              <robot_base_frame>${tf_prefix_ext}base_link</robot_base_frame>
             </plugin>
           </gazebo>
@@ -159,12 +165,12 @@
         <gazebo>
           <plugin name="joint_states" filename="libgazebo_ros_joint_state_publisher.so">
-            <joint_name>fl_wheel_joint</joint_name>
-            <joint_name>fr_wheel_joint</joint_name>
-            <joint_name>rl_wheel_joint</joint_name>
-            <joint_name>rr_wheel_joint</joint_name>
+            <joint_name>${tf_prefix_ext}fl_wheel_joint</joint_name>
+            <joint_name>${tf_prefix_ext}fr_wheel_joint</joint_name>
+            <joint_name>${tf_prefix_ext}rl_wheel_joint</joint_name>
+            <joint_name>${tf_prefix_ext}rr_wheel_joint</joint_name>
           </plugin>
         </gazebo>
         <!-- publish IMU -->
-        <gazebo reference="imu_link">
+        <gazebo reference="${tf_prefix_ext}imu_link">
           <sensor type="imu" name="imu">
             <always_on>true</always_on>

File: rosbot_description/urdf/wheel.urdf.xacro (robot description, xacro)
@@ -2,5 +2,11 @@
 <robot xmlns:xacro="http://www.ros.org/wiki/xacro">
   <!-- wheel defining macro -->
-  <xacro:macro name="wheel" params="wheel_radius prefix mecanum">
+  <xacro:macro name="wheel" params="wheel_radius side mecanum tf_prefix">
+    <xacro:if value="${tf_prefix == 'None'}">
+      <xacro:property name="tf_prefix_ext" value="" />
+    </xacro:if>
+    <xacro:unless value="${tf_prefix == 'None'}">
+      <xacro:property name="tf_prefix_ext" value="${tf_prefix}_" />
+    </xacro:unless>
     <xacro:property name="wheel_separation_x" value="0.106" />
     <xacro:if value="${mecanum}">
@@ -22,5 +28,5 @@
       <xacro:property name="wheel_separation_y" value="0.192" />
     </xacro:unless>
-    <xacro:if value="${prefix == 'fl'}">
+    <xacro:if value="${side == 'fl'}">
       <xacro:property name="x" value="${wheel_separation_x/2.0}" />
       <xacro:property name="y" value="${wheel_separation_y/2.0}" />
@@ -29,5 +35,5 @@
       <xacro:property name="fdir" value="1.0 -1.0 0.0" />
     </xacro:if>
-    <xacro:if value="${prefix == 'fr'}">
+    <xacro:if value="${side == 'fr'}">
       <xacro:property name="x" value="${wheel_separation_x/2.0}" />
       <xacro:property name="y" value="${-wheel_separation_y/2.0}" />
@@ -36,5 +42,5 @@
       <xacro:property name="fdir" value="1.0 1.0 0.0" />
     </xacro:if>
-    <xacro:if value="${prefix == 'rl'}">
+    <xacro:if value="${side == 'rl'}">
       <xacro:property name="x" value="${-wheel_separation_x/2}" />
       <xacro:property name="y" value="${wheel_separation_y/2}" />
@@ -43,5 +49,5 @@
       <xacro:property name="fdir" value="1.0 1.0 0.0" />
     </xacro:if>
-    <xacro:if value="${prefix == 'rr'}">
+    <xacro:if value="${side == 'rr'}">
       <xacro:property name="x" value="${-wheel_separation_x/2}" />
       <xacro:property name="y" value="${-wheel_separation_y/2}" />
@@ -50,7 +56,7 @@
       <xacro:property name="fdir" value="1.0 -1.0 0.0" />
     </xacro:if>
-    <joint name="${prefix}_wheel_joint" type="continuous">
-      <parent link="body_link" />
-      <child link="${prefix}_wheel_link" />
+    <joint name="${tf_prefix_ext}${side}_wheel_joint" type="continuous">
+      <parent link="${tf_prefix_ext}body_link" />
+      <child link="${tf_prefix_ext}${side}_wheel_link" />
       <origin xyz="${x} ${y} 0.0" rpy="0.0 0.0 0.0" />
       <axis xyz="0.0 1.0 0.0" />
@@ -58,5 +64,5 @@
       <dynamics damping="0.001" friction="0.001" />
     </joint>
-    <link name="${prefix}_wheel_link">
+    <link name="${tf_prefix_ext}${side}_wheel_link">
       <visual>
         <geometry>
@@ -78,5 +84,5 @@
       </inertial>
     </link>
-    <gazebo reference="${prefix}_wheel_link" xmlns:ignition="http://ignitionrobotics.org/schema">
+    <gazebo reference="${tf_prefix_ext}${side}_wheel_link" xmlns:ignition="http://ignitionrobotics.org/schema">
       <collision>
         <surface>
@@ -85,5 +91,5 @@
               <mu>1.0</mu>
               <mu2>0.0</mu2>
-              <fdir1 ignition:expressed_in="base_link">${fdir}</fdir1>
+              <fdir1 ignition:expressed_in="${tf_prefix_ext}base_link">${fdir}</fdir1>
             </ode>
           </friction>
