Commit message: Simplify code and use robot_state_publisher for ns

File: rosbot_description/urdf/body.urdf.xacro (robot description, xacro)
@@ -4,17 +4,15 @@
   <xacro:macro name="body" params="wheel_radius mecanum use_gpu tf_prefix">
     <xacro:include filename="$(find rosbot_description)/urdf/components/vl53lox.urdf.xacro" ns="range_sensor" />
-    <xacro:if value="${tf_prefix == 'None'}">
-      <xacro:property name="tf_prefix_ext" value="" />
+    <xacro:property name="prefix" value="$(arg tf_prefix)" lazy_eval="false"/>
+    <xacro:if value="${prefix != ''}">
+      <xacro:property name="prefix" value="${prefix}_" />
     </xacro:if>
-    <xacro:unless value="${tf_prefix == 'None'}">
-      <xacro:property name="tf_prefix_ext" value="${tf_prefix}_" />
-    </xacro:unless>
-    <link name="${tf_prefix_ext}base_link" />
-    <joint name="${tf_prefix_ext}base_to_${tf_prefix_ext}body_joint" type="fixed">
+    <link name="${prefix}base_link" />
+    <joint name="${prefix}base_to_${prefix}body_joint" type="fixed">
       <origin xyz="0.0 0.0 ${wheel_radius}" rpy="0.0 0.0 0.0" />
-      <parent link="${tf_prefix_ext}base_link" />
-      <child link="${tf_prefix_ext}body_link" />
+      <parent link="${prefix}base_link" />
+      <child link="${prefix}body_link" />
     </joint>
-    <link name="${tf_prefix_ext}body_link">
+    <link name="${prefix}body_link">
       <visual>
         <geometry>
@@ -40,13 +38,13 @@
       </inertial>
     </link>
-    <gazebo reference="${tf_prefix_ext}body_link">
+    <gazebo reference="${prefix}body_link">
       <material>Gazebo/White</material>
     </gazebo>
-    <joint name="${tf_prefix_ext}body_to_${tf_prefix_ext}cover_joint" type="fixed">
+    <joint name="${prefix}body_to_${prefix}cover_joint" type="fixed">
       <origin xyz="0.0 0.0 0.0603" rpy="0.0 0.0 0.0" />
-      <parent link="${tf_prefix_ext}body_link" />
-      <child link="${tf_prefix_ext}cover_link" />
+      <parent link="${prefix}body_link" />
+      <child link="${prefix}cover_link" />
     </joint>
-    <link name="${tf_prefix_ext}cover_link">
+    <link name="${prefix}cover_link">
       <visual>
         <geometry>
@@ -58,24 +56,24 @@
         </material>
       </visual>
-      <gazebo reference="${tf_prefix_ext}cover_link">
+      <gazebo reference="${prefix}cover_link">
         <material>Gazebo/Red</material>
       </gazebo>
     </link>
-    <joint name="${tf_prefix_ext}body_to_${tf_prefix_ext}imu_joint" type="fixed">
+    <joint name="${prefix}body_to_${prefix}imu_joint" type="fixed">
       <origin xyz="0.003 -0.0495 0.04332" rpy="0.0 0.0 0.0" />
-      <parent link="${tf_prefix_ext}body_link" />
-      <child link="${tf_prefix_ext}imu_link" />
+      <parent link="${prefix}body_link" />
+      <child link="${prefix}imu_link" />
     </joint>
-    <link name="${tf_prefix_ext}imu_link" />
-    <joint name="${tf_prefix_ext}body_to_${tf_prefix_ext}camera_joint" type="fixed">
+    <link name="${prefix}imu_link" />
+    <joint name="${prefix}body_to_${prefix}camera_joint" type="fixed">
       <origin xyz="-0.0141 0.0 0.125" rpy="0.0 0.0 0.0" />
-      <parent link="${tf_prefix_ext}body_link" />
-      <child link="${tf_prefix_ext}camera_link" />
+      <parent link="${prefix}body_link" />
+      <child link="${prefix}camera_link" />
     </joint>
-    <link name="${tf_prefix_ext}camera_link" />
-    <xacro:range_sensor.vl53lox parent="${tf_prefix_ext}body_link" xyz="0.0926  0.05 0.015"   rpy="0.0 0.0 ${radians(12.5)}"  side="fl" tf_prefix="${tf_prefix}" />
-    <xacro:range_sensor.vl53lox parent="${tf_prefix_ext}body_link" xyz="0.0926 -0.05 0.015"   rpy="0.0 0.0 ${radians(-12.5)}" side="fr" tf_prefix="${tf_prefix}" />
-    <xacro:range_sensor.vl53lox parent="${tf_prefix_ext}body_link" xyz="-0.0926 0.05 0.0115"  rpy="0.0 0.0 ${radians(167.5)}" side="rl" tf_prefix="${tf_prefix}" />
-    <xacro:range_sensor.vl53lox parent="${tf_prefix_ext}body_link" xyz="-0.0926 -0.05 0.0115" rpy="0.0 0.0 ${radians(192.5)}" side="rr" tf_prefix="${tf_prefix}" />
+    <link name="${prefix}camera_link" />
+    <xacro:range_sensor.vl53lox parent="${prefix}body_link" xyz="0.0926  0.05 0.015"   rpy="0.0 0.0 ${radians(12.5)}"  side="fl" tf_prefix="${tf_prefix}" />
+    <xacro:range_sensor.vl53lox parent="${prefix}body_link" xyz="0.0926 -0.05 0.015"   rpy="0.0 0.0 ${radians(-12.5)}" side="fr" tf_prefix="${tf_prefix}" />
+    <xacro:range_sensor.vl53lox parent="${prefix}body_link" xyz="-0.0926 0.05 0.0115"  rpy="0.0 0.0 ${radians(167.5)}" side="rl" tf_prefix="${tf_prefix}" />
+    <xacro:range_sensor.vl53lox parent="${prefix}body_link" xyz="-0.0926 -0.05 0.0115" rpy="0.0 0.0 ${radians(192.5)}" side="rr" tf_prefix="${tf_prefix}" />
   </xacro:macro>
 </robot>

File: rosbot_description/urdf/components/vl53lox.urdf.xacro (robot description, xacro)
@@ -3,24 +3,22 @@
   <!-- vl53lox defining macro -->
   <xacro:macro name="vl53lox" params="parent xyz rpy side tf_prefix">
-    <xacro:if value="${tf_prefix == 'None'}">
-      <xacro:property name="tf_prefix_ext" value="" />
-    </xacro:if>
-    <xacro:unless value="${tf_prefix == 'None'}">
-      <xacro:property name="tf_prefix_ext" value="${tf_prefix}_" />
-    </xacro:unless>
-    <joint name="${parent.rstrip('_link')}_${tf_prefix_ext}${side}_range_joint" type="fixed">
+  <xacro:property name="prefix" value="${tf_prefix}" lazy_eval="false" />
+  <xacro:if value="${prefix != ''}">
+    <xacro:property name="prefix" value="${tf_prefix}_" />
+  </xacro:if>
+    <joint name="${parent.rstrip('_link')}_${prefix}${side}_range_joint" type="fixed">
       <origin xyz="${xyz}" rpy="${rpy}" />
       <parent link="${parent}" />
-      <child link="${tf_prefix_ext}${side}_range" />
+      <child link="${prefix}${side}_range" />
     </joint>
-    <link name="${tf_prefix_ext}${side}_range" />
+    <link name="${prefix}${side}_range" />
     <!-- an IR sensor or a sonar are not implemented yet
     https://github.com/gazebosim/gz-sensors/issues/19 -->
     <xacro:if value="${simulation_engine == 'ignition-gazebo'}">
-      <gazebo reference="${tf_prefix_ext}${side}_range">
-        <sensor name="${tf_prefix_ext}${side}_range" type='gpu_lidar'>
+      <gazebo reference="${prefix}${side}_range">
+        <sensor name="${prefix}${side}_range" type='gpu_lidar'>
           <topic>/range/${side}</topic>
-          <frame_id>${tf_prefix_ext}${side}_range</frame_id>
-          <ignition_frame_id>${tf_prefix_ext}${side}_range</ignition_frame_id>
+          <frame_id>${prefix}${side}_range</frame_id>
+          <ignition_frame_id>${prefix}${side}_range</ignition_frame_id>
           <update_rate>5.0</update_rate>
           <ray>

File: rosbot_description/urdf/rosbot.urdf.xacro (robot description, xacro)
@@ -1,16 +1,15 @@
 <?xml version='1.0'?>
 <robot name="rosbot" xmlns:xacro="http://www.ros.org/wiki/xacro">
+  <!-- Default arguments -->
   <xacro:arg name="use_sim" default="false" />
   <xacro:arg name="use_gpu" default="false" />
   <xacro:arg name="mecanum" default="false" />
   <xacro:arg name="simulation_engine" default="" />
-  <xacro:arg name="tf_prefix" default="None" />
-  <xacro:property name="tf_prefix" value="$(arg tf_prefix)" />
-  <xacro:if value="${tf_prefix == 'None'}">
-    <xacro:property name="tf_prefix_ext" value="" />
+  <xacro:arg name="tf_prefix" default="" />
+  <xacro:property name="prefix" value="$(arg tf_prefix)" lazy_eval="false"/>
+  <xacro:if value="${prefix != ''}">
+    <xacro:property name="prefix" value="${prefix}_" />
   </xacro:if>
-  <xacro:unless value="${ tf_prefix == 'None'}">
-    <xacro:property name="tf_prefix_ext" value="${tf_prefix}_" />
-  </xacro:unless>
+  <!-- Include rosbot_macro.urdf.xacro -->
   <xacro:include filename="$(find rosbot_description)/urdf/rosbot_macro.urdf.xacro" ns="husarion" />
   <xacro:husarion.rosbot_robot
@@ -20,7 +19,8 @@
     simulation_engine="$(arg simulation_engine)"
     tf_prefix="$(arg tf_prefix)" />
+  <!-- Include slamtec_rplidar_a2.urdf.xacro -->
   <xacro:include filename="$(find ros_components_description)/urdf/slamtec_rplidar_a2.urdf.xacro" ns="lidar" />
   <xacro:lidar.slamtec_rplidar_a2
-    parent_link="${tf_prefix_ext}cover_link"
+    parent_link="${prefix}cover_link"
     xyz="0.02 0.0 0.0"
     rpy="0.0 0.0 0.0"
@@ -28,7 +28,8 @@
     simulation_engine="$(arg simulation_engine)"
     tf_prefix="$(arg tf_prefix)" />
+  <!-- Include orbbec_astra.urdf.xacro -->
   <xacro:include filename="$(find ros_components_description)/urdf/orbbec_astra.urdf.xacro" ns="camera" />
   <xacro:camera.orbbec_astra
-    parent_link="${tf_prefix_ext}camera_link"
+    parent_link="${prefix}camera_link"
     xyz="0.0 0.0 0.0"
     rpy="0.0 0.0 0.0"

File: rosbot_description/urdf/rosbot_macro.urdf.xacro (robot description, xacro)
@@ -8,10 +8,8 @@
       <xacro:property name="wheel_radius" value="0.0425" />
     </xacro:unless>
-    <xacro:if value="${tf_prefix == 'None'}">
-      <xacro:property name="tf_prefix_ext" value="" />
+    <xacro:property name="prefix" value="$(arg tf_prefix)" lazy_eval="false"/>
+    <xacro:if value="${prefix != ''}">
+      <xacro:property name="prefix" value="${prefix}_" />
     </xacro:if>
-    <xacro:unless value="${tf_prefix == 'None'}">
-      <xacro:property name="tf_prefix_ext" value="${tf_prefix}_" />
-    </xacro:unless>
     <!-- INCLUDE ROBOT PARTS DEFINITIONS -->
     <xacro:include filename="$(find rosbot_description)/urdf/body.urdf.xacro" ns="body" />
@@ -61,5 +59,5 @@
                 fl_wheel_joint
           </param>
-          <param name="tf_prefix">${tf_prefix_ext}</param>
+          <param name="tf_prefix">${prefix}</param>
         </xacro:unless>
         <xacro:if value="$(arg use_sim)">
@@ -72,20 +70,20 @@
         </xacro:if>
       </hardware>
-      <joint name="${tf_prefix_ext}fl_wheel_joint">
-        <command_interface name="velocity" />
-        <state_interface name="position" />
-        <state_interface name="velocity" />
-      </joint>
-      <joint name="${tf_prefix_ext}fr_wheel_joint">
-        <command_interface name="velocity" />
-        <state_interface name="position" />
-        <state_interface name="velocity" />
-      </joint>
-      <joint name="${tf_prefix_ext}rl_wheel_joint">
-        <command_interface name="velocity" />
-        <state_interface name="position" />
-        <state_interface name="velocity" />
-      </joint>
-      <joint name="${tf_prefix_ext}rr_wheel_joint">
+      <joint name="${prefix}fl_wheel_joint">
+        <command_interface name="velocity" />
+        <state_interface name="position" />
+        <state_interface name="velocity" />
+      </joint>
+      <joint name="${prefix}fr_wheel_joint">
+        <command_interface name="velocity" />
+        <state_interface name="position" />
+        <state_interface name="velocity" />
+      </joint>
+      <joint name="${prefix}rl_wheel_joint">
+        <command_interface name="velocity" />
+        <state_interface name="position" />
+        <state_interface name="velocity" />
+      </joint>
+      <joint name="${prefix}rr_wheel_joint">
         <command_interface name="velocity" />
         <state_interface name="position" />
@@ -126,5 +124,5 @@
           </plugin>
         </gazebo>
-        <gazebo reference="${tf_prefix_ext}imu_link">
+        <gazebo reference="${prefix}imu_link">
           <sensor name="imu" type="imu">
             <plugin filename="ignition-gazebo-imu-system" name="ignition::gazebo::systems::Imu"></plugin>
@@ -134,6 +132,6 @@
             <visualize>false</visualize>
             <enable_metrics>false</enable_metrics>
-            <frame_id>${tf_prefix_ext}imu_link</frame_id>
-            <ignition_frame_id>${tf_prefix_ext}imu_link</ignition_frame_id>
+            <frame_id>${prefix}imu_link</frame_id>
+            <ignition_frame_id>${prefix}imu_link</ignition_frame_id>
           </sensor>
         </gazebo>
@@ -147,8 +145,8 @@
               <update_rate>10.0</update_rate>
               <num_wheel_pairs>2</num_wheel_pairs>
-              <left_joint>${tf_prefix_ext}fl_wheel_joint</left_joint>
-              <right_joint>${tf_prefix_ext}fr_wheel_joint</right_joint>
-              <left_joint>${tf_prefix_ext}rl_wheel_joint</left_joint>
-              <right_joint>${tf_prefix_ext}rr_wheel_joint</right_joint>
+              <left_joint>${prefix}fl_wheel_joint</left_joint>
+              <right_joint>${prefix}fr_wheel_joint</right_joint>
+              <left_joint>${prefix}rl_wheel_joint</left_joint>
+              <right_joint>${prefix}rr_wheel_joint</right_joint>
               <wheel_separation>0.192</wheel_separation>
               <wheel_separation>0.192</wheel_separation>
@@ -160,6 +158,6 @@
               <publish_odom_tf>true</publish_odom_tf>
               <publish_wheel_tf>true</publish_wheel_tf>
-              <odometry_frame>${tf_prefix_ext}odom</odometry_frame>
-              <robot_base_frame>${tf_prefix_ext}base_link</robot_base_frame>
+              <odometry_frame>${prefix}odom</odometry_frame>
+              <robot_base_frame>${prefix}base_link</robot_base_frame>
             </plugin>
           </gazebo>
@@ -168,12 +166,12 @@
         <gazebo>
           <plugin name="joint_states" filename="libgazebo_ros_joint_state_publisher.so">
-            <joint_name>${tf_prefix_ext}fl_wheel_joint</joint_name>
-            <joint_name>${tf_prefix_ext}fr_wheel_joint</joint_name>
-            <joint_name>${tf_prefix_ext}rl_wheel_joint</joint_name>
-            <joint_name>${tf_prefix_ext}rr_wheel_joint</joint_name>
+            <joint_name>${prefix}fl_wheel_joint</joint_name>
+            <joint_name>${prefix}fr_wheel_joint</joint_name>
+            <joint_name>${prefix}rl_wheel_joint</joint_name>
+            <joint_name>${prefix}rr_wheel_joint</joint_name>
           </plugin>
         </gazebo>
         <!-- publish IMU -->
-        <gazebo reference="${tf_prefix_ext}imu_link">
+        <gazebo reference="${prefix}imu_link">
           <sensor type="imu" name="imu">
             <always_on>true</always_on>

File: rosbot_description/urdf/wheel.urdf.xacro (robot description, xacro)
@@ -3,10 +3,8 @@
   <!-- wheel defining macro -->
   <xacro:macro name="wheel" params="wheel_radius side mecanum tf_prefix">
-    <xacro:if value="${tf_prefix == 'None'}">
-      <xacro:property name="tf_prefix_ext" value="" />
-    </xacro:if>
-    <xacro:unless value="${tf_prefix == 'None'}">
-      <xacro:property name="tf_prefix_ext" value="${tf_prefix}_" />
-    </xacro:unless>
+  <xacro:property name="prefix" value="${tf_prefix}" lazy_eval="false" />
+  <xacro:if value="${prefix != ''}">
+    <xacro:property name="prefix" value="${tf_prefix}_" />
+  </xacro:if>
     <xacro:property name="wheel_separation_x" value="0.106" />
     <xacro:if value="${mecanum}">
@@ -56,7 +54,7 @@
       <xacro:property name="fdir" value="1.0 -1.0 0.0" />
     </xacro:if>
-    <joint name="${tf_prefix_ext}${side}_wheel_joint" type="continuous">
-      <parent link="${tf_prefix_ext}body_link" />
-      <child link="${tf_prefix_ext}${side}_wheel_link" />
+    <joint name="${prefix}${side}_wheel_joint" type="continuous">
+      <parent link="${prefix}body_link" />
+      <child link="${prefix}${side}_wheel_link" />
       <origin xyz="${x} ${y} 0.0" rpy="0.0 0.0 0.0" />
       <axis xyz="0.0 1.0 0.0" />
@@ -64,5 +62,5 @@
       <dynamics damping="0.001" friction="0.001" />
     </joint>
-    <link name="${tf_prefix_ext}${side}_wheel_link">
+    <link name="${prefix}${side}_wheel_link">
       <visual>
         <geometry>
@@ -84,5 +82,5 @@
       </inertial>
     </link>
-    <gazebo reference="${tf_prefix_ext}${side}_wheel_link" xmlns:ignition="http://ignitionrobotics.org/schema">
+    <gazebo reference="${prefix}${side}_wheel_link" xmlns:ignition="http://ignitionrobotics.org/schema">
       <collision>
         <surface>
@@ -91,5 +89,5 @@
               <mu>1.0</mu>
               <mu2>0.0</mu2>
-              <fdir1 ignition:expressed_in="${tf_prefix_ext}base_link">${fdir}</fdir1>
+              <fdir1 ignition:expressed_in="${prefix}base_link">${fdir}</fdir1>
             </ode>
           </friction>

Commit message: Fix

File: rosbot_description/urdf/body.urdf.xacro (robot description, xacro)
@@ -4,7 +4,7 @@
   <xacro:macro name="body" params="wheel_radius mecanum use_gpu tf_prefix">
     <xacro:include filename="$(find rosbot_description)/urdf/components/vl53lox.urdf.xacro" ns="range_sensor" />
-    <xacro:property name="prefix" value="$(arg tf_prefix)" lazy_eval="false"/>
+    <xacro:property name="prefix" value="${tf_prefix}" lazy_eval="false"/>
     <xacro:if value="${prefix != ''}">
-      <xacro:property name="prefix" value="${prefix}_" />
+      <xacro:property name="prefix" value="${tf_prefix}_" />
     </xacro:if>
     <link name="${prefix}base_link" />

File: rosbot_description/urdf/rosbot.urdf.xacro (robot description, xacro)
@@ -9,5 +9,5 @@
   <xacro:property name="prefix" value="$(arg tf_prefix)" lazy_eval="false"/>
   <xacro:if value="${prefix != ''}">
-    <xacro:property name="prefix" value="${prefix}_" />
+    <xacro:property name="prefix" value="$(arg tf_prefix)_" />
   </xacro:if>
   <!-- Include rosbot_macro.urdf.xacro -->

File: rosbot_description/urdf/rosbot_macro.urdf.xacro (robot description, xacro)
@@ -8,7 +8,7 @@
       <xacro:property name="wheel_radius" value="0.0425" />
     </xacro:unless>
-    <xacro:property name="prefix" value="$(arg tf_prefix)" lazy_eval="false"/>
+    <xacro:property name="prefix" value="${tf_prefix}" lazy_eval="false"/>
     <xacro:if value="${prefix != ''}">
-      <xacro:property name="prefix" value="${prefix}_" />
+      <xacro:property name="prefix" value="${tf_prefix}_" />
     </xacro:if>
     <!-- INCLUDE ROBOT PARTS DEFINITIONS -->

Commit message: Use package:// instead of file://

File: rosbot_description/urdf/body.urdf.xacro (robot description, xacro)
@@ -13,5 +13,5 @@
       <visual>
         <geometry>
-          <mesh filename="file://$(find rosbot_description)/meshes/body.stl" scale="0.001 0.001 0.001" />
+          <mesh filename="package://rosbot_description/meshes/body.stl" scale="0.001 0.001 0.001" />
         </geometry>
         <origin xyz="0.0 0.0 -0.0173" rpy="${pi/2} 0.0 ${pi/2}" />
@@ -45,5 +45,5 @@
       <visual>
         <geometry>
-          <mesh filename="file://$(find rosbot_description)/meshes/cover.stl" scale="0.001 0.001 0.001" />
+          <mesh filename="package://rosbot_description/meshes/cover.stl" scale="0.001 0.001 0.001" />
         </geometry>
         <origin xyz="0.0 0.0 -0.002" rpy="${pi/2} 0.0 ${pi/2}" />

File: rosbot_description/urdf/wheel.urdf.xacro (robot description, xacro)
@@ -25,5 +25,5 @@
       <xacro:property name="x" value="${wheel_separation_x/2.0}" />
       <xacro:property name="y" value="${wheel_separation_y/2.0}" />
-      <xacro:property name="mesh" value="file://$(find rosbot_description)/meshes/${wheel_file}_b.dae" />
+      <xacro:property name="mesh" value="package://rosbot_description/meshes/${wheel_file}_b.dae" />
       <xacro:property name="visual_rotation" value="${pi}" />
       <xacro:property name="fdir" value="1.0 -1.0 0.0" />
@@ -32,5 +32,5 @@
       <xacro:property name="x" value="${wheel_separation_x/2.0}" />
       <xacro:property name="y" value="${-wheel_separation_y/2.0}" />
-      <xacro:property name="mesh" value="file://$(find rosbot_description)/meshes/${wheel_file}_a.dae" />
+      <xacro:property name="mesh" value="package://rosbot_description/meshes/${wheel_file}_a.dae" />
       <xacro:property name="visual_rotation" value="${pi}" />
       <xacro:property name="fdir" value="1.0 1.0 0.0" />
@@ -39,5 +39,5 @@
       <xacro:property name="x" value="${-wheel_separation_x/2}" />
       <xacro:property name="y" value="${wheel_separation_y/2}" />
-      <xacro:property name="mesh" value="file://$(find rosbot_description)/meshes/${wheel_file}_a.dae" />
+      <xacro:property name="mesh" value="package://rosbot_description/meshes/${wheel_file}_a.dae" />
       <xacro:property name="visual_rotation" value="${0.0}" />
       <xacro:property name="fdir" value="1.0 1.0 0.0" />
@@ -46,5 +46,5 @@
       <xacro:property name="x" value="${-wheel_separation_x/2}" />
       <xacro:property name="y" value="${-wheel_separation_y/2}" />
-      <xacro:property name="mesh" value="file://$(find rosbot_description)/meshes/${wheel_file}_b.dae" />
+      <xacro:property name="mesh" value="package://rosbot_description/meshes/${wheel_file}_b.dae" />
       <xacro:property name="visual_rotation" value="${0.0}" />
       <xacro:property name="fdir" value="1.0 -1.0 0.0" />
