Commit message: Revert to None

File: rosbot_description/urdf/body.urdf.xacro (robot description, xacro)
@@ -4,8 +4,10 @@
   <xacro:macro name="body" params="wheel_radius mecanum use_gpu tf_prefix">
     <xacro:include filename="$(find rosbot_description)/urdf/components/vl53lox.urdf.xacro" ns="range_sensor" />
-    <xacro:property name="prefix" value="${tf_prefix}" lazy_eval="false"/>
-    <xacro:if value="${prefix != ''}">
+    <xacro:if value="${tf_prefix == 'None'}">
+      <xacro:property name="prefix" value="" />
+    </xacro:if>
+    <xacro:unless value="${tf_prefix == 'None'}">
       <xacro:property name="prefix" value="${tf_prefix}_" />
-    </xacro:if>
+    </xacro:unless>
     <link name="${prefix}base_link" />
     <joint name="${prefix}base_to_${prefix}body_joint" type="fixed">

File: rosbot_description/urdf/components/vl53lox.urdf.xacro (robot description, xacro)
@@ -3,8 +3,10 @@
   <!-- vl53lox defining macro -->
   <xacro:macro name="vl53lox" params="parent xyz rpy side tf_prefix">
-  <xacro:property name="prefix" value="${tf_prefix}" lazy_eval="false" />
-  <xacro:if value="${prefix != ''}">
-    <xacro:property name="prefix" value="${tf_prefix}_" />
-  </xacro:if>
+    <xacro:if value="${tf_prefix == 'None'}">
+      <xacro:property name="prefix" value="" />
+    </xacro:if>
+    <xacro:unless value="${tf_prefix == 'None'}">
+      <xacro:property name="prefix" value="${tf_prefix}_" />
+    </xacro:unless>
     <joint name="${parent.rstrip('_link')}_${prefix}${side}_range_joint" type="fixed">
       <origin xyz="${xyz}" rpy="${rpy}" />

File: rosbot_description/urdf/rosbot_macro.urdf.xacro (robot description, xacro)
@@ -12,8 +12,10 @@
       <xacro:property name="namespace" value="$(arg namespace)/" />
     </xacro:if>
-    <xacro:property name="prefix" value="${tf_prefix}" lazy_eval="false"/>
-    <xacro:if value="${prefix != ''}">
+    <xacro:if value="${tf_prefix == 'None'}">
+      <xacro:property name="prefix" value="" />
+    </xacro:if>
+    <xacro:unless value="${tf_prefix == 'None'}">
       <xacro:property name="prefix" value="${tf_prefix}_" />
-    </xacro:if>
+    </xacro:unless>
     <!-- INCLUDE ROBOT PARTS DEFINITIONS -->
     <xacro:include filename="$(find rosbot_description)/urdf/body.urdf.xacro" ns="body" />

File: rosbot_description/urdf/wheel.urdf.xacro (robot description, xacro)
@@ -3,8 +3,10 @@
   <!-- wheel defining macro -->
   <xacro:macro name="wheel" params="wheel_radius side mecanum tf_prefix">
-  <xacro:property name="prefix" value="${tf_prefix}" lazy_eval="false" />
-  <xacro:if value="${prefix != ''}">
-    <xacro:property name="prefix" value="${tf_prefix}_" />
-  </xacro:if>
+    <xacro:if value="${tf_prefix == 'None'}">
+      <xacro:property name="prefix" value="" />
+    </xacro:if>
+    <xacro:unless value="${tf_prefix == 'None'}">
+      <xacro:property name="prefix" value="${tf_prefix}_" />
+    </xacro:unless>
     <xacro:property name="wheel_separation_x" value="0.106" />
     <xacro:if value="${mecanum}">
