Commit message: Multi robot diff drive example
Signed-off-by: Jakub Delicat <jakub.delicat@husarion.com>

File: rosbot_description/urdf/body.urdf.xacro (robot description, xacro)
@@ -2,22 +2,16 @@
 <robot xmlns:xacro="http://www.ros.org/wiki/xacro">
   <!-- body defining macro -->
-  <xacro:macro name="body" params="wheel_radius mecanum use_gpu tf_prefix">
+  <xacro:macro name="body" params="wheel_radius mecanum use_gpu">
     <xacro:include filename="$(find rosbot_description)/urdf/components/vl53lox.urdf.xacro" ns="range_sensor" />
-    <xacro:if value="${tf_prefix == 'None'}">
-      <xacro:property name="tf_prefix_ext" value="" />
-    </xacro:if>
-    <xacro:unless value="${tf_prefix == 'None'}">
-      <xacro:property name="tf_prefix_ext" value="${tf_prefix}_" />
-    </xacro:unless>
-    <link name="${tf_prefix_ext}base_link" />
-    <joint name="${tf_prefix_ext}base_to_${tf_prefix_ext}body_joint" type="fixed">
+    <link name="base_link" />
+    <joint name="base_to_body_joint" type="fixed">
       <origin xyz="0.0 0.0 ${wheel_radius}" rpy="0.0 0.0 0.0" />
-      <parent link="${tf_prefix_ext}base_link" />
-      <child link="${tf_prefix_ext}body_link" />
+      <parent link="base_link" />
+      <child link="body_link" />
     </joint>
-    <link name="${tf_prefix_ext}body_link">
+    <link name="body_link">
       <visual>
         <geometry>
-          <mesh filename="file://$(find rosbot_description)/meshes/body.stl" scale="0.001 0.001 0.001" />
+          <mesh filename="package://rosbot_description/meshes/body.stl" scale="0.001 0.001 0.001" />
         </geometry>
         <origin xyz="0.0 0.0 -0.0173" rpy="${pi/2} 0.0 ${pi/2}" />
@@ -40,16 +34,16 @@
       </inertial>
     </link>
-    <gazebo reference="${tf_prefix_ext}body_link">
+    <gazebo reference="body_link">
       <material>Gazebo/White</material>
     </gazebo>
-    <joint name="${tf_prefix_ext}body_to_${tf_prefix_ext}cover_joint" type="fixed">
+    <joint name="body_to_cover_joint" type="fixed">
       <origin xyz="0.0 0.0 0.0603" rpy="0.0 0.0 0.0" />
-      <parent link="${tf_prefix_ext}body_link" />
-      <child link="${tf_prefix_ext}cover_link" />
+      <parent link="body_link" />
+      <child link="cover_link" />
     </joint>
-    <link name="${tf_prefix_ext}cover_link">
+    <link name="cover_link">
       <visual>
         <geometry>
-          <mesh filename="file://$(find rosbot_description)/meshes/cover.stl" scale="0.001 0.001 0.001" />
+          <mesh filename="package://rosbot_description/meshes/cover.stl" scale="0.001 0.001 0.001" />
         </geometry>
         <origin xyz="0.0 0.0 -0.002" rpy="${pi/2} 0.0 ${pi/2}" />
@@ -58,24 +52,24 @@
         </material>
       </visual>
-      <gazebo reference="${tf_prefix_ext}cover_link">
+      <gazebo reference="cover_link">
         <material>Gazebo/Red</material>
       </gazebo>
     </link>
-    <joint name="${tf_prefix_ext}body_to_${tf_prefix_ext}imu_joint" type="fixed">
+    <joint name="body_to_imu_joint" type="fixed">
       <origin xyz="0.003 -0.0495 0.04332" rpy="0.0 0.0 0.0" />
-      <parent link="${tf_prefix_ext}body_link" />
-      <child link="${tf_prefix_ext}imu_link" />
+      <parent link="body_link" />
+      <child link="imu_link" />
     </joint>
-    <link name="${tf_prefix_ext}imu_link" />
-    <joint name="${tf_prefix_ext}body_to_${tf_prefix_ext}camera_joint" type="fixed">
+    <link name="imu_link" />
+    <joint name="body_to_camera_joint" type="fixed">
       <origin xyz="-0.0141 0.0 0.125" rpy="0.0 0.0 0.0" />
-      <parent link="${tf_prefix_ext}body_link" />
-      <child link="${tf_prefix_ext}camera_link" />
+      <parent link="body_link" />
+      <child link="camera_link" />
     </joint>
-    <link name="${tf_prefix_ext}camera_link" />
-    <xacro:range_sensor.vl53lox parent="${tf_prefix_ext}body_link" xyz="0.0926  0.05 0.015"   rpy="0.0 0.0 ${radians(12.5)}"  side="fl" tf_prefix="${tf_prefix}" />
-    <xacro:range_sensor.vl53lox parent="${tf_prefix_ext}body_link" xyz="0.0926 -0.05 0.015"   rpy="0.0 0.0 ${radians(-12.5)}" side="fr" tf_prefix="${tf_prefix}" />
-    <xacro:range_sensor.vl53lox parent="${tf_prefix_ext}body_link" xyz="-0.0926 0.05 0.0115"  rpy="0.0 0.0 ${radians(167.5)}" side="rl" tf_prefix="${tf_prefix}" />
-    <xacro:range_sensor.vl53lox parent="${tf_prefix_ext}body_link" xyz="-0.0926 -0.05 0.0115" rpy="0.0 0.0 ${radians(192.5)}" side="rr" tf_prefix="${tf_prefix}" />
+    <link name="camera_link" />
+    <xacro:range_sensor.vl53lox parent="body_link" xyz="0.0926  0.05 0.015"   rpy="0.0 0.0 ${radians(12.5)}"  prefix="fl" />
+    <xacro:range_sensor.vl53lox parent="body_link" xyz="0.0926 -0.05 0.015"   rpy="0.0 0.0 ${radians(-12.5)}" prefix="fr" />
+    <xacro:range_sensor.vl53lox parent="body_link" xyz="-0.0926 0.05 0.0115"  rpy="0.0 0.0 ${radians(167.5)}" prefix="rl" />
+    <xacro:range_sensor.vl53lox parent="body_link" xyz="-0.0926 -0.05 0.0115" rpy="0.0 0.0 ${radians(192.5)}" prefix="rr" />
   </xacro:macro>
 </robot>

File: rosbot_description/urdf/components/vl53lox.urdf.xacro (robot description, xacro)
@@ -2,25 +2,19 @@
 <robot xmlns:xacro="http://www.ros.org/wiki/xacro">
   <!-- vl53lox defining macro -->
-  <xacro:macro name="vl53lox" params="parent xyz rpy side tf_prefix">
-    <xacro:if value="${tf_prefix == 'None'}">
-      <xacro:property name="tf_prefix_ext" value="" />
-    </xacro:if>
-    <xacro:unless value="${tf_prefix == 'None'}">
-      <xacro:property name="tf_prefix_ext" value="${tf_prefix}_" />
-    </xacro:unless>
-    <joint name="${parent.rstrip('_link')}_${tf_prefix_ext}${side}_range_joint" type="fixed">
+  <xacro:macro name="vl53lox" params="parent xyz rpy prefix">
+    <joint name="${parent}_${prefix}_range_joint" type="fixed">
       <origin xyz="${xyz}" rpy="${rpy}" />
       <parent link="${parent}" />
-      <child link="${tf_prefix_ext}${side}_range" />
+      <child link="${prefix}_range" />
     </joint>
-    <link name="${tf_prefix_ext}${side}_range" />
+    <link name="${prefix}_range" />
     <!-- an IR sensor or a sonar are not implemented yet
     https://github.com/gazebosim/gz-sensors/issues/19 -->
-    <xacro:if value="${simulation_engine == 'ignition-gazebo'}">
-      <gazebo reference="${tf_prefix_ext}${side}_range">
-        <sensor name="${tf_prefix_ext}${side}_range" type='gpu_lidar'>
-          <topic>/range/${side}</topic>
-          <frame_id>${tf_prefix_ext}${side}_range</frame_id>
-          <ignition_frame_id>${tf_prefix_ext}${side}_range</ignition_frame_id>
+    <!-- <xacro:if value="${simulation_engine == 'ignition-gazebo'}">
+      <gazebo reference="${prefix}_range">
+        <sensor name="${prefix}_range" type='gpu_lidar'>
+          <topic>/range/${prefix}</topic>
+          <frame_id>${prefix}_range</frame_id>
+          <ignition_frame_id>${prefix}_range</ignition_frame_id>
           <update_rate>5.0</update_rate>
           <ray>
@@ -48,5 +42,5 @@
         </sensor>
       </gazebo>
-    </xacro:if>
+    </xacro:if> -->
   </xacro:macro>
 </robot>

File: rosbot_description/urdf/rosbot.urdf.xacro (robot description, xacro)
@@ -5,12 +5,5 @@
   <xacro:arg name="mecanum" default="false" />
   <xacro:arg name="simulation_engine" default="" />
-  <xacro:arg name="tf_prefix" default="None" />
-  <xacro:property name="tf_prefix" value="$(arg tf_prefix)" />
-  <xacro:if value="${tf_prefix == 'None'}">
-    <xacro:property name="tf_prefix_ext" value="" />
-  </xacro:if>
-  <xacro:unless value="${ tf_prefix == 'None'}">
-    <xacro:property name="tf_prefix_ext" value="${tf_prefix}_" />
-  </xacro:unless>
+  <xacro:arg name="namespace" default="" />
   <xacro:include filename="$(find rosbot_description)/urdf/rosbot_macro.urdf.xacro" ns="husarion" />
   <xacro:husarion.rosbot_robot
@@ -19,19 +12,17 @@
     use_gpu="$(arg use_gpu)"
     simulation_engine="$(arg simulation_engine)"
-    tf_prefix="$(arg tf_prefix)" />
-  <xacro:include filename="$(find ros_components_description)/urdf/slamtec_rplidar_a2.urdf.xacro" ns="lidar" />
+    namespace="$(arg namespace)" />
+  <!-- <xacro:include filename="$(find ros_components_description)/urdf/slamtec_rplidar_a2.urdf.xacro" ns="lidar" />
   <xacro:lidar.slamtec_rplidar_a2
-    parent_link="${tf_prefix_ext}cover_link"
+    parent_link="cover_link"
     xyz="0.02 0.0 0.0"
     rpy="0.0 0.0 0.0"
     use_gpu="$(arg use_gpu)"
-    simulation_engine="$(arg simulation_engine)"
-    tf_prefix="$(arg tf_prefix)" />
+    simulation_engine="$(arg simulation_engine)" />
   <xacro:include filename="$(find ros_components_description)/urdf/orbbec_astra.urdf.xacro" ns="camera" />
   <xacro:camera.orbbec_astra
-    parent_link="${tf_prefix_ext}camera_link"
+    parent_link="camera_link"
     xyz="0.0 0.0 0.0"
     rpy="0.0 0.0 0.0"
-    simulation_engine="$(arg simulation_engine)"
-    tf_prefix="$(arg tf_prefix)" />
+    simulation_engine="$(arg simulation_engine)" /> -->
 </robot>

File: rosbot_description/urdf/rosbot_macro.urdf.xacro (robot description, xacro)
@@ -1,5 +1,11 @@
 <?xml version='1.0'?>
 <robot xmlns:xacro="http://wiki.ros.org/xacro">
-  <xacro:macro name="rosbot_robot" params="mecanum use_sim use_gpu tf_prefix simulation_engine">
+  <xacro:macro name="rosbot_robot" params="mecanum use_sim use_gpu simulation_engine namespace">
+    <xacro:if value="${namespace == 'None'}">
+      <xacro:property name="namespace_ext" value="" />
+    </xacro:if>
+    <xacro:unless value="${namespace == 'None'}">
+      <xacro:property name="namespace_ext" value="${namespace}/" />
+    </xacro:unless>
     <xacro:if value="${mecanum}">
       <xacro:property name="wheel_radius" value="0.0470" />
@@ -8,23 +14,17 @@
       <xacro:property name="wheel_radius" value="0.0425" />
     </xacro:unless>
-    <xacro:if value="${tf_prefix == 'None'}">
-      <xacro:property name="tf_prefix_ext" value="" />
-    </xacro:if>
-    <xacro:unless value="${tf_prefix == 'None'}">
-      <xacro:property name="tf_prefix_ext" value="${tf_prefix}_" />
-    </xacro:unless>
     <!-- INCLUDE ROBOT PARTS DEFINITIONS -->
     <xacro:include filename="$(find rosbot_description)/urdf/body.urdf.xacro" ns="body" />
     <xacro:include filename="$(find rosbot_description)/urdf/wheel.urdf.xacro" ns="wheel" />
     <!-- BODY DECLARATION -->
-    <xacro:body.body wheel_radius="${wheel_radius}" mecanum="${mecanum}" use_gpu="${use_gpu}" tf_prefix="${tf_prefix}" />
+    <xacro:body.body wheel_radius="${wheel_radius}" mecanum="${mecanum}" use_gpu="${use_gpu}" />
     <!-- WHEEL DECLARATION -->
-    <xacro:wheel.wheel wheel_radius="${wheel_radius}" side="fr" mecanum="${mecanum}" tf_prefix="${tf_prefix}" />
-    <xacro:wheel.wheel wheel_radius="${wheel_radius}" side="fl" mecanum="${mecanum}" tf_prefix="${tf_prefix}" />
-    <xacro:wheel.wheel wheel_radius="${wheel_radius}" side="rl" mecanum="${mecanum}" tf_prefix="${tf_prefix}" />
-    <xacro:wheel.wheel wheel_radius="${wheel_radius}" side="rr" mecanum="${mecanum}" tf_prefix="${tf_prefix}" />
+    <xacro:wheel.wheel wheel_radius="${wheel_radius}" side="fr" mecanum="${mecanum}" namespace="${namespace}" />
+    <xacro:wheel.wheel wheel_radius="${wheel_radius}" side="fl" mecanum="${mecanum}" namespace="${namespace}" />
+    <xacro:wheel.wheel wheel_radius="${wheel_radius}" side="rl" mecanum="${mecanum}" namespace="${namespace}" />
+    <xacro:wheel.wheel wheel_radius="${wheel_radius}" side="rr" mecanum="${mecanum}" namespace="${namespace}" />
     <!-- ROS2 CONTROL -->
     <xacro:unless value="$(arg use_sim)">
-      <ros2_control name="imu" type="sensor">
+      <ros2_control name="${namespace_ext}imu" type="sensor">
         <hardware>
           <plugin>rosbot_hardware_interfaces/RosbotImuSensor</plugin>
@@ -32,5 +32,5 @@
           <param name="connection_check_period_ms">500</param>
         </hardware>
-        <sensor name="imu">
+        <sensor name="${namespace_ext}imu">
           <state_interface name="orientation.x" />
           <state_interface name="orientation.y" />
@@ -46,5 +46,5 @@
       </ros2_control>
     </xacro:unless>
-    <ros2_control name="wheels" type="system">
+    <ros2_control name="${namespace_ext}wheels" type="system">
       <hardware>
         <xacro:unless value="$(arg use_sim)">
@@ -61,5 +61,5 @@
                 fl_wheel_joint
           </param>
-          <param name="tf_prefix">${tf_prefix_ext}</param>
+          <param name="tf_prefix">${namespace_ext}</param>
         </xacro:unless>
         <xacro:if value="$(arg use_sim)">
@@ -72,27 +72,27 @@
         </xacro:if>
       </hardware>
-      <joint name="${tf_prefix_ext}fl_wheel_joint">
-        <command_interface name="velocity" />
-        <state_interface name="position" />
-        <state_interface name="velocity" />
-      </joint>
-      <joint name="${tf_prefix_ext}fr_wheel_joint">
-        <command_interface name="velocity" />
-        <state_interface name="position" />
-        <state_interface name="velocity" />
-      </joint>
-      <joint name="${tf_prefix_ext}rl_wheel_joint">
-        <command_interface name="velocity" />
-        <state_interface name="position" />
-        <state_interface name="velocity" />
-      </joint>
-      <joint name="${tf_prefix_ext}rr_wheel_joint">
-        <command_interface name="velocity" />
-        <state_interface name="position" />
-        <state_interface name="velocity" />
-      </joint>
-      <xacro:if value="${use_sim}">
+      <joint name="${namespace_ext}fl_wheel_joint">
+        <command_interface name="velocity" />
+        <state_interface name="position" />
+        <state_interface name="velocity" />
+      </joint>
+      <joint name="${namespace_ext}fr_wheel_joint">
+        <command_interface name="velocity" />
+        <state_interface name="position" />
+        <state_interface name="velocity" />
+      </joint>
+      <joint name="${namespace_ext}rl_wheel_joint">
+        <command_interface name="velocity" />
+        <state_interface name="position" />
+        <state_interface name="velocity" />
+      </joint>
+      <joint name="${namespace_ext}rr_wheel_joint">
+        <command_interface name="velocity" />
+        <state_interface name="position" />
+        <state_interface name="velocity" />
+      </joint>
+      <!-- <xacro:if value="${use_sim}">
         <xacro:if value="${simulation_engine == 'ignition-gazebo'}">
-          <sensor name="imu">
+          <sensor name="${namespace_ext}imu">
             <state_interface name="orientation.x" />
             <state_interface name="orientation.y" />
@@ -107,5 +107,5 @@
           </sensor>
         </xacro:if>
-      </xacro:if>
+      </xacro:if> -->
     </ros2_control>
     <!-- GAZEBO PLUGINS DECLARATION -->
@@ -114,18 +114,29 @@
         <gazebo>
           <plugin filename="ign_ros2_control-system" name="ign_ros2_control::IgnitionROS2ControlPlugin">
-            <xacro:if value="${mecanum}">
-              <parameters>$(find rosbot_controller)/config/mecanum_drive_controller.yaml</parameters>
+            <xacro:unless value="${namespace == 'None'}">
+              <xacro:if value="${mecanum}">
+                <parameters>$(find rosbot_gazebo)/config/multi_mecanum_drive_controller.yaml</parameters>
+              </xacro:if>
+              <xacro:unless value="${mecanum}">
+                <parameters>$(find rosbot_gazebo)/config/multi_diff_drive_controller.yaml</parameters>
+              </xacro:unless>
+            </xacro:unless>
+            <xacro:if value="${namespace == 'None'}">
+              <xacro:if value="${mecanum}">
+                <parameters>$(find rosbot_bringup)/config/mecanum_drive_controller.yaml</parameters>
+              </xacro:if>
+              <xacro:unless value="${mecanum}">
+                <parameters>$(find rosbot_bringup)/config/diff_drive_controller.yaml</parameters>
+              </xacro:unless>
             </xacro:if>
-            <xacro:unless value="${mecanum}">
-              <parameters>$(find rosbot_controller)/config/diff_drive_controller.yaml</parameters>
-            </xacro:unless>
-            <controller_manager_prefix_node_name>simulation</controller_manager_prefix_node_name>
             <ros>
-              <remapping>/rosbot_base_controller/cmd_vel_unstamped:=/cmd_vel</remapping>
+              <namespace>${namespace}</namespace>
+              <remapping>rosbot_base_controller/cmd_vel_unstamped:=cmd_vel</remapping>
+              <remapping>/tf:=tf</remapping>
             </ros>
           </plugin>
         </gazebo>
-        <gazebo reference="${tf_prefix_ext}imu_link">
-          <sensor name="imu" type="imu">
+        <!-- <gazebo reference="imu_link">
+          <sensor name="${namespace_ext}imu" type="imu">
             <plugin filename="ignition-gazebo-imu-system" name="ignition::gazebo::systems::Imu"></plugin>
             <always_on>true</always_on>
@@ -134,8 +145,11 @@
             <visualize>false</visualize>
             <enable_metrics>false</enable_metrics>
-            <frame_id>${tf_prefix_ext}imu_link</frame_id>
-            <ignition_frame_id>${tf_prefix_ext}imu_link</ignition_frame_id>
+            <frame_id>imu_link</frame_id>
+            <ignition_frame_id>imu_link</ignition_frame_id>
+            <ros>
+              <namespace>${namespace}</namespace>
+            </ros>
           </sensor>
-        </gazebo>
+        </gazebo>-->
       </xacro:if>
       <xacro:if value="${simulation_engine == 'gazebo-classic'}">
@@ -147,8 +161,8 @@
               <update_rate>10.0</update_rate>
               <num_wheel_pairs>2</num_wheel_pairs>
-              <left_joint>${tf_prefix_ext}fl_wheel_joint</left_joint>
-              <right_joint>${tf_prefix_ext}fr_wheel_joint</right_joint>
-              <left_joint>${tf_prefix_ext}rl_wheel_joint</left_joint>
-              <right_joint>${tf_prefix_ext}rr_wheel_joint</right_joint>
+              <left_joint>fl_wheel_joint</left_joint>
+              <right_joint>fr_wheel_joint</right_joint>
+              <left_joint>rl_wheel_joint</left_joint>
+              <right_joint>rr_wheel_joint</right_joint>
               <wheel_separation>0.192</wheel_separation>
               <wheel_separation>0.192</wheel_separation>
@@ -160,6 +174,6 @@
               <publish_odom_tf>true</publish_odom_tf>
               <publish_wheel_tf>true</publish_wheel_tf>
-              <odometry_frame>${tf_prefix_ext}odom</odometry_frame>
-              <robot_base_frame>${tf_prefix_ext}base_link</robot_base_frame>
+              <odometry_frame>odom</odometry_frame>
+              <robot_base_frame>base_link</robot_base_frame>
             </plugin>
           </gazebo>
@@ -168,12 +182,12 @@
         <gazebo>
           <plugin name="joint_states" filename="libgazebo_ros_joint_state_publisher.so">
-            <joint_name>${tf_prefix_ext}fl_wheel_joint</joint_name>
-            <joint_name>${tf_prefix_ext}fr_wheel_joint</joint_name>
-            <joint_name>${tf_prefix_ext}rl_wheel_joint</joint_name>
-            <joint_name>${tf_prefix_ext}rr_wheel_joint</joint_name>
+            <joint_name>fl_wheel_joint</joint_name>
+            <joint_name>fr_wheel_joint</joint_name>
+            <joint_name>rl_wheel_joint</joint_name>
+            <joint_name>rr_wheel_joint</joint_name>
           </plugin>
         </gazebo>
         <!-- publish IMU -->
-        <gazebo reference="${tf_prefix_ext}imu_link">
+        <gazebo reference="imu_link">
           <sensor type="imu" name="imu">
             <always_on>true</always_on>

File: rosbot_description/urdf/wheel.urdf.xacro (robot description, xacro)
@@ -2,10 +2,10 @@
 <robot xmlns:xacro="http://www.ros.org/wiki/xacro">
   <!-- wheel defining macro -->
-  <xacro:macro name="wheel" params="wheel_radius side mecanum tf_prefix">
-    <xacro:if value="${tf_prefix == 'None'}">
-      <xacro:property name="tf_prefix_ext" value="" />
+  <xacro:macro name="wheel" params="wheel_radius side mecanum namespace=None">
+    <xacro:if value="${namespace == 'None'}">
+      <xacro:property name="namespace_ext" value="" />
     </xacro:if>
-    <xacro:unless value="${tf_prefix == 'None'}">
-      <xacro:property name="tf_prefix_ext" value="${tf_prefix}_" />
+    <xacro:unless value="${namespace == 'None'}">
+      <xacro:property name="namespace_ext" value="${namespace}/" />
     </xacro:unless>
     <xacro:property name="wheel_separation_x" value="0.106" />
@@ -56,7 +56,7 @@
       <xacro:property name="fdir" value="1.0 -1.0 0.0" />
     </xacro:if>
-    <joint name="${tf_prefix_ext}${side}_wheel_joint" type="continuous">
-      <parent link="${tf_prefix_ext}body_link" />
-      <child link="${tf_prefix_ext}${side}_wheel_link" />
+    <joint name="${namespace_ext}${side}_wheel_joint" type="continuous">
+      <parent link="body_link" />
+      <child link="${side}_wheel_link" />
       <origin xyz="${x} ${y} 0.0" rpy="0.0 0.0 0.0" />
       <axis xyz="0.0 1.0 0.0" />
@@ -64,5 +64,5 @@
       <dynamics damping="0.001" friction="0.001" />
     </joint>
-    <link name="${tf_prefix_ext}${side}_wheel_link">
+    <link name="${side}_wheel_link">
       <visual>
         <geometry>
@@ -84,5 +84,5 @@
       </inertial>
     </link>
-    <gazebo reference="${tf_prefix_ext}${side}_wheel_link" xmlns:ignition="http://ignitionrobotics.org/schema">
+    <gazebo reference="${side}_wheel_link" xmlns:ignition="http://ignitionrobotics.org/schema">
       <collision>
         <surface>
@@ -91,5 +91,5 @@
               <mu>1.0</mu>
               <mu2>0.0</mu2>
-              <fdir1 ignition:expressed_in="${tf_prefix_ext}base_link">${fdir}</fdir1>
+              <fdir1 ignition:expressed_in="base_link">${fdir}</fdir1>
             </ode>
           </friction>
