Commit message: Added use_multirobot_system | found imu error
Signed-off-by: Jakub Delicat <jakub.delicat@husarion.com>

File: rosbot_description/urdf/body.urdf.xacro (robot description, xacro)
@@ -2,5 +2,5 @@
 <robot xmlns:xacro="http://www.ros.org/wiki/xacro">
   <!-- body defining macro -->
-  <xacro:macro name="body" params="wheel_radius mecanum use_gpu">
+  <xacro:macro name="body" params="wheel_radius mecanum use_gpu use_multirobot_system">
     <xacro:include filename="$(find rosbot_description)/urdf/components/vl53lox.urdf.xacro" ns="range_sensor" />
     <link name="base_link" />

File: rosbot_description/urdf/components/vl53lox.urdf.xacro (robot description, xacro)
@@ -11,5 +11,5 @@
     <!-- an IR sensor or a sonar are not implemented yet
     https://github.com/gazebosim/gz-sensors/issues/19 -->
-    <!-- <xacro:if value="${simulation_engine == 'ignition-gazebo'}">
+    <xacro:if value="${simulation_engine == 'ignition-gazebo'}">
       <gazebo reference="${prefix}_range">
         <sensor name="${prefix}_range" type='gpu_lidar'>
@@ -41,6 +41,9 @@
           <visualize>false</visualize>
         </sensor>
+        <plugin filename="libignition-gazebo-sensors-system.so"  name="ignition::gazebo::systems::Sensors">
+          <render_engine>ogre2</render_engine>
+        </plugin>
       </gazebo>
-    </xacro:if> -->
+    </xacro:if>
   </xacro:macro>
 </robot>

File: rosbot_description/urdf/rosbot.urdf.xacro (robot description, xacro)
@@ -5,5 +5,6 @@
   <xacro:arg name="mecanum" default="false" />
   <xacro:arg name="simulation_engine" default="" />
-  <xacro:arg name="namespace" default="" />
+  <xacro:arg name="namespace" default="None" />
+  <xacro:arg name="use_multirobot_system" default="true"/>
   <xacro:include filename="$(find rosbot_description)/urdf/rosbot_macro.urdf.xacro" ns="husarion" />
   <xacro:husarion.rosbot_robot
@@ -12,17 +13,5 @@
     use_gpu="$(arg use_gpu)"
     simulation_engine="$(arg simulation_engine)"
-    namespace="$(arg namespace)" />
-  <!-- <xacro:include filename="$(find ros_components_description)/urdf/slamtec_rplidar_a2.urdf.xacro" ns="lidar" />
-  <xacro:lidar.slamtec_rplidar_a2
-    parent_link="cover_link"
-    xyz="0.02 0.0 0.0"
-    rpy="0.0 0.0 0.0"
-    use_gpu="$(arg use_gpu)"
-    simulation_engine="$(arg simulation_engine)" />
-  <xacro:include filename="$(find ros_components_description)/urdf/orbbec_astra.urdf.xacro" ns="camera" />
-  <xacro:camera.orbbec_astra
-    parent_link="camera_link"
-    xyz="0.0 0.0 0.0"
-    rpy="0.0 0.0 0.0"
-    simulation_engine="$(arg simulation_engine)" /> -->
+    namespace="$(arg namespace)"
+    use_multirobot_system="$(arg use_multirobot_system)" />
 </robot>

File: rosbot_description/urdf/rosbot_macro.urdf.xacro (robot description, xacro)
@@ -1,5 +1,5 @@
 <?xml version='1.0'?>
 <robot xmlns:xacro="http://wiki.ros.org/xacro">
-  <xacro:macro name="rosbot_robot" params="mecanum use_sim use_gpu simulation_engine namespace">
+  <xacro:macro name="rosbot_robot" params="mecanum use_sim use_gpu simulation_engine namespace use_multirobot_system">
     <xacro:if value="${namespace == 'None'}">
       <xacro:property name="namespace_ext" value="" />
@@ -18,5 +18,5 @@
     <xacro:include filename="$(find rosbot_description)/urdf/wheel.urdf.xacro" ns="wheel" />
     <!-- BODY DECLARATION -->
-    <xacro:body.body wheel_radius="${wheel_radius}" mecanum="${mecanum}" use_gpu="${use_gpu}" />
+    <xacro:body.body wheel_radius="${wheel_radius}" mecanum="${mecanum}" use_gpu="${use_gpu}" use_multirobot_system="${use_multirobot_system}"/>
     <!-- WHEEL DECLARATION -->
     <xacro:wheel.wheel wheel_radius="${wheel_radius}" side="fr" mecanum="${mecanum}" namespace="${namespace}" />
@@ -114,5 +114,5 @@
         <gazebo>
           <plugin filename="ign_ros2_control-system" name="ign_ros2_control::IgnitionROS2ControlPlugin">
-            <xacro:unless value="${namespace == 'None'}">
+            <xacro:if value="${use_multirobot_system}">
               <xacro:if value="${mecanum}">
                 <parameters>$(find rosbot_gazebo)/config/multi_mecanum_drive_controller.yaml</parameters>
@@ -121,6 +121,6 @@
                 <parameters>$(find rosbot_gazebo)/config/multi_diff_drive_controller.yaml</parameters>
               </xacro:unless>
-            </xacro:unless>
-            <xacro:if value="${namespace == 'None'}">
+            </xacro:if>
+            <xacro:unless value="${use_multirobot_system}">
               <xacro:if value="${mecanum}">
                 <parameters>$(find rosbot_bringup)/config/mecanum_drive_controller.yaml</parameters>
@@ -129,5 +129,5 @@
                 <parameters>$(find rosbot_bringup)/config/diff_drive_controller.yaml</parameters>
               </xacro:unless>
-            </xacro:if>
+            </xacro:unless>
             <ros>
               <namespace>${namespace}</namespace>
@@ -142,5 +142,5 @@
             <always_on>true</always_on>
             <update_rate>25</update_rate>
-            <topic>imu/data_raw</topic>
+            <topic>${namespace_ext}imu/data_raw</topic>
             <visualize>false</visualize>
             <enable_metrics>false</enable_metrics>

Commit message: working without multisystem
Signed-off-by: Jakub Delicat <jakub.delicat@husarion.com>

File: rosbot_description/urdf/body.urdf.xacro (robot description, xacro)
@@ -2,5 +2,5 @@
 <robot xmlns:xacro="http://www.ros.org/wiki/xacro">
   <!-- body defining macro -->
-  <xacro:macro name="body" params="wheel_radius mecanum use_gpu use_multirobot_system">
+  <xacro:macro name="body" params="wheel_radius mecanum use_gpu">
     <xacro:include filename="$(find rosbot_description)/urdf/components/vl53lox.urdf.xacro" ns="range_sensor" />
     <link name="base_link" />

File: rosbot_description/urdf/rosbot_macro.urdf.xacro (robot description, xacro)
@@ -2,10 +2,4 @@
 <robot xmlns:xacro="http://wiki.ros.org/xacro">
   <xacro:macro name="rosbot_robot" params="mecanum use_sim use_gpu simulation_engine namespace use_multirobot_system">
-    <!-- Namespaces are necessary only with multiple robot system in Ignition Gazebo because
-         the same joint states crashes the simulator.
-    -->
-    <xacro:unless value="${use_multirobot_system}">
-      <xacro:property name="namespace" value="None" />
-    </xacro:unless>
     <xacro:if value="${namespace == 'None'}">
       <xacro:property name="namespace_ext" value="" />
@@ -24,10 +18,10 @@
     <xacro:include filename="$(find rosbot_description)/urdf/wheel.urdf.xacro" ns="wheel" />
     <!-- BODY DECLARATION -->
-    <xacro:body.body wheel_radius="${wheel_radius}" mecanum="${mecanum}" use_gpu="${use_gpu}" use_multirobot_system="${use_multirobot_system}"/>
+    <xacro:body.body wheel_radius="${wheel_radius}" mecanum="${mecanum}" use_gpu="${use_gpu}" />
     <!-- WHEEL DECLARATION -->
-    <xacro:wheel.wheel wheel_radius="${wheel_radius}" side="fr" mecanum="${mecanum}" namespace="${namespace}" />
-    <xacro:wheel.wheel wheel_radius="${wheel_radius}" side="fl" mecanum="${mecanum}" namespace="${namespace}" />
-    <xacro:wheel.wheel wheel_radius="${wheel_radius}" side="rl" mecanum="${mecanum}" namespace="${namespace}" />
-    <xacro:wheel.wheel wheel_radius="${wheel_radius}" side="rr" mecanum="${mecanum}" namespace="${namespace}" />
+    <xacro:wheel.wheel wheel_radius="${wheel_radius}" side="fr" mecanum="${mecanum}" />
+    <xacro:wheel.wheel wheel_radius="${wheel_radius}" side="fl" mecanum="${mecanum}" />
+    <xacro:wheel.wheel wheel_radius="${wheel_radius}" side="rl" mecanum="${mecanum}" />
+    <xacro:wheel.wheel wheel_radius="${wheel_radius}" side="rr" mecanum="${mecanum}" />
     <!-- ROS2 CONTROL -->
     <xacro:unless value="$(arg use_sim)">
@@ -75,20 +69,20 @@
         </xacro:if>
       </hardware>
-      <joint name="${namespace_ext}fl_wheel_joint">
-        <command_interface name="velocity" />
-        <state_interface name="position" />
-        <state_interface name="velocity" />
-      </joint>
-      <joint name="${namespace_ext}fr_wheel_joint">
-        <command_interface name="velocity" />
-        <state_interface name="position" />
-        <state_interface name="velocity" />
-      </joint>
-      <joint name="${namespace_ext}rl_wheel_joint">
-        <command_interface name="velocity" />
-        <state_interface name="position" />
-        <state_interface name="velocity" />
-      </joint>
-      <joint name="${namespace_ext}rr_wheel_joint">
+      <joint name="fl_wheel_joint">
+        <command_interface name="velocity" />
+        <state_interface name="position" />
+        <state_interface name="velocity" />
+      </joint>
+      <joint name="fr_wheel_joint">
+        <command_interface name="velocity" />
+        <state_interface name="position" />
+        <state_interface name="velocity" />
+      </joint>
+      <joint name="rl_wheel_joint">
+        <command_interface name="velocity" />
+        <state_interface name="position" />
+        <state_interface name="velocity" />
+      </joint>
+      <joint name="rr_wheel_joint">
         <command_interface name="velocity" />
         <state_interface name="position" />
@@ -118,5 +112,5 @@
           <plugin filename="ign_ros2_control-system" name="ign_ros2_control::IgnitionROS2ControlPlugin">
             <xacro:if value="${use_multirobot_system}">
-              <xacro:property name="controller_config_prefix" value="multi_" />
+              <xacro:property name="controller_config_prefix" value="" />
             </xacro:if>
             <xacro:unless value="${use_multirobot_system}">
@@ -124,13 +118,11 @@
             </xacro:unless>
             <xacro:if value="${mecanum}">
-              <parameters>$(find rosbot_controller)/config/${controller_config_prefix}mecanum_drive_controller.yaml</parameters>
+              <parameters>$(find rosbot_controller)/config/mecanum_drive_controller.yaml</parameters>
             </xacro:if>
             <xacro:unless value="${mecanum}">
-              <parameters>$(find rosbot_controller)/config/${controller_config_prefix}diff_drive_controller.yaml</parameters>
+              <parameters>$(find rosbot_controller)/config/diff_drive_controller.yaml</parameters>
             </xacro:unless>
             <ros>
-              <xacro:unless value="${namespace == 'None'}">
-                <namespace>${namespace}</namespace>
-              </xacro:unless>
+              <namespace>${namespace}</namespace>
               <remapping>rosbot_base_controller/cmd_vel_unstamped:=cmd_vel</remapping>
               <remapping>/tf:=tf</remapping>

File: rosbot_description/urdf/wheel.urdf.xacro (robot description, xacro)
@@ -2,11 +2,5 @@
 <robot xmlns:xacro="http://www.ros.org/wiki/xacro">
   <!-- wheel defining macro -->
-  <xacro:macro name="wheel" params="wheel_radius side mecanum namespace=None">
-    <xacro:if value="${namespace == 'None'}">
-      <xacro:property name="namespace_ext" value="" />
-    </xacro:if>
-    <xacro:unless value="${namespace == 'None'}">
-      <xacro:property name="namespace_ext" value="${namespace}/" />
-    </xacro:unless>
+  <xacro:macro name="wheel" params="wheel_radius side mecanum ">
     <xacro:property name="wheel_separation_x" value="0.106" />
     <xacro:if value="${mecanum}">
@@ -56,5 +50,5 @@
       <xacro:property name="fdir" value="1.0 -1.0 0.0" />
     </xacro:if>
-    <joint name="${namespace_ext}${side}_wheel_joint" type="continuous">
+    <joint name="${side}_wheel_joint" type="continuous">
       <parent link="body_link" />
       <child link="${side}_wheel_link" />

Commit message: Added range sensor
Signed-off-by: Jakub Delicat <jakub.delicat@husarion.com>

File: rosbot_description/urdf/body.urdf.xacro (robot description, xacro)
@@ -2,5 +2,5 @@
 <robot xmlns:xacro="http://www.ros.org/wiki/xacro">
   <!-- body defining macro -->
-  <xacro:macro name="body" params="wheel_radius mecanum use_gpu">
+  <xacro:macro name="body" params="wheel_radius mecanum use_gpu namespace">
     <xacro:include filename="$(find rosbot_description)/urdf/components/vl53lox.urdf.xacro" ns="range_sensor" />
     <link name="base_link" />
@@ -68,8 +68,8 @@
     </joint>
     <link name="camera_link" />
-    <xacro:range_sensor.vl53lox parent="body_link" xyz="0.0926  0.05 0.015"   rpy="0.0 0.0 ${radians(12.5)}"  prefix="fl" />
-    <xacro:range_sensor.vl53lox parent="body_link" xyz="0.0926 -0.05 0.015"   rpy="0.0 0.0 ${radians(-12.5)}" prefix="fr" />
-    <xacro:range_sensor.vl53lox parent="body_link" xyz="-0.0926 0.05 0.0115"  rpy="0.0 0.0 ${radians(167.5)}" prefix="rl" />
-    <xacro:range_sensor.vl53lox parent="body_link" xyz="-0.0926 -0.05 0.0115" rpy="0.0 0.0 ${radians(192.5)}" prefix="rr" />
+    <xacro:range_sensor.vl53lox parent="body_link" xyz="0.0926  0.05 0.015"   rpy="0.0 0.0 ${radians(12.5)}"  prefix="fl" namespace="${namespace}" />
+    <xacro:range_sensor.vl53lox parent="body_link" xyz="0.0926 -0.05 0.015"   rpy="0.0 0.0 ${radians(-12.5)}" prefix="fr" namespace="${namespace}" />
+    <xacro:range_sensor.vl53lox parent="body_link" xyz="-0.0926 0.05 0.0115"  rpy="0.0 0.0 ${radians(167.5)}" prefix="rl" namespace="${namespace}" />
+    <xacro:range_sensor.vl53lox parent="body_link" xyz="-0.0926 -0.05 0.0115" rpy="0.0 0.0 ${radians(192.5)}" prefix="rr" namespace="${namespace}" />
   </xacro:macro>
 </robot>

File: rosbot_description/urdf/components/vl53lox.urdf.xacro (robot description, xacro)
@@ -2,5 +2,13 @@
 <robot xmlns:xacro="http://www.ros.org/wiki/xacro">
   <!-- vl53lox defining macro -->
-  <xacro:macro name="vl53lox" params="parent xyz rpy prefix">
+  <xacro:macro name="vl53lox" params="parent xyz rpy prefix namespace">
+    <xacro:if value="${namespace == 'None'}">
+      <xacro:property name="namespace_ext" value="" />
+      <xacro:property name="gz_control_namespace" value="/" />
+    </xacro:if>
+    <xacro:unless value="${namespace == 'None'}">
+        <xacro:property name="namespace_ext" value="${namespace}/" />
+        <xacro:property name="gz_control_namespace" value="${namespace}" />
+    </xacro:unless>
     <joint name="${parent}_${prefix}_range_joint" type="fixed">
       <origin xyz="${xyz}" rpy="${rpy}" />
@@ -9,4 +17,44 @@
     </joint>
     <link name="${prefix}_range" />
+    <!-- an IR sensor or a sonar are not implemented yet
+    https://github.com/gazebosim/gz-sensors/issues/19 -->
+    <xacro:if value="${simulation_engine == 'ignition-gazebo'}">
+      <gazebo reference="${prefix}_range">
+        <sensor name="${namespace_ext}${prefix}_range" type='gpu_lidar'>
+          <topic>${gz_control_namespace}range/${prefix}</topic>
+          <frame_id>${prefix}_range</frame_id>
+          <ignition_frame_id>${prefix}_range</ignition_frame_id>
+          <update_rate>5.0</update_rate>
+          <ray>
+            <scan>
+              <horizontal>
+                <samples>1</samples>
+                <resolution>1</resolution>
+                <min_angle>-0.01</min_angle>
+                <max_angle>0.01</max_angle>
+              </horizontal>
+            </scan>
+            <range>
+              <min>0.01</min>
+              <max>0.90</max>
+              <resolution>0.02</resolution>
+            </range>
+            <noise>
+              <type>gaussian</type>
+              <mean>0.1</mean>
+              <stddev>0.005</stddev>
+            </noise>
+          </ray>
+          <always_on>true</always_on>
+          <visualize>false</visualize>
+          <ros>
+            <namespace></namespace>
+          </ros>
+        </sensor>
+        <plugin filename="libignition-gazebo-sensors-system.so"  name="ignition::gazebo::systems::Sensors">
+          <render_engine>ogre2</render_engine>
+        </plugin>
+      </gazebo>
+    </xacro:if>
   </xacro:macro>
 </robot>

File: rosbot_description/urdf/rosbot_macro.urdf.xacro (robot description, xacro)
@@ -20,5 +20,5 @@
     <xacro:include filename="$(find rosbot_description)/urdf/wheel.urdf.xacro" ns="wheel" />
     <!-- BODY DECLARATION -->
-    <xacro:body.body wheel_radius="${wheel_radius}" mecanum="${mecanum}" use_gpu="${use_gpu}" />
+    <xacro:body.body wheel_radius="${wheel_radius}" mecanum="${mecanum}" use_gpu="${use_gpu}" namespace="${namespace}" />
     <!-- WHEEL DECLARATION -->
     <xacro:wheel.wheel wheel_radius="${wheel_radius}" side="fr" mecanum="${mecanum}" />
