Commit message: Add gazebo namespace (#93)
* added namespaces to ros2_control

Signed-off-by: Jakub Delicat <jakub.delicat@husarion.com>

* removed action group

Signed-off-by: Jakub Delicat <jakub.delicat@husarion.com>

* Added namespace to robot description

Signed-off-by: Jakub Delicat <jakub.delicat@husarion.com>

* added tests for namespaces in rosbot_controller

Signed-off-by: Jakub Delicat <jakub.delicat@husarion.com>

* update worldlist

Signed-off-by: Jakub Delicat <jakub.delicat@husarion.com>

* fixed ros2_control namespaces | added namespace to ekf

Signed-off-by: Jakub Delicat <jakub.delicat@husarion.com>

* added mecanum

Signed-off-by: Jakub Delicat <jakub.delicat@husarion.com>

* added ros2_controllers to .gitignore

Signed-off-by: Jakub Delicat <jakub.delicat@husarion.com>

* ignored ros2_controllers during Industrial CI

Signed-off-by: Jakub Delicat <jakub.delicat@husarion.com>

* fixed tests

Signed-off-by: Jakub Delicat <jakub.delicat@husarion.com>

* added tf_prefix to imu_sensor_broadcaster

Signed-off-by: Jakub Delicat <jakub.delicat@husarion.com>

* copied only diff_drive and imu_broadcaster

Signed-off-by: Jakub Delicat <jakub.delicat@husarion.com>

* changed comments | changed timeout for controller test

Signed-off-by: Jakub Delicat <jakub.delicat@husarion.com>

* param changed to parameter

Signed-off-by: Jakub Delicat <jakub.delicat@husarion.com>

* Multi robot diff drive example

Signed-off-by: Jakub Delicat <jakub.delicat@husarion.com>

* imu also works

Signed-off-by: Jakub Delicat <jakub.delicat@husarion.com>

* Added use_multirobot_system | found imu error

Signed-off-by: Jakub Delicat <jakub.delicat@husarion.com>

* changed all topics to ns

Signed-off-by: Jakub Delicat <jakub.delicat@husarion.com>

* removed tf_prefix from xacro tests

Signed-off-by: Jakub Delicat <jakub.delicat@husarion.com>

* removed comments | add use_multirobot_system arg

Signed-off-by: Jakub Delicat <jakub.delicat@husarion.com>

* moved multi robot system controllers config to rosbot_controller

Signed-off-by: Jakub Delicat <jakub.delicat@husarion.com>

* fixed rosbot_gazebo test

Signed-off-by: Jakub Delicat <jakub.delicat@husarion.com>

* separated namespaced tests | added multirobot gazebo example with broken imu

Signed-off-by: Jakub Delicat <jakub.delicat@husarion.com>

* add multicontroller test

Signed-off-by: Jakub Delicat <jakub.delicat@husarion.com>

* add multibringup test

Signed-off-by: Jakub Delicat <jakub.delicat@husarion.com>

* add multibringup test

Signed-off-by: Jakub Delicat <jakub.delicat@husarion.com>

* Added remove rosbot_macro

Signed-off-by: Jakub Delicat <jakub.delicat@husarion.com>

* fixed miss spelling

Signed-off-by: Jakub Delicat <jakub.delicat@husarion.com>

* The change from robot_hardware_interface seems to be unnecessary

Signed-off-by: Jakub Delicat <jakub.delicat@husarion.com>

* moved multirobot tests to arrays

Signed-off-by: Jakub Delicat <jakub.delicat@husarion.com>

* move rosbot_hardware_interfaces to main

Signed-off-by: Jakub Delicat <jakub.delicat@husarion.com>

* Fixed len

Signed-off-by: Jakub Delicat <jakub.delicat@husarion.com>

* Added updated controllers info to readme

Signed-off-by: Jakub Delicat <jakub.delicat@husarion.com>

* Gazebo test (#86)

* Wait for velocity stabilization

* Apply suggestions from code review

Co-authored-by: Jakub Delicat <109142865+delihus@users.noreply.github.com>

* Apply suggestions from code review

* refactor

* test

* headless

* fix sim time

* update

* Update rosbot_gazebo/test/test_mecanum_simulation.py

Co-authored-by: Jakub Delicat <109142865+delihus@users.noreply.github.com>

---------

Co-authored-by: Jakub Delicat <109142865+delihus@users.noreply.github.com>

* Update changelog

* 0.10.5

* Added gazebo remappings file

Signed-off-by: Jakub Delicat <jakub.delicat@husarion.com>

* Added namespace to mappings

Signed-off-by: Jakub Delicat <jakub.delicat@husarion.com>

* fixed clock | added camera

Signed-off-by: Jakub Delicat <jakub.delicat@husarion.com>

* working without multisystem

Signed-off-by: Jakub Delicat <jakub.delicat@husarion.com>

* parse robots arg | removed delays from rosbot_controller

Signed-off-by: Jakub Delicat <jakub.delicat@husarion.com>

* TEsting

Signed-off-by: Jakub Delicat <jakub.delicat@husarion.com>

* fixed imu while testing

Signed-off-by: Jakub Delicat <jakub.delicat@husarion.com>

* Multirobots tests

Signed-off-by: Jakub Delicat <jakub.delicat@husarion.com>

* all gazebo tests

Signed-off-by: Jakub Delicat <jakub.delicat@husarion.com>

* changed to namespaced repositories

Signed-off-by: Jakub Delicat <jakub.delicat@husarion.com>

* revert headless to tests

Signed-off-by: Jakub Delicat <jakub.delicat@husarion.com>

* IMU name with slash

Signed-off-by: Jakub Delicat <jakub.delicat@husarion.com>

* removed delay from spawning

Signed-off-by: Jakub Delicat <jakub.delicat@husarion.com>

* added name for ign_ros2_controller

Signed-off-by: Jakub Delicat <jakub.delicat@husarion.com>

* fixed submodule

Signed-off-by: Jakub Delicat <jakub.delicat@husarion.com>

* checking mecanum controller sim time true

Signed-off-by: Jakub Delicat <jakub.delicat@husarion.com>

* Update industrial_ci.yaml

* removed coltroller test for testing timeout

Signed-off-by: Jakub Delicat <jakub.delicat@husarion.com>

* removed bringup tests for testing timeout

Signed-off-by: Jakub Delicat <jakub.delicat@husarion.com>

* used launch_ros features

Signed-off-by: Jakub Delicat <jakub.delicat@husarion.com>

* Added unbuffered to skip list

Signed-off-by: Jakub Delicat <jakub.delicat@husarion.com>

* added microros submodules to ignore and removed ros2 control demos from tests

Signed-off-by: Jakub Delicat <jakub.delicat@husarion.com>

* Revert "removed bringup tests for testing timeout"

This reverts commit f58a96780568bc4edd9cd976dc4f4d8bb29ab554.

* Revert "removed coltroller test for testing timeout"

This reverts commit 50c90e5028450640f9b2ce78584a76bceb3e6989.

* Added nav2_common to dependencies

Signed-off-by: Jakub Delicat <jakub.delicat@husarion.com>

* added readme

Signed-off-by: Jakub Delicat <jakub.delicat@husarion.com>

* Get the newest version of gz_ros2_control

Signed-off-by: Jakub Delicat <jakub.delicat@husarion.com>

* removed sim_time from yaml

Signed-off-by: Jakub Delicat <jakub.delicat@husarion.com>

* Added range sensor

Signed-off-by: Jakub Delicat <jakub.delicat@husarion.com>

* Added tests for ranges and camera

Signed-off-by: Jakub Delicat <jakub.delicat@husarion.com>

* removed unnecesary if

Signed-off-by: Jakub Delicat <jakub.delicat@husarion.com>

* Added me to the authors

Signed-off-by: Jakub Delicat <jakub.delicat@husarion.com>

* Update rosbot_hardware.repos

* Update rosbot_simulation.repos

* Update .github/workflows/industrial_ci.yaml

Co-authored-by: rafal-gorecki <126687345+rafal-gorecki@users.noreply.github.com>

* Update .github/workflows/industrial_ci.yaml

Co-authored-by: rafal-gorecki <126687345+rafal-gorecki@users.noreply.github.com>

* default simulator is ignition-gazebo

Signed-off-by: Jakub Delicat <jakub.delicat@husarion.com>

* merged multiple_simulation.launch.py with simulation.launch.py

Signed-off-by: Jakub Delicat <jakub.delicat@husarion.com>

* unnecessary event

Signed-off-by: Jakub Delicat <jakub.delicat@husarion.com>

* fix simulation.launch.py

* test max 3 robots + env(NS) + readme

* Better diagnostic in multirobot test

* simplify test

---------

Signed-off-by: Jakub Delicat <jakub.delicat@husarion.com>
Co-authored-by: rafal-gorecki <126687345+rafal-gorecki@users.noreply.github.com>
Co-authored-by: action-bot <action-bot@action-bot.com>
Co-authored-by: rafal-gorecki <rafal.gorecki@husarion.com>

File: rosbot_description/urdf/body.urdf.xacro (robot description, xacro)
@@ -2,5 +2,5 @@
 <robot xmlns:xacro="http://www.ros.org/wiki/xacro">
   <!-- body defining macro -->
-  <xacro:macro name="body" params="wheel_radius mecanum use_gpu use_multirobot_system">
+  <xacro:macro name="body" params="wheel_radius mecanum use_gpu namespace">
     <xacro:include filename="$(find rosbot_description)/urdf/components/vl53lox.urdf.xacro" ns="range_sensor" />
     <link name="base_link" />
@@ -68,8 +68,8 @@
     </joint>
     <link name="camera_link" />
-    <xacro:range_sensor.vl53lox parent="body_link" xyz="0.0926  0.05 0.015"   rpy="0.0 0.0 ${radians(12.5)}"  prefix="fl" />
-    <xacro:range_sensor.vl53lox parent="body_link" xyz="0.0926 -0.05 0.015"   rpy="0.0 0.0 ${radians(-12.5)}" prefix="fr" />
-    <xacro:range_sensor.vl53lox parent="body_link" xyz="-0.0926 0.05 0.0115"  rpy="0.0 0.0 ${radians(167.5)}" prefix="rl" />
-    <xacro:range_sensor.vl53lox parent="body_link" xyz="-0.0926 -0.05 0.0115" rpy="0.0 0.0 ${radians(192.5)}" prefix="rr" />
+    <xacro:range_sensor.vl53lox parent="body_link" xyz="0.0926  0.05 0.015"   rpy="0.0 0.0 ${radians(12.5)}"  prefix="fl" namespace="${namespace}" />
+    <xacro:range_sensor.vl53lox parent="body_link" xyz="0.0926 -0.05 0.015"   rpy="0.0 0.0 ${radians(-12.5)}" prefix="fr" namespace="${namespace}" />
+    <xacro:range_sensor.vl53lox parent="body_link" xyz="-0.0926 0.05 0.0115"  rpy="0.0 0.0 ${radians(167.5)}" prefix="rl" namespace="${namespace}" />
+    <xacro:range_sensor.vl53lox parent="body_link" xyz="-0.0926 -0.05 0.0115" rpy="0.0 0.0 ${radians(192.5)}" prefix="rr" namespace="${namespace}" />
   </xacro:macro>
 </robot>

File: rosbot_description/urdf/components/vl53lox.urdf.xacro (robot description, xacro)
@@ -2,5 +2,11 @@
 <robot xmlns:xacro="http://www.ros.org/wiki/xacro">
   <!-- vl53lox defining macro -->
-  <xacro:macro name="vl53lox" params="parent xyz rpy prefix">
+  <xacro:macro name="vl53lox" params="parent xyz rpy prefix namespace">
+    <xacro:if value="${namespace == 'None'}">
+      <xacro:property name="namespace_ext" value="" />
+    </xacro:if>
+    <xacro:unless value="${namespace == 'None'}">
+        <xacro:property name="namespace_ext" value="${namespace}/" />
+    </xacro:unless>
     <joint name="${parent}_${prefix}_range_joint" type="fixed">
       <origin xyz="${xyz}" rpy="${rpy}" />
@@ -13,6 +19,6 @@
     <xacro:if value="${simulation_engine == 'ignition-gazebo'}">
       <gazebo reference="${prefix}_range">
-        <sensor name="${prefix}_range" type='gpu_lidar'>
-          <topic>/range/${prefix}</topic>
+        <sensor name="${namespace_ext}${prefix}_range" type='gpu_lidar'>
+          <topic>${namespace_ext}range/${prefix}</topic>
           <frame_id>${prefix}_range</frame_id>
           <ignition_frame_id>${prefix}_range</ignition_frame_id>
@@ -40,8 +46,8 @@
           <always_on>true</always_on>
           <visualize>false</visualize>
+          <ros>
+            <namespace>${namespace_ext}</namespace>
+          </ros>
         </sensor>
-        <plugin filename="libignition-gazebo-sensors-system.so"  name="ignition::gazebo::systems::Sensors">
-          <render_engine>ogre2</render_engine>
-        </plugin>
       </gazebo>
     </xacro:if>

File: rosbot_description/urdf/rosbot.urdf.xacro (robot description, xacro)
@@ -4,7 +4,6 @@
   <xacro:arg name="use_gpu" default="false" />
   <xacro:arg name="mecanum" default="false" />
-  <xacro:arg name="simulation_engine" default="" />
+  <xacro:arg name="simulation_engine" default="ignition-gazebo" />
   <xacro:arg name="namespace" default="None" />
-  <xacro:arg name="use_multirobot_system" default="false"/>
   <xacro:include filename="$(find rosbot_description)/urdf/rosbot_macro.urdf.xacro" ns="husarion" />
   <xacro:husarion.rosbot_robot
@@ -13,20 +12,19 @@
     use_gpu="$(arg use_gpu)"
     simulation_engine="$(arg simulation_engine)"
-    namespace="$(arg namespace)"
-    use_multirobot_system="$(arg use_multirobot_system)" />
-    <xacro:unless value="$(arg use_multirobot_system)">
-      <xacro:include filename="$(find ros_components_description)/urdf/slamtec_rplidar_a2.urdf.xacro" ns="lidar" />
-      <xacro:lidar.slamtec_rplidar_a2
-        parent_link="cover_link"
-        xyz="0.02 0.0 0.0"
-        rpy="0.0 0.0 0.0"
-        use_gpu="$(arg use_gpu)"
-        simulation_engine="$(arg simulation_engine)" />
-      <xacro:include filename="$(find ros_components_description)/urdf/orbbec_astra.urdf.xacro" ns="camera" />
-      <xacro:camera.orbbec_astra
-        parent_link="camera_link"
-        xyz="0.0 0.0 0.0"
-        rpy="0.0 0.0 0.0"
-        simulation_engine="$(arg simulation_engine)" />
-    </xacro:unless>
+    namespace="$(arg namespace)" />
+    <xacro:include filename="$(find ros_components_description)/urdf/slamtec_rplidar_a2.urdf.xacro" ns="lidar" />
+    <xacro:lidar.slamtec_rplidar_a2
+      parent_link="cover_link"
+      xyz="0.02 0.0 0.0"
+      rpy="0.0 0.0 0.0"
+      use_gpu="$(arg use_gpu)"
+      namespace="$(arg namespace)"
+      simulation_engine="$(arg simulation_engine)" />
+    <xacro:include filename="$(find ros_components_description)/urdf/orbbec_astra.urdf.xacro" ns="camera" />
+    <xacro:camera.orbbec_astra
+      parent_link="camera_link"
+      xyz="0.0 0.0 0.0"
+      rpy="0.0 0.0 0.0"
+      namespace="$(arg namespace)"
+      simulation_engine="$(arg simulation_engine)" />
 </robot>

File: rosbot_description/urdf/rosbot_macro.urdf.xacro (robot description, xacro)
@@ -1,11 +1,5 @@
 <?xml version='1.0'?>
 <robot xmlns:xacro="http://wiki.ros.org/xacro">
-  <xacro:macro name="rosbot_robot" params="mecanum use_sim use_gpu simulation_engine namespace use_multirobot_system">
-    <!-- Namespaces are necessary only with multiple robot system in Ignition Gazebo because
-         the same joint states crashes the simulator.
-    -->
-    <xacro:unless value="${use_multirobot_system}">
-      <xacro:property name="namespace" value="None" />
-    </xacro:unless>
+  <xacro:macro name="rosbot_robot" params="mecanum use_sim use_gpu simulation_engine namespace ">
     <xacro:if value="${namespace == 'None'}">
       <xacro:property name="namespace_ext" value="" />
@@ -24,10 +18,10 @@
     <xacro:include filename="$(find rosbot_description)/urdf/wheel.urdf.xacro" ns="wheel" />
     <!-- BODY DECLARATION -->
-    <xacro:body.body wheel_radius="${wheel_radius}" mecanum="${mecanum}" use_gpu="${use_gpu}" use_multirobot_system="${use_multirobot_system}"/>
+    <xacro:body.body wheel_radius="${wheel_radius}" mecanum="${mecanum}" use_gpu="${use_gpu}" namespace="${namespace}" />
     <!-- WHEEL DECLARATION -->
-    <xacro:wheel.wheel wheel_radius="${wheel_radius}" side="fr" mecanum="${mecanum}" namespace="${namespace}" />
-    <xacro:wheel.wheel wheel_radius="${wheel_radius}" side="fl" mecanum="${mecanum}" namespace="${namespace}" />
-    <xacro:wheel.wheel wheel_radius="${wheel_radius}" side="rl" mecanum="${mecanum}" namespace="${namespace}" />
-    <xacro:wheel.wheel wheel_radius="${wheel_radius}" side="rr" mecanum="${mecanum}" namespace="${namespace}" />
+    <xacro:wheel.wheel wheel_radius="${wheel_radius}" side="fr" mecanum="${mecanum}" />
+    <xacro:wheel.wheel wheel_radius="${wheel_radius}" side="fl" mecanum="${mecanum}" />
+    <xacro:wheel.wheel wheel_radius="${wheel_radius}" side="rl" mecanum="${mecanum}" />
+    <xacro:wheel.wheel wheel_radius="${wheel_radius}" side="rr" mecanum="${mecanum}" />
     <!-- ROS2 CONTROL -->
     <xacro:unless value="$(arg use_sim)">
@@ -75,20 +69,20 @@
         </xacro:if>
       </hardware>
-      <joint name="${namespace_ext}fl_wheel_joint">
-        <command_interface name="velocity" />
-        <state_interface name="position" />
-        <state_interface name="velocity" />
-      </joint>
-      <joint name="${namespace_ext}fr_wheel_joint">
-        <command_interface name="velocity" />
-        <state_interface name="position" />
-        <state_interface name="velocity" />
-      </joint>
-      <joint name="${namespace_ext}rl_wheel_joint">
-        <command_interface name="velocity" />
-        <state_interface name="position" />
-        <state_interface name="velocity" />
-      </joint>
-      <joint name="${namespace_ext}rr_wheel_joint">
+      <joint name="fl_wheel_joint">
+        <command_interface name="velocity" />
+        <state_interface name="position" />
+        <state_interface name="velocity" />
+      </joint>
+      <joint name="fr_wheel_joint">
+        <command_interface name="velocity" />
+        <state_interface name="position" />
+        <state_interface name="velocity" />
+      </joint>
+      <joint name="rl_wheel_joint">
+        <command_interface name="velocity" />
+        <state_interface name="position" />
+        <state_interface name="velocity" />
+      </joint>
+      <joint name="rr_wheel_joint">
         <command_interface name="velocity" />
         <state_interface name="position" />
@@ -117,15 +111,9 @@
         <gazebo>
           <plugin filename="ign_ros2_control-system" name="ign_ros2_control::IgnitionROS2ControlPlugin">
-            <xacro:if value="${use_multirobot_system}">
-              <xacro:property name="controller_config_prefix" value="multi_" />
-            </xacro:if>
-            <xacro:unless value="${use_multirobot_system}">
-              <xacro:property name="controller_config_prefix" value="" />
-            </xacro:unless>
             <xacro:if value="${mecanum}">
-              <parameters>$(find rosbot_controller)/config/${controller_config_prefix}mecanum_drive_controller.yaml</parameters>
+              <parameters>$(find rosbot_controller)/config/mecanum_drive_controller.yaml</parameters>
             </xacro:if>
             <xacro:unless value="${mecanum}">
-              <parameters>$(find rosbot_controller)/config/${controller_config_prefix}diff_drive_controller.yaml</parameters>
+              <parameters>$(find rosbot_controller)/config/diff_drive_controller.yaml</parameters>
             </xacro:unless>
             <ros>
@@ -140,5 +128,4 @@
         <gazebo reference="imu_link">
           <sensor name="${namespace_ext}imu" type="imu">
-            <plugin filename="ignition-gazebo-imu-system" name="ignition::gazebo::systems::Imu"></plugin>
             <always_on>true</always_on>
             <update_rate>25</update_rate>
@@ -148,9 +135,7 @@
             <frame_id>imu_link</frame_id>
             <ignition_frame_id>imu_link</ignition_frame_id>
-            <xacro:unless value="${namespace == 'None'}">
-              <ros>
-                <namespace>${namespace}</namespace>
-              </ros>
-            </xacro:unless>
+            <ros>
+              <namespace>${namespace_ext}</namespace>
+            </ros>
           </sensor>
         </gazebo>

Commit message: Fix lidar in simulation

File: rosbot_description/urdf/body.urdf.xacro (robot description, xacro)
@@ -2,5 +2,5 @@
 <robot xmlns:xacro="http://www.ros.org/wiki/xacro">
   <!-- body defining macro -->
-  <xacro:macro name="body" params="wheel_radius mecanum use_gpu namespace">
+  <xacro:macro name="body" params="wheel_radius mecanum namespace">
     <xacro:include filename="$(find rosbot_description)/urdf/components/vl53lox.urdf.xacro" ns="range_sensor" />
     <link name="base_link" />

File: rosbot_description/urdf/rosbot.urdf.xacro (robot description, xacro)
@@ -2,5 +2,4 @@
 <robot name="rosbot" xmlns:xacro="http://www.ros.org/wiki/xacro">
   <xacro:arg name="use_sim" default="false" />
-  <xacro:arg name="use_gpu" default="false" />
   <xacro:arg name="mecanum" default="false" />
   <xacro:arg name="simulation_engine" default="ignition-gazebo" />
@@ -10,5 +9,4 @@
     mecanum="$(arg mecanum)"
     use_sim="$(arg use_sim)"
-    use_gpu="$(arg use_gpu)"
     simulation_engine="$(arg simulation_engine)"
     namespace="$(arg namespace)" />
@@ -18,5 +16,5 @@
       xyz="0.02 0.0 0.0"
       rpy="0.0 0.0 0.0"
-      use_gpu="$(arg use_gpu)"
+      use_gpu="true"
       namespace="$(arg namespace)"
       simulation_engine="$(arg simulation_engine)" />

File: rosbot_description/urdf/rosbot_macro.urdf.xacro (robot description, xacro)
@@ -1,5 +1,5 @@
 <?xml version='1.0'?>
 <robot xmlns:xacro="http://wiki.ros.org/xacro">
-  <xacro:macro name="rosbot_robot" params="mecanum use_sim use_gpu simulation_engine namespace ">
+  <xacro:macro name="rosbot_robot" params="mecanum use_sim simulation_engine namespace ">
     <xacro:if value="${namespace == 'None'}">
       <xacro:property name="namespace_ext" value="" />
@@ -18,5 +18,5 @@
     <xacro:include filename="$(find rosbot_description)/urdf/wheel.urdf.xacro" ns="wheel" />
     <!-- BODY DECLARATION -->
-    <xacro:body.body wheel_radius="${wheel_radius}" mecanum="${mecanum}" use_gpu="${use_gpu}" namespace="${namespace}" />
+    <xacro:body.body wheel_radius="${wheel_radius}" mecanum="${mecanum}" namespace="${namespace}" />
     <!-- WHEEL DECLARATION -->
     <xacro:wheel.wheel wheel_radius="${wheel_radius}" side="fr" mecanum="${mecanum}" />
