Commit message: Fix simulation

File: rosbot_description/urdf/body.urdf.xacro (robot description, xacro)
@@ -65,7 +65,7 @@
       <origin xyz="-0.0141 0.0 0.125" rpy="0.0 0.0 0.0" />
       <parent link="body_link" />
-      <child link="camera_link" />
+      <child link="camera_mount_link" />
     </joint>
-    <link name="camera_link" />
+    <link name="camera_mount_link" />
     <xacro:range_sensor.vl53lox parent="body_link" xyz="0.0926  0.05 0.015"   rpy="0.0 0.0 ${radians(12.5)}"  prefix="fl" namespace="${namespace}" />
     <xacro:range_sensor.vl53lox parent="body_link" xyz="0.0926 -0.05 0.015"   rpy="0.0 0.0 ${radians(-12.5)}" prefix="fr" namespace="${namespace}" />

File: rosbot_description/urdf/components/vl53lox.urdf.xacro (robot description, xacro)
@@ -17,39 +17,33 @@
     <!-- an IR sensor or a sonar are not implemented yet
     https://github.com/gazebosim/gz-sensors/issues/19 -->
-    <xacro:if value="${simulation_engine == 'ignition-gazebo'}">
-      <gazebo reference="${prefix}_range">
-        <sensor name="${namespace_ext}${prefix}_range" type='gpu_lidar'>
-          <topic>${namespace_ext}range/${prefix}</topic>
-          <frame_id>${prefix}_range</frame_id>
-          <ignition_frame_id>${prefix}_range</ignition_frame_id>
-          <update_rate>5.0</update_rate>
-          <ray>
-            <scan>
-              <horizontal>
-                <samples>1</samples>
-                <resolution>1</resolution>
-                <min_angle>-0.01</min_angle>
-                <max_angle>0.01</max_angle>
-              </horizontal>
-            </scan>
-            <range>
-              <min>0.01</min>
-              <max>0.90</max>
-              <resolution>0.02</resolution>
-            </range>
-            <noise>
-              <type>gaussian</type>
-              <mean>0.1</mean>
-              <stddev>0.005</stddev>
-            </noise>
-          </ray>
-          <always_on>true</always_on>
-          <visualize>false</visualize>
-          <ros>
-            <namespace>${namespace_ext}</namespace>
-          </ros>
-        </sensor>
-      </gazebo>
-    </xacro:if>
+    <gazebo reference="${prefix}_range">
+      <sensor name="${namespace_ext}${prefix}_range" type='gpu_lidar'>
+        <topic>${namespace_ext}range/${prefix}</topic>
+        <gz_frame_id>${prefix}_range</gz_frame_id>
+        <update_rate>5.0</update_rate>
+        <ray>
+          <scan>
+            <horizontal>
+              <samples>1</samples>
+              <resolution>1</resolution>
+              <min_angle>-0.01</min_angle>
+              <max_angle>0.01</max_angle>
+            </horizontal>
+          </scan>
+          <range>
+            <min>0.01</min>
+            <max>0.90</max>
+            <resolution>0.02</resolution>
+          </range>
+          <noise>
+            <type>gaussian</type>
+            <mean>0.1</mean>
+            <stddev>0.005</stddev>
+          </noise>
+        </ray>
+        <always_on>true</always_on>
+        <visualize>false</visualize>
+      </sensor>
+    </gazebo>
   </xacro:macro>
 </robot>

File: rosbot_description/urdf/rosbot.urdf.xacro (robot description, xacro)
@@ -3,5 +3,4 @@
   <xacro:arg name="use_sim" default="false" />
   <xacro:arg name="mecanum" default="false" />
-  <xacro:arg name="simulation_engine" default="ignition-gazebo" />
   <xacro:arg name="namespace" default="None" />
   <xacro:include filename="$(find rosbot_description)/urdf/rosbot_macro.urdf.xacro" ns="husarion" />
@@ -9,20 +8,15 @@
     mecanum="$(arg mecanum)"
     use_sim="$(arg use_sim)"
-    simulation_engine="$(arg simulation_engine)"
     namespace="$(arg namespace)" />
-    <xacro:include filename="$(find ros_components_description)/urdf/slamtec_rplidar_a2.urdf.xacro" ns="lidar" />
-    <xacro:lidar.slamtec_rplidar_a2
+    <xacro:include filename="$(find ros_components_description)/urdf/slamtec_rplidar.urdf.xacro" ns="lidar" />
+    <xacro:lidar.slamtec_rplidar
       parent_link="cover_link"
       xyz="0.02 0.0 0.0"
       rpy="0.0 0.0 0.0"
-      use_gpu="true"
-      namespace="$(arg namespace)"
-      simulation_engine="$(arg simulation_engine)" />
+      model="a3" />
     <xacro:include filename="$(find ros_components_description)/urdf/orbbec_astra.urdf.xacro" ns="camera" />
     <xacro:camera.orbbec_astra
-      parent_link="camera_link"
+      parent_link="camera_mount_link"
       xyz="0.0 0.0 0.0"
-      rpy="0.0 0.0 0.0"
-      namespace="$(arg namespace)"
-      simulation_engine="$(arg simulation_engine)" />
+      rpy="0.0 0.0 0.0" />
 </robot>

File: rosbot_description/urdf/rosbot_macro.urdf.xacro (robot description, xacro)
@@ -1,5 +1,5 @@
 <?xml version='1.0'?>
 <robot xmlns:xacro="http://wiki.ros.org/xacro">
-  <xacro:macro name="rosbot_robot" params="mecanum use_sim simulation_engine namespace ">
+  <xacro:macro name="rosbot_robot" params="mecanum use_sim namespace">
     <xacro:property name="ns" value="${namespace + '/' if namespace != 'None' else ''}" />
     <xacro:property name="wheel_radius" value="${0.0470 if mecanum else 0.0425}" />
@@ -16,5 +16,5 @@
     <!-- ROS2 CONTROL -->
     <xacro:unless value="$(arg use_sim)">
-      <ros2_control name="${ns}imu" type="sensor">
+      <ros2_control name="imu" type="sensor">
         <hardware>
           <plugin>rosbot_hardware_interfaces/RosbotImuSensor</plugin>
@@ -22,5 +22,5 @@
           <param name="connection_check_period_ms">1000</param>
         </hardware>
-        <sensor name="${ns}imu">
+        <sensor name="imu">
           <state_interface name="orientation.x" />
           <state_interface name="orientation.y" />
@@ -51,10 +51,5 @@
         </xacro:unless>
         <xacro:if value="$(arg use_sim)">
-          <xacro:if value="${simulation_engine == 'ignition-gazebo'}">
-            <plugin>gz_ros2_control/GazeboSimSystem</plugin>
-          </xacro:if>
-          <xacro:if value="${simulation_engine == 'webots'}">
-            <plugin>webots_ros2_control::Ros2ControlSystem</plugin>
-          </xacro:if>
+          <plugin>gz_ros2_control/GazeboSimSystem</plugin>
         </xacro:if>
       </hardware>
@@ -80,117 +75,50 @@
       </joint>
       <xacro:if value="${use_sim}">
-        <xacro:if value="${simulation_engine == 'ignition-gazebo'}">
-          <sensor name="${ns}imu">
-            <state_interface name="orientation.x" />
-            <state_interface name="orientation.y" />
-            <state_interface name="orientation.z" />
-            <state_interface name="orientation.w" />
-            <state_interface name="angular_velocity.x" />
-            <state_interface name="angular_velocity.y" />
-            <state_interface name="angular_velocity.z" />
-            <state_interface name="linear_acceleration.x" />
-            <state_interface name="linear_acceleration.y" />
-            <state_interface name="linear_acceleration.z" />
-          </sensor>
-        </xacro:if>
+        <sensor name="imu">
+          <state_interface name="orientation.x" />
+          <state_interface name="orientation.y" />
+          <state_interface name="orientation.z" />
+          <state_interface name="orientation.w" />
+          <state_interface name="angular_velocity.x" />
+          <state_interface name="angular_velocity.y" />
+          <state_interface name="angular_velocity.z" />
+          <state_interface name="linear_acceleration.x" />
+          <state_interface name="linear_acceleration.y" />
+          <state_interface name="linear_acceleration.z" />
+        </sensor>
       </xacro:if>
     </ros2_control>
     <!-- GAZEBO PLUGINS DECLARATION -->
     <xacro:if value="${use_sim}">
-      <xacro:if value="${simulation_engine == 'ignition-gazebo'}">
-        <gazebo>
-          <plugin filename="gz_ros2_control-system" name="gz_ros2_control::GazeboSimROS2ControlPlugin">
-            <xacro:if value="${mecanum}">
-              <parameters>$(find rosbot_controller)/config/mecanum_drive_controller.yaml</parameters>
-            </xacro:if>
-            <xacro:unless value="${mecanum}">
-              <parameters>$(find rosbot_controller)/config/diff_drive_controller.yaml</parameters>
+      <gazebo>
+        <plugin filename="gz_ros2_control-system" name="gz_ros2_control::GazeboSimROS2ControlPlugin">
+          <xacro:if value="${mecanum}">
+            <parameters>$(find rosbot_controller)/config/mecanum_drive_controller.yaml</parameters>
+          </xacro:if>
+          <xacro:unless value="${mecanum}">
+            <parameters>$(find rosbot_controller)/config/diff_drive_controller.yaml</parameters>
+          </xacro:unless>
+          <ros>
+            <xacro:unless value="${namespace == 'None'}">
+              <namespace>${namespace}</namespace>
             </xacro:unless>
-            <ros>
-              <xacro:unless value="${namespace == 'None'}">
-                <namespace>${namespace}</namespace>
-              </xacro:unless>
-              <remapping>rosbot_base_controller/cmd_vel:=cmd_vel</remapping>
-              <remapping>/tf:=tf</remapping>
-            </ros>
-          </plugin>
-        </gazebo>
-        <gazebo reference="imu_link">
-          <sensor name="${ns}imu" type="imu">
-            <always_on>true</always_on>
-            <update_rate>25</update_rate>
-            <topic>${ns}imu/data_raw</topic>
-            <visualize>false</visualize>
-            <enable_metrics>false</enable_metrics>
-            <frame_id>imu_link</frame_id>
-            <ignition_frame_id>imu_link</ignition_frame_id>
-            <ros>
-              <namespace>${namespace}</namespace>
-            </ros>
-          </sensor>
-        </gazebo>
-      </xacro:if>
-      <xacro:if value="${simulation_engine == 'gazebo-classic'}">
-        <!-- Control robot wheels -->
-        <xacro:unless value="${mecanum}">
-          <gazebo>
-            <plugin name='skid_steer_drive' filename='libgazebo_ros_diff_drive.so'>
-              <ros></ros>
-              <update_rate>10.0</update_rate>
-              <num_wheel_pairs>2</num_wheel_pairs>
-              <left_joint>fl_wheel_joint</left_joint>
-              <right_joint>fr_wheel_joint</right_joint>
-              <left_joint>rl_wheel_joint</left_joint>
-              <right_joint>rr_wheel_joint</right_joint>
-              <wheel_separation>0.192</wheel_separation>
-              <wheel_separation>0.192</wheel_separation>
-              <wheel_diameter>${wheel_radius*2.0}</wheel_diameter>
-              <wheel_diameter>${wheel_radius*2.0}</wheel_diameter>
-              <max_wheel_torque>1.5</max_wheel_torque>
-              <max_wheel_acceleration>1.0</max_wheel_acceleration>
-              <publish_odom>true</publish_odom>
-              <publish_odom_tf>true</publish_odom_tf>
-              <publish_wheel_tf>true</publish_wheel_tf>
-              <odometry_frame>odom</odometry_frame>
-              <robot_base_frame>base_link</robot_base_frame>
-            </plugin>
-          </gazebo>
-        </xacro:unless>
-        <!-- publish joint states -->
-        <gazebo>
-          <plugin name="joint_states" filename="libgazebo_ros_joint_state_publisher.so">
-            <joint_name>fl_wheel_joint</joint_name>
-            <joint_name>fr_wheel_joint</joint_name>
-            <joint_name>rl_wheel_joint</joint_name>
-            <joint_name>rr_wheel_joint</joint_name>
-          </plugin>
-        </gazebo>
-        <!-- publish IMU -->
-        <gazebo reference="imu_link">
-          <sensor type="imu" name="imu">
-            <always_on>true</always_on>
-            <update_rate>25</update_rate>
-            <plugin name="bno055_imu_plugin" filename="libgazebo_ros_imu_sensor.so">
-              <ros>
-                <argument>~/out:=imu/data/raw</argument>
-              </ros>
-            </plugin>
-          </sensor>
-        </gazebo>
-      </xacro:if>
-      <xacro:if value="${simulation_engine == 'webots'}">
-        <webots>
-          <plugin type="webots_ros2_control::Ros2Control" />
-          <plugin type="webots_ros2_driver::Ros2IMU">
-            <enabled>true</enabled>
-            <topicName>/imu_broadcaster/imu</topicName>
-            <alwaysOn>true</alwaysOn>
-            <frameName>imu_link</frameName>
-            <gyroName>imu gyro</gyroName>
-            <accelerometerName>imu accelerometer</accelerometerName>
-            <inertialUnitName>imu inertial_unit</inertialUnitName>
-          </plugin>
-        </webots>
-      </xacro:if>
+            <remapping>rosbot_base_controller/cmd_vel:=cmd_vel</remapping>
+            <remapping>/tf:=tf</remapping>
+          </ros>
+        </plugin>
+      </gazebo>
+      <gazebo reference="imu_link">
+        <sensor name="imu" type="imu">
+          <always_on>true</always_on>
+          <update_rate>25</update_rate>
+          <topic>imu/data_raw</topic>
+          <visualize>false</visualize>
+          <enable_metrics>false</enable_metrics>
+          <gz_frame_id>imu_link</gz_frame_id>
+          <ros>
+            <namespace>${namespace}</namespace>
+          </ros>
+        </sensor>
+      </gazebo>
     </xacro:if>
   </xacro:macro>

Commit message: Update URDF, fix mecanum sim, fix laser_filter ns, remove tf renaming

File: rosbot_description/urdf/body.urdf.xacro (robot description, xacro)
@@ -16,6 +16,6 @@
         </geometry>
         <origin xyz="0.0 0.0 -0.0173" rpy="${pi/2} 0.0 ${pi/2}" />
-        <material name="White">
-          <color rgba="1.0 1.0 1.0 1.0" />
+        <material name="Black">
+          <color rgba="0.1 0.1 0.1 0.1" />
         </material>
       </visual>
@@ -35,5 +35,5 @@
     </link>
     <gazebo reference="body_link">
-      <material>Gazebo/White</material>
+      <material>Gazebo/Black</material>
     </gazebo>
     <joint name="body_to_cover_joint" type="fixed">

File: rosbot_description/urdf/rosbot.urdf.xacro (robot description, xacro)
@@ -5,5 +5,5 @@
   <xacro:arg name="namespace" default="None" />
   <xacro:include filename="$(find rosbot_description)/urdf/rosbot_macro.urdf.xacro" ns="husarion" />
-  <xacro:husarion.rosbot_robot
+  <xacro:husarion.rosbot
     mecanum="$(arg mecanum)"
     use_sim="$(arg use_sim)"
@@ -14,9 +14,11 @@
       xyz="0.02 0.0 0.0"
       rpy="0.0 0.0 0.0"
-      model="a3" />
-    <xacro:include filename="$(find ros_components_description)/urdf/orbbec_astra.urdf.xacro" ns="camera" />
-    <xacro:camera.orbbec_astra
-      parent_link="camera_mount_link"
-      xyz="0.0 0.0 0.0"
-      rpy="0.0 0.0 0.0" />
+      model="s2"
+      namespace="$(arg namespace)" />
+	<xacro:include filename="$(find depthai_descriptions)/urdf/include/depthai_macro.urdf.xacro" ns="camera" />
+	<xacro:camera.depthai_camera camera_name="oak_camera" parent="camera_mount_link"
+		camera_model="OAK-D-PRO" base_frame="oak_camera"
+		cam_pos_x="0.0" cam_pos_y="0.0" cam_pos_z="0.02"
+		cam_roll="0.0" cam_pitch="0.0" cam_yaw="0.0"
+    r="0.2" g="0.2" b="0.2" a="1.0"	rs_compat="false" simulation="$(arg use_sim)" />
 </robot>

File: rosbot_description/urdf/rosbot_macro.urdf.xacro (robot description, xacro)
@@ -1,5 +1,5 @@
 <?xml version='1.0'?>
 <robot xmlns:xacro="http://wiki.ros.org/xacro">
-  <xacro:macro name="rosbot_robot" params="mecanum use_sim namespace">
+  <xacro:macro name="rosbot" params="mecanum use_sim namespace">
     <xacro:property name="ns" value="${namespace + '/' if namespace != 'None' else ''}" />
     <xacro:property name="wheel_radius" value="${0.0470 if mecanum else 0.0425}" />
@@ -104,5 +104,4 @@
             </xacro:unless>
             <remapping>rosbot_base_controller/cmd_vel:=cmd_vel</remapping>
-            <remapping>/tf:=tf</remapping>
           </ros>
         </plugin>

File: rosbot_description/urdf/wheel.urdf.xacro (robot description, xacro)
@@ -37,6 +37,6 @@
     </xacro:if>
     <xacro:if value="${side == 'rl'}">
-      <xacro:property name="x" value="${-wheel_separation_x/2}" />
-      <xacro:property name="y" value="${wheel_separation_y/2}" />
+      <xacro:property name="x" value="${-wheel_separation_x/2.0}" />
+      <xacro:property name="y" value="${wheel_separation_y/2.0}" />
       <xacro:property name="mesh" value="package://rosbot_description/meshes/${wheel_file}_a.dae" />
       <xacro:property name="visual_rotation" value="${0.0}" />
@@ -44,6 +44,6 @@
     </xacro:if>
     <xacro:if value="${side == 'rr'}">
-      <xacro:property name="x" value="${-wheel_separation_x/2}" />
-      <xacro:property name="y" value="${-wheel_separation_y/2}" />
+      <xacro:property name="x" value="${-wheel_separation_x/2.0}" />
+      <xacro:property name="y" value="${-wheel_separation_y/2.0}" />
       <xacro:property name="mesh" value="package://rosbot_description/meshes/${wheel_file}_b.dae" />
       <xacro:property name="visual_rotation" value="${0.0}" />
@@ -78,19 +78,36 @@
       </inertial>
     </link>
-    <xacro:if value="${mecanum}">
-      <gazebo reference="${side}_wheel_link" xmlns:ignition="http://ignitionrobotics.org/schema">
+    <gazebo reference="${side}_wheel_link" xmlns:gz="http://gazeborobotics.org/schema">
+      <xacro:unless value="${mecanum}">
         <collision>
           <surface>
             <friction>
               <ode>
-                <mu>1.0</mu>
-                <mu2>0.0</mu2>
-                <fdir1 ignition:expressed_in="base_link">${fdir}</fdir1>
+                <mu>1</mu>
+                <mu2>1</mu2>
+                <slip1>0.035</slip1>
+                <slip2>0</slip2>
+                <fdir1>0 0 1</fdir1>
               </ode>
             </friction>
           </surface>
         </collision>
-      </gazebo>
-    </xacro:if>
+      </xacro:unless>
+      <xacro:if value="${mecanum}">
+        <collision>
+          <surface>
+            <friction>
+              <ode>
+                <mu>0.8</mu>
+                <mu2>0.2</mu2>
+                  <slip1>0.035</slip1>
+                <slip2>0</slip2>
+                <fdir1 gz:expressed_in="base_link">${fdir}</fdir1>
+              </ode>
+            </friction>
+          </surface>
+        </collision>
+      </xacro:if>
+    </gazebo>
   </xacro:macro>
 </robot>
