Commit message: Jazzy - General code maintenance (#123)
* support for RPi5

* restart ros2_control_node if error

* minor fixes

* Update controller.launch.py

* fix mecanum lauch

* Fix controller namespace (#115)

* Fix controller namespace

* spellcheck fix

* use husarion-controller from main branch (#116)

* added docker setup for local build

* ros2 humble works without custom controllers

* Cleaner logs from flash script (#108)

* Clean up output of flash script

* Pre commit

* Cleaner

* Specify concrete commands

* Simplify

* pre-commit fix

* Clean up usb firmware

* Clean up unused arguments (#118)

* Add scan filter

* Clean up

* undo

* added docker setup for local build

* broken ros2 controller - previous worked fine

* Clean up unused arguments

* Fix workflow: Remove spellcheck (redundant), fix integration check

* Fix multiple robot spawn

* fixes

* Delete tools folder

* Pre-commit update and remove redundant flake8

* Fix some tests and set hash in vcs

* Clean up

* Move controller test to bringup and reduce test time

* Fix lidar in simulation

* Rename test files

* Fix tests

* Add scan_filtered test and improve workpace tree

---------

Co-authored-by: Dominik Nowak <dominik.nwk@gmail.com>

* Applied xml schemas for xmllint (#101)

* applied package.xml template

Signed-off-by: Jakub Delicat <jakub.delicat@husarion.com>

* chronology

Signed-off-by: Jakub Delicat <jakub.delicat@husarion.com>

* Support

Signed-off-by: Jakub Delicat <jakub.delicat@husarion.com>

* Removed unnecessary dep

Signed-off-by: Jakub Delicat <jakub.delicat@husarion.com>

* DDS xml lint

---------

Signed-off-by: Jakub Delicat <jakub.delicat@husarion.com>
Co-authored-by: rafal-gorecki <rafal.gorecki@husarion.com>

* Some fixes

* test

* Pre-commit

* pre-commit

* Humble docker (#124)

* Add hardware and sim Docker

* Fix hardware docker

* Fixes

* Use packages-up-to

* Add description to compose

* Jazzy docker (#125)

* Add hardware and sim Docker

* Fix hardware docker

* Fixes

* Fixes

* Simulation gz_gui fixes + use TwistStamped

* Use packages-up-to

* Add healthcheck + clean up

* Add healthcheck + clean up

* Remove combined.launch.py

* Add User env to docker

* Add devcontainer

* Changes in healthcheck

* Fix simulation

* Red error info

* Change healthcheck

* Remove healthcheck arg

* Fix workflow

* Remove building imu_broadcaster

* One more removal

* update repos

* Clean up

* Update docs

* Add launch arguments info

* Add status info

* add unsaved

* fix

* Simplify

* Update URDF, fix mecanum sim, fix laser_filter ns, remove tf renaming

* pre-commit

* Fix ros2 controller with namespace

* Fix building instructions

* Fix indent

* Fix mecanum controller

* Remove camera test from sim

* update

* Adjust wheel_separation_multiplier param

* Simplify docker

---------

Signed-off-by: Jakub Delicat <jakub.delicat@husarion.com>
Co-authored-by: dominikn <dominik.nwk@gmail.com>
Co-authored-by: Jakub Delicat <109142865+delihus@users.noreply.github.com>

File: rosbot_description/urdf/body.urdf.xacro (robot description, xacro)
@@ -2,5 +2,5 @@
 <robot xmlns:xacro="http://www.ros.org/wiki/xacro">
   <!-- body defining macro -->
-  <xacro:macro name="body" params="wheel_radius mecanum use_gpu namespace">
+  <xacro:macro name="body" params="wheel_radius mecanum namespace">
     <xacro:include filename="$(find rosbot_description)/urdf/components/vl53lox.urdf.xacro" ns="range_sensor" />
     <link name="base_link" />
@@ -16,6 +16,6 @@
         </geometry>
         <origin xyz="0.0 0.0 -0.0173" rpy="${pi/2} 0.0 ${pi/2}" />
-        <material name="White">
-          <color rgba="1.0 1.0 1.0 1.0" />
+        <material name="Black">
+          <color rgba="0.1 0.1 0.1 0.1" />
         </material>
       </visual>
@@ -35,5 +35,5 @@
     </link>
     <gazebo reference="body_link">
-      <material>Gazebo/White</material>
+      <material>Gazebo/Black</material>
     </gazebo>
     <joint name="body_to_cover_joint" type="fixed">
@@ -65,7 +65,7 @@
       <origin xyz="-0.0141 0.0 0.125" rpy="0.0 0.0 0.0" />
       <parent link="body_link" />
-      <child link="camera_link" />
+      <child link="camera_mount_link" />
     </joint>
-    <link name="camera_link" />
+    <link name="camera_mount_link" />
     <xacro:range_sensor.vl53lox parent="body_link" xyz="0.0926  0.05 0.015"   rpy="0.0 0.0 ${radians(12.5)}"  prefix="fl" namespace="${namespace}" />
     <xacro:range_sensor.vl53lox parent="body_link" xyz="0.0926 -0.05 0.015"   rpy="0.0 0.0 ${radians(-12.5)}" prefix="fr" namespace="${namespace}" />

File: rosbot_description/urdf/rosbot.urdf.xacro (robot description, xacro)
@@ -2,29 +2,23 @@
 <robot name="rosbot" xmlns:xacro="http://www.ros.org/wiki/xacro">
   <xacro:arg name="use_sim" default="false" />
-  <xacro:arg name="use_gpu" default="false" />
   <xacro:arg name="mecanum" default="false" />
-  <xacro:arg name="simulation_engine" default="ignition-gazebo" />
   <xacro:arg name="namespace" default="None" />
   <xacro:include filename="$(find rosbot_description)/urdf/rosbot_macro.urdf.xacro" ns="husarion" />
-  <xacro:husarion.rosbot_robot
+  <xacro:husarion.rosbot
     mecanum="$(arg mecanum)"
     use_sim="$(arg use_sim)"
-    use_gpu="$(arg use_gpu)"
-    simulation_engine="$(arg simulation_engine)"
     namespace="$(arg namespace)" />
-    <xacro:include filename="$(find ros_components_description)/urdf/slamtec_rplidar_a2.urdf.xacro" ns="lidar" />
-    <xacro:lidar.slamtec_rplidar_a2
+    <xacro:include filename="$(find ros_components_description)/urdf/slamtec_rplidar.urdf.xacro" ns="lidar" />
+    <xacro:lidar.slamtec_rplidar
       parent_link="cover_link"
       xyz="0.02 0.0 0.0"
       rpy="0.0 0.0 0.0"
-      use_gpu="$(arg use_gpu)"
-      namespace="$(arg namespace)"
-      simulation_engine="$(arg simulation_engine)" />
-    <xacro:include filename="$(find ros_components_description)/urdf/orbbec_astra.urdf.xacro" ns="camera" />
-    <xacro:camera.orbbec_astra
-      parent_link="camera_link"
-      xyz="0.0 0.0 0.0"
-      rpy="0.0 0.0 0.0"
-      namespace="$(arg namespace)"
-      simulation_engine="$(arg simulation_engine)" />
+      model="s2"
+      namespace="$(arg namespace)" />
+	<xacro:include filename="$(find depthai_descriptions)/urdf/include/depthai_macro.urdf.xacro" ns="camera" />
+	<xacro:camera.depthai_camera camera_name="oak_camera" parent="camera_mount_link"
+		camera_model="OAK-D-PRO" base_frame="oak_camera"
+		cam_pos_x="0.0" cam_pos_y="0.0" cam_pos_z="0.02"
+		cam_roll="0.0" cam_pitch="0.0" cam_yaw="0.0"
+    r="0.2" g="0.2" b="0.2" a="1.0"	rs_compat="false" simulation="$(arg use_sim)" />
 </robot>

File: rosbot_description/urdf/rosbot_macro.urdf.xacro (robot description, xacro)
@@ -1,22 +1,12 @@
 <?xml version='1.0'?>
 <robot xmlns:xacro="http://wiki.ros.org/xacro">
-  <xacro:macro name="rosbot_robot" params="mecanum use_sim use_gpu simulation_engine namespace ">
-    <xacro:if value="${namespace == 'None'}">
-      <xacro:property name="namespace_ext" value="" />
-    </xacro:if>
-    <xacro:unless value="${namespace == 'None'}">
-        <xacro:property name="namespace_ext" value="${namespace}/" />
-    </xacro:unless>
-    <xacro:if value="${mecanum}">
-      <xacro:property name="wheel_radius" value="0.0470" />
-    </xacro:if>
-    <xacro:unless value="${mecanum}">
-      <xacro:property name="wheel_radius" value="0.0425" />
-    </xacro:unless>
+  <xacro:macro name="rosbot" params="mecanum use_sim namespace">
+    <xacro:property name="ns" value="${namespace + '/' if namespace != 'None' else ''}" />
+    <xacro:property name="wheel_radius" value="${0.0470 if mecanum else 0.0425}" />
     <!-- INCLUDE ROBOT PARTS DEFINITIONS -->
     <xacro:include filename="$(find rosbot_description)/urdf/body.urdf.xacro" ns="body" />
     <xacro:include filename="$(find rosbot_description)/urdf/wheel.urdf.xacro" ns="wheel" />
     <!-- BODY DECLARATION -->
-    <xacro:body.body wheel_radius="${wheel_radius}" mecanum="${mecanum}" use_gpu="${use_gpu}" namespace="${namespace}" />
+    <xacro:body.body wheel_radius="${wheel_radius}" mecanum="${mecanum}" namespace="${namespace}" />
     <!-- WHEEL DECLARATION -->
     <xacro:wheel.wheel wheel_radius="${wheel_radius}" side="fr" mecanum="${mecanum}" />
@@ -26,11 +16,11 @@
     <!-- ROS2 CONTROL -->
     <xacro:unless value="$(arg use_sim)">
-      <ros2_control name="${namespace_ext}imu" type="sensor">
+      <ros2_control name="${ns}imu" type="sensor">
         <hardware>
           <plugin>rosbot_hardware_interfaces/RosbotImuSensor</plugin>
-          <param name="connection_timeout_ms">120000</param>
-          <param name="connection_check_period_ms">500</param>
+          <param name="connection_timeout_ms">30000</param>
+          <param name="connection_check_period_ms">1000</param>
         </hardware>
-        <sensor name="${namespace_ext}imu">
+        <sensor name="${ns}imu">
           <state_interface name="orientation.x" />
           <state_interface name="orientation.y" />
@@ -46,10 +36,10 @@
       </ros2_control>
     </xacro:unless>
-    <ros2_control name="${namespace_ext}wheels" type="system">
+    <ros2_control name="${ns}rosbot_system" type="system">
       <hardware>
         <xacro:unless value="$(arg use_sim)">
           <plugin>rosbot_hardware_interfaces/RosbotSystem</plugin>
-          <param name="connection_timeout_ms">120000</param>
-          <param name="connection_check_period_ms">500</param>
+          <param name="connection_timeout_ms">30000</param>
+          <param name="connection_check_period_ms">1000</param>
           <!-- Firmware from https://github.com/husarion/rosbot_ros2_firmware could not override this names -->
           <param name="velocity_command_joint_order">
@@ -61,10 +51,5 @@
         </xacro:unless>
         <xacro:if value="$(arg use_sim)">
-          <xacro:if value="${simulation_engine == 'ignition-gazebo'}">
-            <plugin>gz_ros2_control/GazeboSimSystem</plugin>
-          </xacro:if>
-          <xacro:if value="${simulation_engine == 'webots'}">
-            <plugin>webots_ros2_control::Ros2ControlSystem</plugin>
-          </xacro:if>
+          <plugin>gz_ros2_control/GazeboSimSystem</plugin>
         </xacro:if>
       </hardware>
@@ -90,117 +75,49 @@
       </joint>
       <xacro:if value="${use_sim}">
-        <xacro:if value="${simulation_engine == 'ignition-gazebo'}">
-          <sensor name="${namespace_ext}imu">
-            <state_interface name="orientation.x" />
-            <state_interface name="orientation.y" />
-            <state_interface name="orientation.z" />
-            <state_interface name="orientation.w" />
-            <state_interface name="angular_velocity.x" />
-            <state_interface name="angular_velocity.y" />
-            <state_interface name="angular_velocity.z" />
-            <state_interface name="linear_acceleration.x" />
-            <state_interface name="linear_acceleration.y" />
-            <state_interface name="linear_acceleration.z" />
-          </sensor>
-        </xacro:if>
+        <sensor name="${ns}imu">
+          <state_interface name="orientation.x" />
+          <state_interface name="orientation.y" />
+          <state_interface name="orientation.z" />
+          <state_interface name="orientation.w" />
+          <state_interface name="angular_velocity.x" />
+          <state_interface name="angular_velocity.y" />
+          <state_interface name="angular_velocity.z" />
+          <state_interface name="linear_acceleration.x" />
+          <state_interface name="linear_acceleration.y" />
+          <state_interface name="linear_acceleration.z" />
+        </sensor>
       </xacro:if>
     </ros2_control>
     <!-- GAZEBO PLUGINS DECLARATION -->
     <xacro:if value="${use_sim}">
-      <xacro:if value="${simulation_engine == 'ignition-gazebo'}">
-        <gazebo>
-          <plugin filename="gz_ros2_control-system" name="gz_ros2_control::GazeboSimROS2ControlPlugin">
-            <xacro:if value="${mecanum}">
-              <parameters>$(find rosbot_controller)/config/mecanum_drive_controller.yaml</parameters>
-            </xacro:if>
-            <xacro:unless value="${mecanum}">
-              <parameters>$(find rosbot_controller)/config/diff_drive_controller.yaml</parameters>
+      <gazebo>
+        <plugin filename="gz_ros2_control-system" name="gz_ros2_control::GazeboSimROS2ControlPlugin">
+          <xacro:if value="${mecanum}">
+            <parameters>$(find rosbot_controller)/config/mecanum_drive_controller.yaml</parameters>
+          </xacro:if>
+          <xacro:unless value="${mecanum}">
+            <parameters>$(find rosbot_controller)/config/diff_drive_controller.yaml</parameters>
+          </xacro:unless>
+          <ros>
+            <xacro:unless value="${namespace == 'None'}">
+              <namespace>${namespace}</namespace>
             </xacro:unless>
-            <ros>
-              <xacro:unless value="${namespace == 'None'}">
-                <namespace>${namespace}</namespace>
-              </xacro:unless>
-              <remapping>rosbot_base_controller/cmd_vel:=cmd_vel</remapping>
-              <remapping>/tf:=tf</remapping>
-            </ros>
-          </plugin>
-        </gazebo>
-        <gazebo reference="imu_link">
-          <sensor name="${namespace_ext}imu" type="imu">
-            <always_on>true</always_on>
-            <update_rate>25</update_rate>
-            <topic>${namespace_ext}imu/data_raw</topic>
-            <visualize>false</visualize>
-            <enable_metrics>false</enable_metrics>
-            <frame_id>imu_link</frame_id>
-            <ignition_frame_id>imu_link</ignition_frame_id>
-            <ros>
-              <namespace>${namespace_ext}</namespace>
-            </ros>
-          </sensor>
-        </gazebo>
-      </xacro:if>
-      <xacro:if value="${simulation_engine == 'gazebo-classic'}">
-        <!-- Control robot wheels -->
-        <xacro:unless value="${mecanum}">
-          <gazebo>
-            <plugin name='skid_steer_drive' filename='libgazebo_ros_diff_drive.so'>
-              <ros></ros>
-              <update_rate>10.0</update_rate>
-              <num_wheel_pairs>2</num_wheel_pairs>
-              <left_joint>fl_wheel_joint</left_joint>
-              <right_joint>fr_wheel_joint</right_joint>
-              <left_joint>rl_wheel_joint</left_joint>
-              <right_joint>rr_wheel_joint</right_joint>
-              <wheel_separation>0.192</wheel_separation>
-              <wheel_separation>0.192</wheel_separation>
-              <wheel_diameter>${wheel_radius*2.0}</wheel_diameter>
-              <wheel_diameter>${wheel_radius*2.0}</wheel_diameter>
-              <max_wheel_torque>1.5</max_wheel_torque>
-              <max_wheel_acceleration>1.0</max_wheel_acceleration>
-              <publish_odom>true</publish_odom>
-              <publish_odom_tf>true</publish_odom_tf>
-              <publish_wheel_tf>true</publish_wheel_tf>
-              <odometry_frame>odom</odometry_frame>
-              <robot_base_frame>base_link</robot_base_frame>
-            </plugin>
-          </gazebo>
-        </xacro:unless>
-        <!-- publish joint states -->
-        <gazebo>
-          <plugin name="joint_states" filename="libgazebo_ros_joint_state_publisher.so">
-            <joint_name>fl_wheel_joint</joint_name>
-            <joint_name>fr_wheel_joint</joint_name>
-            <joint_name>rl_wheel_joint</joint_name>
-            <joint_name>rr_wheel_joint</joint_name>
-          </plugin>
-        </gazebo>
-        <!-- publish IMU -->
-        <gazebo reference="imu_link">
-          <sensor type="imu" name="imu">
-            <always_on>true</always_on>
-            <update_rate>25</update_rate>
-            <plugin name="bno055_imu_plugin" filename="libgazebo_ros_imu_sensor.so">
-              <ros>
-                <argument>~/out:=imu/data/raw</argument>
-              </ros>
-            </plugin>
-          </sensor>
-        </gazebo>
-      </xacro:if>
-      <xacro:if value="${simulation_engine == 'webots'}">
-        <webots>
-          <plugin type="webots_ros2_control::Ros2Control" />
-          <plugin type="webots_ros2_driver::Ros2IMU">
-            <enabled>true</enabled>
-            <topicName>/imu_broadcaster/imu</topicName>
-            <alwaysOn>true</alwaysOn>
-            <frameName>imu_link</frameName>
-            <gyroName>imu gyro</gyroName>
-            <accelerometerName>imu accelerometer</accelerometerName>
-            <inertialUnitName>imu inertial_unit</inertialUnitName>
-          </plugin>
-        </webots>
-      </xacro:if>
+            <remapping>rosbot_base_controller/cmd_vel:=cmd_vel</remapping>
+          </ros>
+        </plugin>
+      </gazebo>
+      <gazebo reference="imu_link">
+        <sensor name="${ns}imu" type="imu">
+          <always_on>true</always_on>
+          <update_rate>25</update_rate>
+          <topic>imu/data_raw</topic>
+          <visualize>false</visualize>
+          <enable_metrics>false</enable_metrics>
+          <gz_frame_id>imu_link</gz_frame_id>
+          <ros>
+            <namespace>${namespace}</namespace>
+          </ros>
+        </sensor>
+      </gazebo>
     </xacro:if>
   </xacro:macro>
