Commit message: added namespace to urdf
Signed-off-by: Jakub Delicat <jakub.delicat@husarion.com>

File: rosbot_description/urdf/rosbot.urdf.xacro (robot description, xacro)
@@ -7,4 +7,5 @@
   <xacro:arg name="simulation_engine" default="" />
   <xacro:arg name="tf_prefix" default="" />
+  <xacro:arg name="namespace" default="" />
   <xacro:property name="prefix" value="$(arg tf_prefix)" lazy_eval="false"/>
   <xacro:if value="${prefix != ''}">
@@ -18,5 +19,6 @@
     use_gpu="$(arg use_gpu)"
     simulation_engine="$(arg simulation_engine)"
-    tf_prefix="$(arg tf_prefix)" />
+    tf_prefix="$(arg tf_prefix)"
+    namespace="$(arg namespace)" />
   <!-- Include slamtec_rplidar_a2.urdf.xacro -->
   <xacro:include filename="$(find ros_components_description)/urdf/slamtec_rplidar_a2.urdf.xacro" ns="lidar" />

File: rosbot_description/urdf/rosbot_macro.urdf.xacro (robot description, xacro)
@@ -1,5 +1,5 @@
 <?xml version='1.0'?>
 <robot xmlns:xacro="http://wiki.ros.org/xacro">
-  <xacro:macro name="rosbot_robot" params="mecanum use_sim use_gpu tf_prefix simulation_engine">
+  <xacro:macro name="rosbot_robot" params="mecanum use_sim use_gpu tf_prefix namespace simulation_engine">
     <xacro:if value="${mecanum}">
       <xacro:property name="wheel_radius" value="0.0470" />
@@ -8,4 +8,8 @@
       <xacro:property name="wheel_radius" value="0.0425" />
     </xacro:unless>
+    <xacro:property name="namespace" value="$(arg namespace)" lazy_eval="false"/>
+    <xacro:if value="${namespace != ''}">
+      <xacro:property name="namespace" value="$(arg namespace)/" />
+    </xacro:if>
     <xacro:property name="prefix" value="${tf_prefix}" lazy_eval="false"/>
     <xacro:if value="${prefix != ''}">
@@ -59,5 +63,5 @@
                 fl_wheel_joint
           </param>
-          <param name="tf_prefix">${prefix}</param>
+          <param name="tf_prefix">${namespace}${prefix}</param>
         </xacro:unless>
         <xacro:if value="$(arg use_sim)">
@@ -70,20 +74,20 @@
         </xacro:if>
       </hardware>
-      <joint name="${prefix}fl_wheel_joint">
-        <command_interface name="velocity" />
-        <state_interface name="position" />
-        <state_interface name="velocity" />
-      </joint>
-      <joint name="${prefix}fr_wheel_joint">
-        <command_interface name="velocity" />
-        <state_interface name="position" />
-        <state_interface name="velocity" />
-      </joint>
-      <joint name="${prefix}rl_wheel_joint">
-        <command_interface name="velocity" />
-        <state_interface name="position" />
-        <state_interface name="velocity" />
-      </joint>
-      <joint name="${prefix}rr_wheel_joint">
+      <joint name="${namespace}${prefix}fl_wheel_joint">
+        <command_interface name="velocity" />
+        <state_interface name="position" />
+        <state_interface name="velocity" />
+      </joint>
+      <joint name="${namespace}${prefix}fr_wheel_joint">
+        <command_interface name="velocity" />
+        <state_interface name="position" />
+        <state_interface name="velocity" />
+      </joint>
+      <joint name="${namespace}${prefix}rl_wheel_joint">
+        <command_interface name="velocity" />
+        <state_interface name="position" />
+        <state_interface name="velocity" />
+      </joint>
+      <joint name="${namespace}${prefix}rr_wheel_joint">
         <command_interface name="velocity" />
         <state_interface name="position" />

Commit message: parse robots arg | removed delays from rosbot_controller
Signed-off-by: Jakub Delicat <jakub.delicat@husarion.com>

File: rosbot_description/urdf/rosbot.urdf.xacro (robot description, xacro)
@@ -6,5 +6,4 @@
   <xacro:arg name="simulation_engine" default="" />
   <xacro:arg name="namespace" default="None" />
-  <xacro:arg name="use_multirobot_system" default="false"/>
   <xacro:include filename="$(find rosbot_description)/urdf/rosbot_macro.urdf.xacro" ns="husarion" />
   <xacro:husarion.rosbot_robot
@@ -13,6 +12,5 @@
     use_gpu="$(arg use_gpu)"
     simulation_engine="$(arg simulation_engine)"
-    namespace="$(arg namespace)"
-    use_multirobot_system="$(arg use_multirobot_system)" />
+    namespace="$(arg namespace)" />
     <xacro:include filename="$(find ros_components_description)/urdf/slamtec_rplidar_a2.urdf.xacro" ns="lidar" />
       <xacro:lidar.slamtec_rplidar_a2

File: rosbot_description/urdf/rosbot_macro.urdf.xacro (robot description, xacro)
@@ -1,10 +1,12 @@
 <?xml version='1.0'?>
 <robot xmlns:xacro="http://wiki.ros.org/xacro">
-  <xacro:macro name="rosbot_robot" params="mecanum use_sim use_gpu simulation_engine namespace use_multirobot_system">
+  <xacro:macro name="rosbot_robot" params="mecanum use_sim use_gpu simulation_engine namespace ">
     <xacro:if value="${namespace == 'None'}">
-      <xacro:property name="namespace_ext" value="" />
+      <xacro:property name="namespace_ext" value="/" />
+      <xacro:property name="gz_control_namespace" value="/" />
     </xacro:if>
     <xacro:unless value="${namespace == 'None'}">
         <xacro:property name="namespace_ext" value="${namespace}/" />
+        <xacro:property name="gz_control_namespace" value="${namespace}" />
     </xacro:unless>
     <xacro:if value="${mecanum}">
@@ -111,10 +113,4 @@
         <gazebo>
           <plugin filename="ign_ros2_control-system" name="ign_ros2_control::IgnitionROS2ControlPlugin">
-            <xacro:if value="${use_multirobot_system}">
-              <xacro:property name="controller_config_prefix" value="" />
-            </xacro:if>
-            <xacro:unless value="${use_multirobot_system}">
-              <xacro:property name="controller_config_prefix" value="" />
-            </xacro:unless>
             <xacro:if value="${mecanum}">
               <parameters>$(find rosbot_controller)/config/mecanum_drive_controller.yaml</parameters>
@@ -124,5 +120,5 @@
             </xacro:unless>
             <ros>
-              <namespace>${namespace}</namespace>
+              <namespace>${gz_control_namespace}</namespace>
               <remapping>rosbot_base_controller/cmd_vel_unstamped:=cmd_vel</remapping>
               <remapping>/tf:=tf</remapping>
@@ -141,5 +137,5 @@
             <xacro:unless value="${namespace == 'None'}">
               <ros>
-                <namespace>${namespace}</namespace>
+                <namespace>${namespace_ext}</namespace>
               </ros>
             </xacro:unless>

Commit message: Fix imu namespace

File: rosbot_description/urdf/rosbot.urdf.xacro (robot description, xacro)
@@ -5,4 +5,5 @@
   <xacro:arg name="simulation_engine" default="ignition-gazebo" />
   <xacro:arg name="namespace" default="None" />
+  <xacro:arg name="controller_config" default="" />
   <xacro:include filename="$(find rosbot_description)/urdf/rosbot_macro.urdf.xacro" ns="husarion" />
   <xacro:husarion.rosbot_robot
@@ -10,5 +11,6 @@
     use_sim="$(arg use_sim)"
     simulation_engine="$(arg simulation_engine)"
-    namespace="$(arg namespace)" />
+    namespace="$(arg namespace)"
+    controller_config="$(arg controller_config)" />
     <xacro:include filename="$(find ros_components_description)/urdf/slamtec_rplidar_a2.urdf.xacro" ns="lidar" />
     <xacro:lidar.slamtec_rplidar_a2

File: rosbot_description/urdf/rosbot_macro.urdf.xacro (robot description, xacro)
@@ -1,5 +1,5 @@
 <?xml version='1.0'?>
 <robot xmlns:xacro="http://wiki.ros.org/xacro">
-  <xacro:macro name="rosbot_robot" params="mecanum use_sim simulation_engine namespace ">
+  <xacro:macro name="rosbot_robot" params="mecanum use_sim simulation_engine namespace controller_config">
     <xacro:property name="ns" value="${namespace + '/' if namespace != 'None' else ''}" />
     <xacro:property name="wheel_radius" value="${0.0470 if mecanum else 0.0425}" />
@@ -101,10 +101,5 @@
         <gazebo>
           <plugin filename="ign_ros2_control-system" name="ign_ros2_control::IgnitionROS2ControlPlugin">
-            <xacro:if value="${mecanum}">
-              <parameters>$(find rosbot_controller)/config/mecanum_drive_controller.yaml</parameters>
-            </xacro:if>
-            <xacro:unless value="${mecanum}">
-              <parameters>$(find rosbot_controller)/config/diff_drive_controller.yaml</parameters>
-            </xacro:unless>
+            <parameters>${controller_config}</parameters>
             <ros>
               <xacro:unless value="${namespace == 'None'}">
