Commit message: Unify with Humble

File: rosbot_description/urdf/rosbot_xl.urdf.xacro (robot description, xacro)
@@ -5,8 +5,8 @@
   <xacro:arg name="controller_config" default="" />
   <xacro:arg name="include_camera_mount" default="false" />
+  <xacro:arg name="manipulator_serial_port" default="/dev/ttyUSB0" />
   <xacro:arg name="mecanum" default="false" />
   <xacro:arg name="namespace" default="" />
   <xacro:arg name="use_sim" default="false" />
-  <xacro:arg name="manipulator_serial_port" default="/dev/ttyUSB0" />
   <xacro:include filename="$(find rosbot_description)/urdf/rosbot_xl/rosbot_xl_macro.urdf.xacro" ns="husarion" />
   <xacro:include filename="$(find ros_components_description)/urdf/components.urdf.xacro" ns="components" />

File: rosbot_description/urdf/rosbot_xl/components/antenna.urdf.xacro (robot description, xacro)
@@ -8,4 +8,6 @@
                        antenna_angle:=0.0">
     <xacro:property name="prefix" value="${tf_prefix + '_' if tf_prefix != '' else ''}" />
+    <xacro:property name="antenna_connector_length" value="0.02" />
+    <xacro:property name="antenna_connector_radius" value="0.007" />
     <xacro:property name="antenna_length" value="0.1" />
     <xacro:property name="antenna_radius" value="0.0052" />
@@ -23,4 +25,10 @@
         <origin xyz="0.0 0.0 0.0" rpy="0.0 0.0 0.0" />
       </visual>
+      <collision>
+        <geometry>
+          <cylinder radius="${antenna_connector_radius}" length="${antenna_connector_length}" />
+        </geometry>
+        <origin xyz="-0.005 0.0 0.0" rpy="0.0 ${-pi/4} 0.0" />
+      </collision>
     </link>
     <joint name="${prefix}antenna_connector_to_${prefix}antenna_joint" type="fixed">

File: rosbot_description/urdf/rosbot_xl/rosbot_xl_macro.urdf.xacro (robot description, xacro)
@@ -19,5 +19,5 @@
     <!-- BODY -->
     <xacro:body.body wheel_radius="${wheel_radius}" />
-    <xacro:antenna.antenna parent_link="cover_link" xyz="-0.155 -0.055 -0.02" />
+    <xacro:antenna.antenna parent_link="cover_link" xyz="-0.155 -0.055 -0.02" rpy="-0.4 0.0 0.0" antenna_angle="0.3" />
     <xacro:if value="${include_camera_mount}">
       <xacro:camera_mount.camera_mount parent_link="cover_link" xyz="-0.1 0.0 0.0" />

Commit message: Cleanup: soft-derive components_config, rename helper, document pre-commit
1. rosbot_xl.urdf.xacro now derives components_config from configuration when
   the former is left empty (soft compat: explicit components_config still
   wins). Removes a two-source-of-truth drift hazard where calling xacro
   with `configuration:=manipulation` but no `components_config` produced a
   robot with the manipulator macro but basic.yaml components.
   test_components_config_derived_from_configuration guards the derivation.

2. rosbot_bringup/test/test_utils.py -> bringup_helpers.py. The file ships
   classes/functions used by test_bringup.py, not tests; pytest no longer
   collects it as a test file (no need for __test__ = False sentinel).

3. CONTRIBUTING.md gains a short Auto-fix workflow section: run pre-commit
   on staged files before `git commit` to avoid the auto-fix -> commit
   abort -> re-stage cycle that bites on every batch commit.

File: rosbot_description/urdf/rosbot_xl.urdf.xacro (robot description, xacro)
@@ -1,5 +1,5 @@
 <?xml version='1.0'?>
 <robot name="rosbot_xl" xmlns:xacro="http://www.ros.org/wiki/xacro">
-  <xacro:arg name="components_config" default="$(find rosbot_description)/config/rosbot_xl/basic.yaml" />
+  <xacro:arg name="components_config" default="" />
   <xacro:arg name="configuration" default="basic" />
   <xacro:arg name="controller_config" default="" />
@@ -9,4 +9,8 @@
   <xacro:arg name="namespace" default="" />
   <xacro:arg name="use_sim" default="False" />
+  <!-- Soft compat: if components_config is not given explicitly, derive it
+       from configuration so the two stay in sync. -->
+  <xacro:property name="components_config_resolved"
+    value="${'$(arg components_config)' if '$(arg components_config)' else '$(find rosbot_description)/config/rosbot_xl/$(arg configuration).yaml'}" />
   <xacro:include filename="$(find rosbot_description)/urdf/rosbot_xl/rosbot_xl_macro.urdf.xacro" ns="husarion" />
   <xacro:include filename="$(find husarion_components_description)/urdf/components.urdf.xacro" ns="components" />
@@ -18,5 +22,5 @@
     use_sim="$(arg use_sim)" />
   <xacro:components.create_components
-    components_config_path="$(arg components_config)"
+    components_config_path="${components_config_resolved}"
     namespace="$(arg namespace)"
     use_sim="$(arg use_sim)"
