Commit message: Move camera_mount to a custom yaml component for ROSbot XL
Was built into rosbot_xl_macro.urdf.xacro behind an internal
include_camera_mount toggle; now telepresence.yaml/autonomy.yaml add
it as a `type: custom` component (like man01_bracket), with
camera_mount_angle_1/2 read straight off that yaml entry via the
new husarion_components_description `component` passthrough (bumped
pin: f059bb6 -> 5f783f8).

File: rosbot_description/urdf/rosbot_xl.urdf.xacro (robot description, xacro)
@@ -4,5 +4,4 @@
   <xacro:arg name="configuration" default="basic" />
   <xacro:arg name="controller_config" default="" />
-  <xacro:arg name="include_camera_mount" default="False" />
   <xacro:arg name="manipulator_serial_port" default="/dev/ttyUSB0" />
   <xacro:arg name="mecanum" default="False" />
@@ -17,5 +16,4 @@
   <xacro:husarion.rosbot_xl
     controller_config="$(arg controller_config)"
-    include_camera_mount="$(arg include_camera_mount)"
     mecanum="$(arg mecanum)"
     namespace="$(arg namespace)"

File: rosbot_description/urdf/rosbot_xl/components/camera_mount.urdf.xacro (robot description, xacro)
@@ -5,8 +5,17 @@
                        xyz:='0.0 0.0 0.0'
                        rpy:='0.0 0.0 0.0'
-                       tf_prefix:=''
-                       camera_mount_angle_1:=0.0
-                       camera_mount_angle_2:=0.0">
-    <xacro:property name="prefix" value="${tf_prefix + '_' if tf_prefix != '' else ''}" />
+                       robot_namespace:=''
+                       component_name:=''
+                       use_tf_prefix:=False
+                       component:={}">
+    <!-- default component_name left empty on purpose: this macro's own link
+         names (camera_mount_bot/mid/top/_link) are already fully qualified,
+         so a non-empty default here would double-prefix them. -->
+    <xacro:property name="prefix" value="${component_name + '_' if component_name != '' else ''}" />
+    <!-- camera_mount_angle_1/2 (rad) tune the bracket's pan/tilt joints - set them
+         directly on this component's yaml entry when a configuration needs a
+         different tilt than the physical bracket's own default. -->
+    <xacro:property name="camera_mount_angle_1" value="${component.get('camera_mount_angle_1', 0.0)}" />
+    <xacro:property name="camera_mount_angle_2" value="${component.get('camera_mount_angle_2', 0.0)}" />
     <joint name="${parent_link.rstrip('_link')}_to_${prefix}camera_mount_bot_joint"
       type="fixed">

File: rosbot_description/urdf/rosbot_xl/components/man01_bracket.urdf.xacro (robot description, xacro)
@@ -7,5 +7,6 @@
                        robot_namespace:=''
                        component_name:=''
-                       use_tf_prefix:=False">
+                       use_tf_prefix:=False
+                       component:={}">
     <xacro:if value="${component_name == ''}">
       <xacro:property name="component_name" value="man01_bracket" />

File: rosbot_description/urdf/rosbot_xl/rosbot_xl_macro.urdf.xacro (robot description, xacro)
@@ -3,5 +3,4 @@
   <xacro:macro name="rosbot_xl"
     params="controller_config
-            include_camera_mount
             mecanum
             namespace
@@ -16,11 +15,7 @@
     <xacro:include filename="$(find rosbot_description)/urdf/rosbot_xl/components/antenna.urdf.xacro" ns="antenna" />
     <xacro:include filename="$(find rosbot_description)/urdf/rosbot_xl/wheel.urdf.xacro" ns="wheel" />
-    <xacro:include filename="$(find rosbot_description)/urdf/rosbot_xl/components/camera_mount.urdf.xacro" ns="camera_mount" />
     <!-- BODY -->
     <xacro:body.body wheel_radius="${wheel_radius}" />
     <xacro:antenna.antenna parent_link="cover_link" xyz="-0.155 -0.055 -0.02" rpy="-0.4 0.0 0.0" antenna_angle="0.3" />
-    <xacro:if value="${include_camera_mount}">
-      <xacro:camera_mount.camera_mount parent_link="cover_link" xyz="-0.1 0.0 0.0" />
-    </xacro:if>
     <!-- WHEEL -->
     <xacro:wheel.wheel wheel_radius="${wheel_radius}" side="fl" mecanum="${mecanum}" />
