Commit message: Add special ROSbot XL nodes: battery_monitor, led_strip_animation

File: rosbot_description/urdf/common/gazebo.urdf.xacro (robot description, xacro)
@@ -41,6 +41,6 @@
       <sensor name="${ns}imu" type="imu">
         <always_on>true</always_on>
-        <update_rate>25</update_rate>
-        <topic>${ns}imu/data_raw</topic>
+        <update_rate>50</update_rate>
+        <topic>${ns}_imu/data</topic>
         <visualize>false</visualize>
         <enable_metrics>false</enable_metrics>

File: rosbot_description/urdf/rosbot/components/vl53lox.urdf.xacro (robot description, xacro)
@@ -10,9 +10,7 @@
     </joint>
     <link name="${prefix}_range" />
-    <!-- an IR sensor or a sonar are not implemented yet
-    https://github.com/gazebosim/gz-sensors/issues/19 -->
     <gazebo reference="${prefix}_range">
       <sensor name="${ns}${prefix}_range" type='gpu_lidar'>
-        <topic>${ns}range/${prefix}</topic>
+        <topic>${ns}ranges</topic>
         <gz_frame_id>${prefix}_range</gz_frame_id>
         <update_rate>5.0</update_rate>

File: rosbot_description/urdf/rosbot_xl/body.urdf.xacro (robot description, xacro)
@@ -36,5 +36,5 @@
     <link name="cover_link" />
     <joint name="body_to_imu_joint" type="fixed">
-      <origin xyz="-0.1369 -0.0419 0.0370" rpy="3.14159 0.0 0.0" />
+      <origin xyz="-0.1369 -0.0419 0.0370" rpy="0.0 0.0 0.0" />
       <parent link="body_link" />
       <child link="imu_link" />
