Commit message: Two controller_managers in sim too; full MoveIt model
Simulation now hosts manipulator_controller_manager in a second
gz_ros2_control plugin, so names and tooling match hardware; the
manipulator_ros2_control / spawn_controllers launch args and the
arm_control controller_manager argument are gone.

move_group and servo read robot_description from
robot_state_publisher instead of building it from manipulation.yaml,
which left manipulation_pro's bracket + ZED out of collision checking.
Existing config_dir copies need the updated rosbot_xl.srdf.

File: rosbot_description/urdf/common/gazebo.urdf.xacro (robot description, xacro)
@@ -1,8 +1,13 @@
 <?xml version="1.0" encoding="utf-8"?>
 <robot xmlns:xacro="http://wiki.ros.org/xacro">
-  <xacro:macro name="controller" params="config_file namespace:=''">
+  <!-- One plugin instance per controller_manager: the drive's controller_manager and the
+       arm's manipulator_controller_manager (which reads its arm-only description from
+       robot_description_topic, published by rosbot_controller/manipulator_supervisor). -->
+  <xacro:macro name="controller"
+    params="config_file namespace:='' controller_manager_name:=controller_manager robot_description_topic:=''">
+    <xacro:property name="cm" value="${controller_manager_name}" />
     <gazebo>
       <plugin filename="gz_ros2_control-system" name="gz_ros2_control::GazeboSimROS2ControlPlugin">
-        <controller_manager_name>controller_manager</controller_manager_name>
+        <controller_manager_name>${cm}</controller_manager_name>
         <parameters>${config_file}</parameters>
         <ros>
@@ -13,18 +18,21 @@
           <remapping>/tf:=tf</remapping>
           <remapping>/tf_static:=tf_static</remapping>
-          <remapping>/controller_manager/cleanup_controller:=controller_manager/cleanup_controller</remapping>
-          <remapping>/controller_manager/configure_controller:=controller_manager/configure_controller</remapping>
-          <remapping>/controller_manager/list_controllers:=controller_manager/list_controllers</remapping>
-          <remapping>/controller_manager/list_controller_types:=controller_manager/list_controller_types</remapping>
-          <remapping>/controller_manager/list_hardware_components:=controller_manager/list_hardware_components</remapping>
-          <remapping>/controller_manager/list_hardware_interfaces:=controller_manager/list_hardware_interfaces</remapping>
-          <remapping>/controller_manager/load_controller:=controller_manager/load_controller</remapping>
-          <remapping>/controller_manager/reload_controller_libraries:=controller_manager/reload_controller_libraries</remapping>
-          <remapping>/controller_manager/set_hardware_component_state:=controller_manager/set_hardware_component_state</remapping>
-          <remapping>/controller_manager/switch_controller:=controller_manager/switch_controller</remapping>
-          <remapping>/controller_manager/unload_controller:=controller_manager/unload_controller</remapping>
-          <remapping>/controller_manager/activity:=controller_manager/activity</remapping>
-          <remapping>/controller_manager/statistics:=controller_manager/statistics</remapping>
-          <remapping>/controller_manager/introspection_data:=controller_manager/introspection_data</remapping>
+          <remapping>/${cm}/cleanup_controller:=${cm}/cleanup_controller</remapping>
+          <remapping>/${cm}/configure_controller:=${cm}/configure_controller</remapping>
+          <remapping>/${cm}/list_controllers:=${cm}/list_controllers</remapping>
+          <remapping>/${cm}/list_controller_types:=${cm}/list_controller_types</remapping>
+          <remapping>/${cm}/list_hardware_components:=${cm}/list_hardware_components</remapping>
+          <remapping>/${cm}/list_hardware_interfaces:=${cm}/list_hardware_interfaces</remapping>
+          <remapping>/${cm}/load_controller:=${cm}/load_controller</remapping>
+          <remapping>/${cm}/reload_controller_libraries:=${cm}/reload_controller_libraries</remapping>
+          <remapping>/${cm}/set_hardware_component_state:=${cm}/set_hardware_component_state</remapping>
+          <remapping>/${cm}/switch_controller:=${cm}/switch_controller</remapping>
+          <remapping>/${cm}/unload_controller:=${cm}/unload_controller</remapping>
+          <remapping>/${cm}/activity:=${cm}/activity</remapping>
+          <remapping>/${cm}/statistics:=${cm}/statistics</remapping>
+          <remapping>/${cm}/introspection_data:=${cm}/introspection_data</remapping>
+          <xacro:if value="${robot_description_topic != ''}">
+            <remapping>robot_description:=${robot_description_topic}</remapping>
+          </xacro:if>
         </ros>
       </plugin>

File: rosbot_description/urdf/rosbot_xl.urdf.xacro (robot description, xacro)
@@ -7,7 +7,9 @@
   <xacro:arg name="mecanum" default="False" />
   <xacro:arg name="namespace" default="" />
-  <!-- On hardware the arm runs under its own controller_manager (see MANIPULATOR.md), so each
-       controller_manager gets a description with only its own <ros2_control> blocks. -->
-  <xacro:arg name="manipulator_ros2_control" default="True" />
+  <!-- The arm runs under its own manipulator_controller_manager (see MANIPULATOR.md), so each
+       controller_manager gets a description with only its own <ros2_control> blocks. The
+       defaults produce the drive's description; manipulator_supervisor builds the arm's with
+       robot_ros2_control:=False manipulator_ros2_control:=True. -->
+  <xacro:arg name="manipulator_ros2_control" default="False" />
   <xacro:arg name="robot_ros2_control" default="True" />
   <xacro:arg name="use_sim" default="False" />
@@ -38,4 +40,14 @@
       port_name="$(arg manipulator_serial_port)"
       ros2_control_enabled="$(arg manipulator_ros2_control)"/>
+    <xacro:if value="$(arg use_sim)">
+      <xacro:if value="$(arg robot_ros2_control)">
+        <xacro:include filename="$(find rosbot_description)/urdf/common/gazebo.urdf.xacro" ns="gazebo" />
+        <xacro:gazebo.controller
+          config_file="$(arg controller_config)"
+          namespace="$(arg namespace)"
+          controller_manager_name="manipulator_controller_manager"
+          robot_description_topic="manipulator_controller_manager/robot_description" />
+      </xacro:if>
+    </xacro:if>
   </xacro:if>
 </robot>

File: rosbot_description/urdf/rosbot_xl/rosbot_xl_macro.urdf.xacro (robot description, xacro)
@@ -33,7 +33,9 @@
     <!-- GAZEBO PLUGINS -->
     <xacro:if value="${use_sim}">
-      <xacro:ros2_control.gz_rosbot_system namespace="${namespace}" />
-      <xacro:gazebo.controller config_file="${controller_config}" namespace="${namespace}" />
-      <xacro:gazebo.imu reference_frame="imu_link" namespace="${namespace}" />
+      <xacro:if value="${ros2_control_enabled}">
+        <xacro:ros2_control.gz_rosbot_system namespace="${namespace}" />
+        <xacro:gazebo.controller config_file="${controller_config}" namespace="${namespace}" />
+        <xacro:gazebo.imu reference_frame="imu_link" namespace="${namespace}" />
+      </xacro:if>
       <!-- <xacro:if value="${simulation_engine == 'webots'}">
         <xacro:webots.controller />
