Commit message: Change cover plate color to black

File: rosbot_description/urdf/rosbot/body.urdf.xacro (robot description, xacro)
@@ -19,4 +19,7 @@
           <color rgba="0.1 0.1 0.1 1.0" />
         </material>
+        <gazebo reference="body_link">
+          <material>Gazebo/Black</material>
+        </gazebo>
       </visual>
       <collision>
@@ -34,7 +37,4 @@
       </inertial>
     </link>
-    <gazebo reference="body_link">
-      <material>Gazebo/Black</material>
-    </gazebo>
     <joint name="body_to_cover_joint" type="fixed">
       <origin xyz="0.0 0.0 0.0603" rpy="0.0 0.0 0.0" />
@@ -48,11 +48,11 @@
         </geometry>
         <origin xyz="0.0 0.0 -0.002" rpy="${pi/2} 0.0 ${pi/2}" />
-        <material name="Red">
-          <color rgba="0.8 0.0 0.0 1.0" />
+        <material name="Black">
+          <color rgba="0.1 0.1 0.1 1.0" />
         </material>
+        <gazebo reference="cover_link">
+          <material>Gazebo/Black</material>
+        </gazebo>
       </visual>
-      <gazebo reference="cover_link">
-        <material>Gazebo/Red</material>
-      </gazebo>
     </link>
     <joint name="body_to_imu_joint" type="fixed">

Commit message: Fixes

File: rosbot_description/urdf/rosbot/body.urdf.xacro (robot description, xacro)
@@ -16,9 +16,9 @@
         </geometry>
         <origin xyz="0.0 0.0 -0.0173" rpy="${pi/2} 0.0 ${pi/2}" />
-        <material name="Black">
-          <color rgba="0.1 0.1 0.1 1.0" />
+        <material name="White">
+          <color rgba="1.0 1.0 1.0 1.0" />
         </material>
         <gazebo reference="body_link">
-          <material>Gazebo/Black</material>
+          <material>Gazebo/White</material>
         </gazebo>
       </visual>
@@ -37,4 +37,7 @@
       </inertial>
     </link>
+    <gazebo reference="body_link">
+      <material>Gazebo/White</material>
+    </gazebo>
     <joint name="body_to_cover_joint" type="fixed">
       <origin xyz="0.0 0.0 0.0603" rpy="0.0 0.0 0.0" />
@@ -48,11 +51,11 @@
         </geometry>
         <origin xyz="0.0 0.0 -0.002" rpy="${pi/2} 0.0 ${pi/2}" />
-        <material name="Black">
-          <color rgba="0.1 0.1 0.1 1.0" />
+        <material name="Red">
+          <color rgba="0.8 0.0 0.0 1.0" />
         </material>
-        <gazebo reference="cover_link">
-          <material>Gazebo/Black</material>
-        </gazebo>
       </visual>
+      <gazebo reference="cover_link">
+        <material>Gazebo/Red</material>
+      </gazebo>
     </link>
     <joint name="body_to_imu_joint" type="fixed">

File: rosbot_description/urdf/rosbot/wheel.urdf.xacro (robot description, xacro)
@@ -78,5 +78,5 @@
       </inertial>
     </link>
-    <gazebo reference="${side}_wheel_link" xmlns:gz="http://gazeborobotics.org/schema">
+    <gazebo reference="${side}_wheel_link" xmlns:ignition="http://gazeborobotics.org/schema">
       <xacro:unless value="${mecanum}">
         <collision>
@@ -103,5 +103,5 @@
                   <slip1>0.035</slip1>
                 <slip2>0</slip2>
-                <fdir1 gz:expressed_in="base_link">${fdir}</fdir1>
+                <fdir1 ignition:expressed_in="base_link">${fdir}</fdir1>
               </ode>
             </friction>

File: rosbot_description/urdf/rosbot_xl/wheel.urdf.xacro (robot description, xacro)
@@ -77,5 +77,5 @@
       </inertial>
     </link>
-    <gazebo reference="${side}_wheel_link" xmlns:gz="http://gazeborobotics.org/schema">
+    <gazebo reference="${side}_wheel_link" xmlns:ignition="http://gazeborobotics.org/schema">
       <xacro:unless value="${mecanum}">
         <collision>
@@ -102,5 +102,5 @@
                   <slip1>0.035</slip1>
                 <slip2>0</slip2>
-                <fdir1 gz:expressed_in="base_link">${fdir}</fdir1>
+                <fdir1 ignition:expressed_in="base_link">${fdir}</fdir1>
               </ode>
             </friction>

Commit message: Update rosbot body mesh; retune camera mount; bump husarion_components_description

File: rosbot_description/urdf/rosbot/body.urdf.xacro (robot description, xacro)
@@ -12,14 +12,8 @@
     <link name="body_link">
       <visual>
+        <origin xyz="0.0 0.0 -0.0173" rpy="${pi/2} 0.0 ${pi/2}" />
         <geometry>
-          <mesh filename="package://rosbot_description/meshes/rosbot/body.stl" scale="0.001 0.001 0.001" />
+          <mesh filename="package://rosbot_description/meshes/rosbot/body.glb" scale="0.001 0.001 0.001" />
         </geometry>
-        <origin xyz="0.0 0.0 -0.0173" rpy="${pi/2} 0.0 ${pi/2}" />
-        <material name="Black">
-          <color rgba="0.1 0.1 0.1 1.0" />
-        </material>
-        <gazebo reference="body_link">
-          <material>Gazebo/Black</material>
-        </gazebo>
       </visual>
       <collision>
@@ -42,18 +36,5 @@
       <child link="cover_link" />
     </joint>
-    <link name="cover_link">
-      <visual>
-        <geometry>
-          <mesh filename="package://rosbot_description/meshes/rosbot/cover.stl" scale="0.001 0.001 0.001" />
-        </geometry>
-        <origin xyz="0.0 0.0 -0.002" rpy="${pi/2} 0.0 ${pi/2}" />
-        <material name="Black">
-          <color rgba="0.1 0.1 0.1 1.0" />
-        </material>
-        <gazebo reference="cover_link">
-          <material>Gazebo/Black</material>
-        </gazebo>
-      </visual>
-    </link>
+    <link name="cover_link" />
     <joint name="body_to_imu_joint" type="fixed">
       <origin xyz="0.003 -0.0495 0.04332" rpy="0.0 0.0 0.0" />
@@ -63,5 +44,5 @@
     <link name="imu_link" />
     <joint name="body_to_camera_joint" type="fixed">
-      <origin xyz="-0.0141 0.0 0.125" rpy="0.0 0.0 0.0" />
+      <origin xyz="0.0179 0.0 0.144" rpy="0.0 0.0 0.0" />
       <parent link="body_link" />
       <child link="camera_mount_link" />
