Commit message: Rework wheel meshes to GLB, add camera collision geometry
wheel/mecanum meshes converted dae->glb; wheel_l/wheel_r are re-extracted
from the ROSbot-3-PRO reference CAD (real rim+tire geometry, metallic rim
/ rubber tire materials) replacing the old low-poly placeholder, while
mecanum_l/mecanum_r are a decimated conversion of the existing mesh
(original ~5MB exceeded the repo's 3MB pre-commit limit).

camera_mount_link gets a collision (previously none) - a simplified STL
of the CAD camera holder bracket, since its shape (two tapering legs)
doesn't reduce well to box/cylinder primitives.

Bump husarion_components_description: depthai_descriptions ships OAK
camera models with visual-only meshes, no collision geometry.

File: rosbot_description/urdf/rosbot/body.urdf.xacro (robot description, xacro)
@@ -48,5 +48,12 @@
       <child link="camera_mount_link" />
     </joint>
-    <link name="camera_mount_link" />
+    <link name="camera_mount_link">
+      <collision>
+        <geometry>
+          <mesh filename="package://rosbot_description/meshes/rosbot/camera_holder_collision.stl" scale="0.001 0.001 0.001" />
+        </geometry>
+        <origin xyz="-0.0179 0.0 -0.1613" rpy="${pi/2} 0.0 ${pi/2}" />
+      </collision>
+    </link>
     <xacro:range_sensor.vl53lox parent="body_link" xyz="0.0926  0.05 0.015"   rpy="0.0 0.0 ${radians(12.5)}"  prefix="fl" namespace="${namespace}" />
     <xacro:range_sensor.vl53lox parent="body_link" xyz="0.0926 -0.05 0.015"   rpy="0.0 0.0 ${radians(-12.5)}" prefix="fr" namespace="${namespace}" />

File: rosbot_description/urdf/rosbot/wheel.urdf.xacro (robot description, xacro)
@@ -25,6 +25,6 @@
       <xacro:property name="x" value="${wheel_separation_x/2.0}" />
       <xacro:property name="y" value="${wheel_separation_y/2.0}" />
-      <xacro:property name="mesh" value="package://rosbot_description/meshes/rosbot/${wheel_file}_b.dae" />
-      <xacro:property name="visual_rotation" value="${pi}" />
+      <xacro:property name="mesh" value="package://rosbot_description/meshes/rosbot/${wheel_file}_l.glb" />
+      <xacro:property name="visual_rotation" value="${pi/2} 0.0 0.0" />
       <xacro:property name="fdir" value="1.0 -1.0 0.0" />
     </xacro:if>
@@ -32,6 +32,6 @@
       <xacro:property name="x" value="${wheel_separation_x/2.0}" />
       <xacro:property name="y" value="${-wheel_separation_y/2.0}" />
-      <xacro:property name="mesh" value="package://rosbot_description/meshes/rosbot/${wheel_file}_a.dae" />
-      <xacro:property name="visual_rotation" value="${pi}" />
+      <xacro:property name="mesh" value="package://rosbot_description/meshes/rosbot/${wheel_file}_r.glb" />
+      <xacro:property name="visual_rotation" value="${pi/2} 0.0 0.0" />
       <xacro:property name="fdir" value="1.0 1.0 0.0" />
     </xacro:if>
@@ -39,6 +39,6 @@
       <xacro:property name="x" value="${-wheel_separation_x/2.0}" />
       <xacro:property name="y" value="${wheel_separation_y/2.0}" />
-      <xacro:property name="mesh" value="package://rosbot_description/meshes/rosbot/${wheel_file}_a.dae" />
-      <xacro:property name="visual_rotation" value="${0.0}" />
+      <xacro:property name="mesh" value="package://rosbot_description/meshes/rosbot/${wheel_file}_l.glb" />
+      <xacro:property name="visual_rotation" value="${pi/2} 0.0 0.0" />
       <xacro:property name="fdir" value="1.0 1.0 0.0" />
     </xacro:if>
@@ -46,6 +46,6 @@
       <xacro:property name="x" value="${-wheel_separation_x/2.0}" />
       <xacro:property name="y" value="${-wheel_separation_y/2.0}" />
-      <xacro:property name="mesh" value="package://rosbot_description/meshes/rosbot/${wheel_file}_b.dae" />
-      <xacro:property name="visual_rotation" value="${0.0}" />
+      <xacro:property name="mesh" value="package://rosbot_description/meshes/rosbot/${wheel_file}_r.glb" />
+      <xacro:property name="visual_rotation" value="${pi/2} 0.0 0.0" />
       <xacro:property name="fdir" value="1.0 -1.0 0.0" />
     </xacro:if>
@@ -63,5 +63,5 @@
           <mesh filename="${mesh}" scale="1.0 1.0 1.0" />
         </geometry>
-        <origin xyz="0.0 0.0 0.0" rpy="0.0 0.0 ${visual_rotation}" />
+        <origin xyz="0.0 0.0 0.0" rpy="${visual_rotation}" />
       </visual>
       <collision>
